Commit message: Changed physics parameters

File: boot1_description/urdf/boot1.xacro (robot description, xacro)
@@ -39,5 +39,5 @@
     <origin rpy="0 0  0.0" xyz="0.0 0.0   -1.8"/>
     <axis xyz="0 1 0"/>
-    <limit effort="100.0" lower="-0.2" upper="0.2" velocity="1.0"/>
+    <limit effort="200.0" lower="-0.2" upper="0.2" velocity="1.0"/>
   </joint>
   <joint name="port_blade_joint" type="revolute">
@@ -46,11 +46,10 @@
     <origin rpy="0.0  0 0.0" xyz="0.0 0.0   1.8"/>
     <axis xyz="0 1 0"/>
-    <limit effort="100.0" lower="-0.2" upper="0.2" velocity="1.0"/>
-  </joint>
-  <!--   <link name="base_link"/> -->
-  <link name="world"/>
+    <limit effort="200.0" lower="-0.2" upper="0.2" velocity="1.0"/>
+  </joint>
+  <link name="base_link"/>
   <!-- Dummy for gazebo   -->
   <joint name="dummy" type="fixed">
-    <parent link="world"/>
+    <parent link="base_link"/>
     <child link="skiff"/>
   </joint>
@@ -123,5 +122,5 @@
       <origin rpy="0 0 0" xyz="0   0   -0.45"/>
       <geometry>
-        <cylinder length="2.7" radius="0.02"/>
+        <cylinder length="2.0" radius="0.02"/>
       </geometry>
     </collision>
@@ -142,5 +141,5 @@
       <origin rpy="0 0 0" xyz="0   0   0.45"/>
       <geometry>
-        <cylinder length="2.7" radius="0.02"/>  <!-- 2.0 to prevent collissions  -->
+        <cylinder length="2.0" radius="0.02"/>  <!-- 2.0 to prevent collissions  -->
       </geometry>
     </collision>

Commit message: =sdfsdf

File: boot1_description/urdf/boot1.xacro (robot description, xacro)
@@ -25,5 +25,5 @@
     <origin rpy="0.0  ${pi/2} -${pi/2}" xyz="0.0 0.0   0.02"/>
     <axis xyz="0 1 0"/>
-    <limit effort="200.0" lower="-0.4" upper="0.0" velocity="1.0"/>
+    <limit effort="1000.0" lower="-0.4" upper="0.0" velocity="1.0"/>
   </joint>
   <joint name="port_rowlock_oar_joint" type="revolute">
@@ -32,5 +32,5 @@
     <origin rpy="0.0  ${pi/2} -${pi/2}" xyz="0.0 0.0   0.02"/>
     <axis xyz="0 1 0"/>
-    <limit effort="200.0" lower="0.0" upper="0.4" velocity="1.0"/>
+    <limit effort="1000.0" lower="0.0" upper="0.4" velocity="1.0"/>
   </joint>
   <joint name="starboard_blade_joint" type="revolute">
@@ -39,5 +39,5 @@
     <origin rpy="0 0  0.0" xyz="0.0 0.0   -1.8"/>
     <axis xyz="0 1 0"/>
-    <limit effort="200.0" lower="-0.2" upper="0.2" velocity="1.0"/>
+    <limit effort="1000.0" lower="-0.4" upper="0.4" velocity="1.0"/>
   </joint>
   <joint name="port_blade_joint" type="revolute">
@@ -46,5 +46,5 @@
     <origin rpy="0.0  0 0.0" xyz="0.0 0.0   1.8"/>
     <axis xyz="0 1 0"/>
-    <limit effort="200.0" lower="-0.2" upper="0.2" velocity="1.0"/>
+    <limit effort="1000.0" lower="-0.4" upper="0.4" velocity="1.0"/>
   </joint>
   <link name="base_link"/>

Commit message: =pid blade changed, d=0

File: boot1_description/urdf/boot1.xacro (robot description, xacro)
@@ -9,5 +9,5 @@
     <parent link="skiff"/>
     <child link="starboard_rowlock"/>
-    <origin rpy="0.0  0.0 0.0" xyz="0.0 0.8 0.32"/>
+    <origin rpy="0.0  0.0 0.0" xyz="0.0 0.8 0.42"/>
     <axis xyz="0 0 1"/>
     <limit effort="1000.0" lower="-1.4" upper="1.4" velocity="1.0"/>
@@ -16,5 +16,5 @@
     <parent link="skiff"/>
     <child link="port_rowlock"/>
-    <origin rpy="0.0  0.0 0.0" xyz="0.0 -0.8 0.3"/>
+    <origin rpy="0.0  0.0 0.0" xyz="0.0 -0.8 0.4"/>
     <axis xyz="0 0 1"/>
     <limit effort="1000.0" lower="-1.4" upper="1.4" velocity="1.0"/>

Commit message: changes topic names, added force sensors

File: boot1_description/urdf/boot1.xacro (robot description, xacro)
@@ -6,5 +6,5 @@
   <!-- Import Rviz colors -->
   <xacro:include filename="$(find boot1_description)/urdf/materials.xacro" />
-  <joint name="starboard_rowlock_joint" type="revolute">
+  <joint name="starboard_rowlock" type="revolute">
     <parent link="skiff"/>
     <child link="starboard_rowlock"/>
@@ -13,5 +13,5 @@
     <limit effort="1000.0" lower="-1.4" upper="1.4" velocity="1.0"/>
   </joint>
-  <joint name="port_rowlock_joint" type="revolute">
+  <joint name="port_rowlock" type="revolute">
     <parent link="skiff"/>
     <child link="port_rowlock"/>
@@ -20,5 +20,5 @@
     <limit effort="1000.0" lower="-1.4" upper="1.4" velocity="1.0"/>
   </joint>
-  <joint name="starboard_rowlock_oar_joint" type="revolute">
+  <joint name="starboard_oar" type="revolute">
     <parent link="starboard_rowlock"/>
     <child link="starboard_oar"/>
@@ -27,5 +27,5 @@
     <limit effort="1000.0" lower="-0.4" upper="0.0" velocity="1.0"/>
   </joint>
-  <joint name="port_rowlock_oar_joint" type="revolute">
+  <joint name="port_oar" type="revolute">
     <parent link="port_rowlock"/>
     <child link="port_oar"/>
@@ -34,5 +34,5 @@
     <limit effort="1000.0" lower="0.0" upper="0.4" velocity="1.0"/>
   </joint>
-  <joint name="starboard_blade_joint" type="revolute">
+  <joint name="starboard_blade" type="revolute">
     <parent link="starboard_oar"/>
     <child link="starboard_blade"/>
@@ -41,5 +41,5 @@
     <limit effort="1000.0" lower="-0.4" upper="0.4" velocity="1.0"/>
   </joint>
-  <joint name="port_blade_joint" type="revolute">
+  <joint name="port_blade" type="revolute">
     <parent link="port_oar"/>
     <child link="port_blade"/>
@@ -191,5 +191,5 @@
   <transmission name="tran1">
     <type>transmission_interface/SimpleTransmission</type>
-    <joint name="starboard_rowlock_joint">
+    <joint name="starboard_rowlock">
       <hardwareInterface>hardware_interface/EffortJointInterface</hardwareInterface>
     </joint>
@@ -200,5 +200,5 @@
   <transmission name="tran2">
     <type>transmission_interface/SimpleTransmission</type>
-    <joint name="port_rowlock_joint">
+    <joint name="port_rowlock">
       <hardwareInterface>hardware_interface/EffortJointInterface</hardwareInterface>
     </joint>
@@ -209,5 +209,5 @@
   <transmission name="tran3">
     <type>transmission_interface/SimpleTransmission</type>
-    <joint name="starboard_rowlock_oar_joint">
+    <joint name="starboard_oar">
       <hardwareInterface>hardware_interface/EffortJointInterface</hardwareInterface>
     </joint>
@@ -218,5 +218,5 @@
   <transmission name="tran4">
     <type>transmission_interface/SimpleTransmission</type>
-    <joint name="port_rowlock_oar_joint">
+    <joint name="port_oar">
       <hardwareInterface>hardware_interface/EffortJointInterface</hardwareInterface>
     </joint>
@@ -227,5 +227,5 @@
   <transmission name="tran5">
     <type>transmission_interface/SimpleTransmission</type>
-    <joint name="starboard_blade_joint">
+    <joint name="starboard_blade">
       <hardwareInterface>hardware_interface/EffortJointInterface</hardwareInterface>
     </joint>
@@ -236,5 +236,5 @@
   <transmission name="tran6">
     <type>transmission_interface/SimpleTransmission</type>
-    <joint name="port_blade_joint">
+    <joint name="port_blade">
       <hardwareInterface>hardware_interface/EffortJointInterface</hardwareInterface>
     </joint>
