Commit message: put boat on prismatic joint

File: boot1_description/urdf/boot1.urdf (robot description, URDF)
Before this commit: robot myboat, 8 links, 7 joints
Links:
- removed link base_link
- added link l1; visual box size=0.01 0.01 0.20
- added link l2; visual box size=0.01 0.01 0.40
- added link world
- link port_blade: geometry collision box size=0.2 0.1 0.03; visual box size=0.2 0.1 0.03
- link port_oar: geometry collision cylinder length=2.0 radius=0.02; visual cylinder length=2.7 radius=0.02
- link skiff: mass 15 -> 75
- link starboard_blade: geometry collision box size=0.2 0.1 0.03; visual box size=0.2 0.1 0.03
- link starboard_oar: geometry collision cylinder length=2.0 radius=0.02; visual cylinder length=2.7 radius=0.02
Joints:
- removed joint dummy
- removed joint port_blade_joint
- removed joint port_rowlock_joint
- removed joint port_rowlock_oar_joint
- removed joint starboard_blade_joint
- removed joint starboard_rowlock_joint
- removed joint starboard_rowlock_oar_joint
- added joint port_blade: type revolute, parent port_oar, child port_blade, origin xyz=0.0 0.0   1.8 rpy=0.0  0 0.0, axis 0 1 0, limit lower=-0.4 upper=0.4 effort=1000.0 velocity=1.0
- added joint port_oar: type revolute, parent port_rowlock, child port_oar, origin xyz=0.0 0.0   0.02 rpy=0.0  1.57079632679 -1.57079632679, axis 0 1 0, limit lower=0.0 upper=0.4 effort=1000.0 velocity=1.0
- added joint port_rowlock: type revolute, parent skiff, child port_rowlock, origin xyz=-1.5 -0.8 0.4 rpy=0.0  0.0 0.0, axis 0 0 1, limit lower=-1.4 upper=1.4 effort=1000.0 velocity=1.0
- added joint prism: type prismatic, parent world, child l1, origin xyz=0 0 0.25 rpy=0 0 0, axis 1 0 0, limit lower=-1000 upper=1000 effort=1000.0 velocity=0.5
- added joint rev1: type revolute, parent l1, child l2, origin xyz=0.0  0 -0.2 rpy=0 1.57079632679 0, axis 0 1 0, limit lower=-1 upper=1 effort=1000.0 velocity=1.0
- added joint rev2: type revolute, parent l2, child skiff, origin xyz=0.0 0.0 0.4 rpy=3.14159265359 1.57079632679 0, axis 0 1 0, limit lower=-1 upper=1 effort=1000.0 velocity=1.0
- added joint starboard_blade: type revolute, parent starboard_oar, child starboard_blade, origin xyz=0.0 0.0   -1.8 rpy=0 0  0.0, axis 0 1 0, limit lower=-0.4 upper=0.4 effort=1000.0 velocity=1.0
- added joint starboard_oar: type revolute, parent starboard_rowlock, child starboard_oar, origin xyz=0.0 0.0   0.02 rpy=0.0  1.57079632679 -1.57079632679, axis 0 1 0, limit lower=-0.4 upper=0.0 effort=1000.0 velocity=1.0
- added joint starboard_rowlock: type revolute, parent skiff, child starboard_rowlock, origin xyz=-1.5 0.8 0.42 rpy=0.0  0.0 0.0, axis 0 0 1, limit lower=-1.4 upper=1.4 effort=1000.0 velocity=1.0

File: boot1_description/urdf/boot1.xacro (robot description, xacro)
@@ -6,8 +6,29 @@
   <!-- Import Rviz colors -->
   <xacro:include filename="$(find boot1_description)/urdf/materials.xacro" />
+  <joint name="prism" type="prismatic">
+    <parent link="world"/>
+    <child link="l1"/>
+    <origin xyz="0 0 0.25" rpy="0 0 0"/>
+    <axis xyz="1 0 0"/>
+    <limit effort="1000.0" lower="-1000" upper="1000" velocity="0.5"/>
+  </joint>
+  <joint name="rev1" type="revolute">
+    <parent link="l1"/>
+    <child link="l2"/>
+    <origin xyz="0.0 0 -0.2" rpy="0 ${pi/2} 0"/>
+    <axis xyz="0 1 0"/>
+    <limit effort="1000.0" lower="-1" upper="1" velocity="1.0"/>
+  </joint>
+  <joint name="rev2" type="revolute">
+    <parent link="l2"/>
+    <child link="skiff"/>
+    <origin xyz="0.0 0.0 0.4" rpy="${pi} ${pi/2} 0"/>
+    <axis xyz="0 1 0"/>
+    <limit effort="1000.0" lower="-1" upper="1" velocity="1.0"/>
+  </joint>
   <joint name="starboard_rowlock" type="revolute">
     <parent link="skiff"/>
     <child link="starboard_rowlock"/>
-    <origin rpy="0.0  0.0 0.0" xyz="0.0 0.8 0.42"/>
+    <origin rpy="0.0  0.0 0.0" xyz="-3 0.8 0.42"/>
     <axis xyz="0 0 1"/>
     <limit effort="1000.0" lower="-1.4" upper="1.4" velocity="1.0"/>
@@ -16,5 +37,5 @@
     <parent link="skiff"/>
     <child link="port_rowlock"/>
-    <origin rpy="0.0  0.0 0.0" xyz="0.0 -0.8 0.4"/>
+    <origin rpy="0.0  0.0 0.0" xyz="-3 -0.8 0.4"/>
     <axis xyz="0 0 1"/>
     <limit effort="1000.0" lower="-1.4" upper="1.4" velocity="1.0"/>
@@ -48,28 +69,49 @@
     <limit effort="1000.0" lower="-0.4" upper="0.4" velocity="1.0"/>
   </joint>
-  <link name="base_link"/>
-  <!-- Dummy for gazebo   -->
-  <joint name="dummy" type="fixed">
-    <parent link="base_link"/>
-    <child link="skiff"/>
-  </joint>
+  <link name="world"/>
+  <link name="l1">
+    <inertial>
+      <mass value="0.01"/>
+      <origin rpy="0 0 0" xyz="0 0.0 -0.1"/>
+      <inertia ixx="0.006" ixy="0" ixz="0" iyy="0.1" iyz="0" izz="0.1"/>
+    </inertial>
+    <visual>
+      <origin rpy="0 0 0" xyz="0.0 0.0 -0.1"/>
+      <geometry>
+        <box size="0.01 0.01 0.20"/>
+      </geometry>
+    </visual>
+  </link>
+  <link name="l2">
+    <inertial>
+      <mass value="0.01"/>
+      <origin rpy="0 0 0" xyz="0 0.0 0.2"/>
+      <inertia ixx="0.006" ixy="0" ixz="0" iyy="0.1" iyz="0" izz="0.1"/>
+    </inertial>
+    <visual>
+      <origin rpy="0 0 0" xyz="0.0 0.0 0.2"/>
+      <geometry>
+        <box size="0.01 0.01 0.40"/>
+      </geometry>
+    </visual>
+  </link>
   <link name="skiff">
     <inertial>
       <mass value="75"/>   <!-- 15 + 60 voor de roeier -->
-      <origin rpy="0 0 0" xyz="0.0 0.0 0.1"/>
+      <origin rpy="0 0 0" xyz="-3 0.0 0.05"/>
       <inertia ixx="3.2" ixy="0" ixz="0" iyy="54.2" iyz="0" izz="57"/>
 <!--      <inertia ixx="0.6" ixy="0" ixz="0" iyy="11" iyz="0" izz="11.8"/>  -->
     </inertial>
     <collision>
-      <origin rpy="0 0 0" xyz="0.0 0.0   0.1"/>
-      <geometry>
-        <box size="3.0 0.7 0.2"/>
+      <origin rpy="0 0 0" xyz="-3 0.0   0.05"/>
+      <geometry>
+        <box size="6.0 0.7 0.2"/>
       </geometry>
     </collision>
     <visual>
       <!-- should be a nice skull shape including riggers-->
-      <origin rpy="0 0 0" xyz="0.0 0.0   0.1"/>
-      <geometry>
-        <box size="3.0 0.7 0.2"/>
+      <origin rpy="0 0 0" xyz="-3 0.0   0.05"/>
+      <geometry>
+        <box size="6.0 0.7 0.2"/>
       </geometry>
     </visual>

Commit message: make sensors work

File: boot1_description/urdf/boot1.urdf (robot description, URDF)
Before this commit: robot myboat, 10 links, 9 joints
Links:
- removed link port_blade
- removed link port_oar
- removed link port_rowlock
- removed link starboard_blade
- removed link starboard_oar
- removed link starboard_rowlock
- added link port_blade_l, mass 1.0; collision box size=0.2 0.1 0.03; visual box size=0.2 0.1 0.03
- added link port_oar_l, mass 1.0; collision cylinder length=2.0 radius=0.02; visual cylinder length=2.7 radius=0.02
- added link port_rowlock_l, mass 0.1; collision box size=0.02 0.02 0.04; visual box size=0.02 0.02 0.04
- added link starboard_blade_l, mass 1.0; collision box size=0.2 0.1 0.03; visual box size=0.2 0.1 0.03
- added link starboard_oar_l, mass 1.0; collision cylinder length=2.0 radius=0.02; visual cylinder length=2.7 radius=0.02
- added link starboard_rowlock_l, mass 0.1; collision box size=0.02 0.02 0.04; visual box size=0.02 0.02 0.04
- link l1: mass None -> 0.01
- link l2: mass None -> 0.01
- link skiff: geometry collision box size=6.0 0.7 0.2; visual box size=6.0 0.7 0.2
Joints:
- joint port_blade: child port_blade -> port_blade_l; parent port_oar -> port_oar_l
- joint port_oar: child port_oar -> port_oar_l; parent port_rowlock -> port_rowlock_l
- joint port_rowlock: child port_rowlock -> port_rowlock_l; origin xyz=-1.5 -0.8 0.4 rpy=0.0  0.0 0.0 -> xyz=-3 -0.8 0.4 rpy=0.0  0.0 0.0
- joint rev1: origin xyz=0.0  0 -0.2 rpy=0 1.57079632679 0 -> xyz=0.0 0 -0.2 rpy=0 1.57079632679 0
- joint starboard_blade: child starboard_blade -> starboard_blade_l; parent starboard_oar -> starboard_oar_l
- joint starboard_oar: child starboard_oar -> starboard_oar_l; parent starboard_rowlock -> starboard_rowlock_l
- joint starboard_rowlock: child starboard_rowlock -> starboard_rowlock_l; origin xyz=-1.5 0.8 0.42 rpy=0.0  0.0 0.0 -> xyz=-3 0.8 0.42 rpy=0.0  0.0 0.0

File: boot1_description/urdf/boot1.xacro (robot description, xacro)
@@ -29,5 +29,5 @@
   <joint name="starboard_rowlock" type="revolute">
     <parent link="skiff"/>
-    <child link="starboard_rowlock"/>
+    <child link="starboard_rowlock_l"/>
     <origin rpy="0.0  0.0 0.0" xyz="-3 0.8 0.42"/>
     <axis xyz="0 0 1"/>
@@ -36,5 +36,5 @@
   <joint name="port_rowlock" type="revolute">
     <parent link="skiff"/>
-    <child link="port_rowlock"/>
+    <child link="port_rowlock_l"/>
     <origin rpy="0.0  0.0 0.0" xyz="-3 -0.8 0.4"/>
     <axis xyz="0 0 1"/>
@@ -42,6 +42,6 @@
   </joint>
   <joint name="starboard_oar" type="revolute">
-    <parent link="starboard_rowlock"/>
-    <child link="starboard_oar"/>
+    <parent link="starboard_rowlock_l"/>
+    <child link="starboard_oar_l"/>
     <origin rpy="0.0  ${pi/2} -${pi/2}" xyz="0.0 0.0   0.02"/>
     <axis xyz="0 1 0"/>
@@ -49,6 +49,6 @@
   </joint>
   <joint name="port_oar" type="revolute">
-    <parent link="port_rowlock"/>
-    <child link="port_oar"/>
+    <parent link="port_rowlock_l"/>
+    <child link="port_oar_l"/>
     <origin rpy="0.0  ${pi/2} -${pi/2}" xyz="0.0 0.0   0.02"/>
     <axis xyz="0 1 0"/>
@@ -56,6 +56,6 @@
   </joint>
   <joint name="starboard_blade" type="revolute">
-    <parent link="starboard_oar"/>
-    <child link="starboard_blade"/>
+    <parent link="starboard_oar_l"/>
+    <child link="starboard_blade_l"/>
     <origin rpy="0 0  0.0" xyz="0.0 0.0   -1.8"/>
     <axis xyz="0 1 0"/>
@@ -63,6 +63,6 @@
   </joint>
   <joint name="port_blade" type="revolute">
-    <parent link="port_oar"/>
-    <child link="port_blade"/>
+    <parent link="port_oar_l"/>
+    <child link="port_blade_l"/>
     <origin rpy="0.0  0 0.0" xyz="0.0 0.0   1.8"/>
     <axis xyz="0 1 0"/>
@@ -117,5 +117,5 @@
     </visual>
   </link>
-  <link name="starboard_rowlock">
+  <link name="starboard_rowlock_l">
     <inertial>
       <mass value="0.1"/>
@@ -136,5 +136,5 @@
     </visual>
   </link>
-  <link name="port_rowlock">
+  <link name="port_rowlock_l">
     <inertial>
       <mass value="0.1"/>
@@ -155,5 +155,5 @@
     </visual>
   </link>
-  <link name="starboard_oar">
+  <link name="starboard_oar_l">
     <inertial>
       <mass value="1.0"/>
@@ -174,5 +174,5 @@
     </visual>
   </link>
-  <link name="port_oar">
+  <link name="port_oar_l">
     <inertial>
       <mass value="1.0"/>
@@ -193,5 +193,5 @@
     </visual>
   </link>
-  <link name="starboard_blade">
+  <link name="starboard_blade_l">
     <inertial>
       <mass value="1.0"/>
@@ -212,5 +212,5 @@
     </visual>
   </link>
-  <link name="port_blade">
+  <link name="port_blade_l">
     <inertial>
       <mass value="1.0"/>
