Commit message: Add first parameters

File: boot2_description/config/param.xacro (robot description, xacro)
@@ -2,9 +2,16 @@
 <robot 	xmlns:xacro="http://www.ros.org/wiki/xacro">
 <!--
-    Generated from param.yaml and code.
-    Describes parameter of the boot model
-    boat: span
-    oar: inner, outer
-    rower: weight, lengths of links, musle power?
+    Describes parameters of the boot model
+-->
+<!-- boat  -->
+<xacro:property name="span" value="1.6" />
+<!-- oar -->
+<xacro:property name="inner" value="0.87" />
+<xacro:property name="outer" value="2.00" />
+<!--  rower -->
+<xacro:property name="weight" value="70" />
+<xacro:property name="lenght" value="1.80" />
+<!--
+ lengths of links, musle power?
 -->
 </robot>

File: boot2_description/urdf/boot2.urdf (robot description, URDF)
Before this commit: robot myboat, 10 links, 9 joints
Links:
- link port_oar_l: geometry collision cylinder length=2.27 radius=0.02; visual cylinder length=2.87 radius=0.02
- link skiff: mass ${15 + weight} -> 85
- link starboard_oar_l: geometry collision cylinder length=2.27 radius=0.02; visual cylinder length=2.87 radius=0.02
Joints:
- joint port_blade: origin xyz=0.0 0.0   ${outer} rpy=0.0  0 0.0 -> xyz=0.0 0.0   2.0 rpy=0.0  0 0.0
- joint port_oar: origin xyz=0.0 0.0   0.02 rpy=0.0  ${pi/2} -${pi/2} -> xyz=0.0 0.0   0.02 rpy=0.0  1.57079632679 -1.57079632679
- joint port_rowlock: origin xyz=-3 -${span/2} 0.4 rpy=0.0  0.0 0.0 -> xyz=-3 -0.8 0.4 rpy=0.0  0.0 0.0
- joint rev1: origin xyz=0.0 0 -0.2 rpy=0 ${pi/2} 0 -> xyz=0.0 0 -0.2 rpy=0 1.57079632679 0
- joint rev2: origin xyz=0.0 0.0 0.4 rpy=${pi} ${pi/2} 0 -> xyz=0.0 0.0 0.4 rpy=3.14159265359 1.57079632679 0
- joint starboard_blade: origin xyz=0.0 0.0   -${outer} rpy=0 0  0.0 -> xyz=0.0 0.0   -2.0 rpy=0 0  0.0
- joint starboard_oar: origin xyz=0.0 0.0   0.02 rpy=0.0  ${pi/2} -${pi/2} -> xyz=0.0 0.0   0.02 rpy=0.0  1.57079632679 -1.57079632679
- joint starboard_rowlock: origin xyz=-3 ${span/2} 0.42 rpy=0.0  0.0 0.0 -> xyz=-3 0.8 0.42 rpy=0.0  0.0 0.0
