Commit message: updated testing

File: testing/crash_boot.urdf (robot description, URDF)
Before this commit: robot myboat, 9 links, 8 joints
Links:
- link back_low: geometry visual mesh filename=model://myboot/meshes/hokuyo.dae scale=10.0004 10.0004 10.0004

File: testing/crash_boot.xacro (robot description, xacro)
@@ -19,5 +19,6 @@
     <origin rpy="0 0 0" xyz="0.15 0.0   0.0"/>
     <geometry>
-      <box size="0.3 0.1 0.05"/>
+      <mesh filename="model://myboot/meshes/hokuyo.dae" scale="10.0004 10.0004 10.0004"/>
+      <!--      <box size="0.3 0.1 0.05"/> -->
     </geometry>
   </visual>
