Commit message: net ik_1.py version

File: boot3_description/config/param.xacro (robot description, xacro)
@@ -3,4 +3,5 @@
 <!--
     Describes parameters of the boot model
+        template version
 -->
 <!-- boat  -->
@@ -15,3 +16,5 @@
  lengths of links, musle power?
 -->
+<!-- Initial position of links that can change-->
+<xacro:property name="starboard_rowlock" value="-0.57" />
 </robot>

Commit message: Close first kinematic loop

File: boot3_description/config/param.xacro (robot description, xacro)
@@ -1,4 +1,3 @@
-<?xml version="1.0"?>
-<robot 	xmlns:xacro="http://www.ros.org/wiki/xacro">
+<robot xmlns:xacro="http://www.ros.org/wiki/xacro">
 <!--
     Describes parameters of the boot model
@@ -6,38 +5,40 @@
 -->
 <!-- boat  -->
-<xacro:property name="span" value="1.6" />
+<xacro:property name="span" value="1.6"/>
 <!-- oar -->
-<xacro:property name="inner" value="0.87" />
-<xacro:property name="outer" value="2.00" />
+<xacro:property name="inner" value="0.87"/>
+<xacro:property name="outer" value="2.00"/>
 <!--  rower -->
-<xacro:property name="weight" value="70" />
-<xacro:property name="lenght" value="1.80" />
+<xacro:property name="weight" value="70"/>
+<xacro:property name="lenght" value="1.80"/>
 <!--
  lengths of links, musle power?
 -->
 <!-- Initial position of links that might change-->
-<xacro:property name="starboard_rowlock" value="-0.57" />
-<xacro:property name="port_rowlock" value="0.61" />
-<xacro:property name="starboard_oar" value="-0.13" />
-<xacro:property name="port_oar" value="0.13" />
-<xacro:property name="hip2" value="0.329" />
-<xacro:property name="back_lh" value="0.011" />
-<xacro:property name="handle_left_j1" value="0.13" />
-<xacro:property name="handle_left_j2" value="0.0" />
-<xacro:property name="handle_left_j3" value="0.04" />
-<xacro:property name="elbow_left" value="-2.0" />
-<xacro:property name="elbow_theta_l" value="0.0" />
-<xacro:property name="elbow_xx_l" value="1.0" />
-<xacro:property name="shoulder_theta_l" value="0.37" />
-<xacro:property name="shoulder_psi_l" value="0.0" />
-<xacro:property name="shoulder_l" value="0.16" />
-<xacro:property name="handle_right_j1" value="-0.07" />
-<xacro:property name="handle_right_j2" value="-0.08" />
-<xacro:property name="handle_right_j3" value="0.1" />
-<xacro:property name="elbow_right" value="1.8" />
-<xacro:property name="elbow_theta_r" value="-0.02" />
-<xacro:property name="elbow_xx_r" value="0.7" />
-<xacro:property name="shoulder_theta_r" value="-0.62" />
-<xacro:property name="shoulder_psi_r" value="3.42" />
-<xacro:property name="shoulder_r" value="0.0" />
+<xacro:property name="starboard_rowlock" value="-0.4939"/>
+<xacro:property name="port_rowlock" value="0.61"/>
+<xacro:property name="starboard_oar" value="-0.1459"/>
+<xacro:property name="port_oar" value="0.13"/>
+<xacro:property name="hip2" value="0.329"/>
+<xacro:property name="back_lh" value="0.011"/>
+<xacro:property name="handle_left_j1" value="0.1427"/>
+<xacro:property name="handle_left_j2" value="0.0808"/>
+<xacro:property name="handle_left_j3" value="-0.0491"/>
+<xacro:property name="elbow_left" value="-1.9209"/>
+<xacro:property name="elbow_theta_l" value="-0.0007"/>
+<xacro:property name="elbow_xx_l" value="0.9758"/>
+<xacro:property name="shoulder_theta_l" value="0.5443"/>
+<xacro:property name="shoulder_psi_l" value="-0.0209"/>
+<xacro:property name="shoulder_l" value="0.1487"/>
+<xacro:property name="handle_right_j1" value="-0.07"/>
+<xacro:property name="handle_right_j2" value="-0.08"/>
+<xacro:property name="handle_right_j3" value="0.1"/>
+<xacro:property name="elbow_right" value="1.8"/>
+<xacro:property name="elbow_theta_r" value="-0.02"/>
+<xacro:property name="elbow_xx_r" value="0.7"/>
+<xacro:property name="shoulder_theta_r" value="-0.62"/>
+<xacro:property name="shoulder_psi_r" value="3.42"/>
+<xacro:property name="shoulder_r" value="0.0"/>
+<!-- Some joints have to change when creating the kinematic loops -->
+<xacro:property name="sliding_type" value="prismatic"/>
 </robot>

File: boot3_description/urdf/boot.urdf (robot description, URDF)
Before this commit: robot myboat, 41 links, 40 joints
Joints:
- joint back_lh: type fixed -> revolute
- joint elbow_left: origin xyz=-0.4 0.0 0.0 rpy=0 0 -2.0 -> xyz=-0.4 0.0 0.0 rpy=0 0 -1.9209
- joint elbow_right: origin xyz=-0.4 0.0 0.0 rpy=3.14159265359 0 4.94159265359 -> xyz=-0.4 0.0 0.0 rpy=3.14159265359 0 4.74209265359
- joint elbow_theta_l: origin xyz=-0.0 0.0  0.0 rpy=0.0 0.0  0.0 -> xyz=-0.0 0.0  0.0 rpy=0.0 -0.0007  0.0
- joint elbow_theta_r: origin xyz=0.0 0.0  0.0 rpy=0.0 -0.02  0.0 -> xyz=0.0 0.0  0.0 rpy=0.0 0.0259  0.0
- joint elbow_xx_l: axis 1.0 0 0 -> 1 0 0; origin xyz=-0.0 0.0  0.0 rpy=1.0 0.0  0.0 -> xyz=-0.0 0.0  0.0 rpy=0.9758 0.0  0.0
- joint elbow_xx_r: origin xyz=0.0 0.0  0.0 rpy=0.7 0.0  0.0 -> xyz=0.0 0.0  0.0 rpy=0.8072 0.0  0.0
- joint handle_left_j1: origin xyz=0 0.0 0.87 rpy=0.13 0 1.57079632679 -> xyz=0 0.0 0.87 rpy=0.1427 0 1.57079632679
- joint handle_left_j2: axis 0  0 1 -> 0 0 1; origin xyz=0 0.0 0.0 rpy=0 0 0.0 -> xyz=0 0.0 0.0 rpy=0 0 0.0808
- joint handle_left_j3: origin xyz=0 0.0 0.0 rpy=0 0.04 0 -> xyz=0 0.0 0.0 rpy=0 -0.0491 0
- joint handle_right_j1: origin xyz=0 0.0 -0.87 rpy=-0.07 0 1.57079632679 -> xyz=0 0.0 -0.87 rpy=-0.0377 0 1.57079632679
- joint handle_right_j2: axis 0  0 1 -> 0 0 1; origin xyz=0 0.0 0.0 rpy=0 0 -0.08 -> xyz=0 0.0 0.0 rpy=0 0 -0.0843
- joint handle_right_j3: origin xyz=0 0.0 0.0 rpy=3.14159265359 0.1 0 -> xyz=0 0.0 0.0 rpy=3.14159265359 0.231 0
- joint hip2: type fixed -> revolute
- joint port_rowlock: origin xyz=-3 -0.8 0.25 rpy=0.0  0.0 0.61 -> xyz=-3 -0.8 0.25 rpy=0.0  0.0 0.5857
- joint shoulder_l: origin xyz=0.0 0.0   0.0 rpy=0.0 0.0 0.16 -> xyz=0.0 0.0   0.0 rpy=0.0 0.0 0.1487
- joint shoulder_psi_l: origin xyz=0.0 0.0   0.0 rpy=0.0 0.0 0.0 -> xyz=0.0 0.0   0.0 rpy=-0.0209 0.0 0.0
- joint shoulder_psi_r: axis 1 0 0 -> -1 0 0; origin xyz=0.0 0.0   0.0 rpy=3.42 0.0 0.0 -> xyz=0.0 0.0   0.0 rpy=3.3329 0.0 0.0
- joint shoulder_r: axis 0 0 1 -> 0 0 -1; origin xyz=0.0 -0.0   0.0 rpy=0.0 3.14159265359  0.0 -> xyz=0.0 -0.0   0.0 rpy=0.0 3.14159265359  -0.0077
- joint shoulder_theta_l: origin xyz=-0.35 0.0 0.0 rpy=0 0.37 0 -> xyz=-0.35 0.0 0.0 rpy=0 0.5443 0
- joint shoulder_theta_r: axis 0 1 0 -> 0 -1 0; origin xyz=0.35 0.0 0.0 rpy=3.14159265359 -0.62 0 -> xyz=0.35 0.0 0.0 rpy=3.14159265359 -0.8444 0
- joint starboard_oar: origin xyz=0.0 0.0   0.02 rpy=0.0  1.44079632679 -1.57079632679 -> xyz=0.0 0.0   0.02 rpy=0.0  1.42489632679 -1.57079632679
- joint starboard_rowlock: origin xyz=-3 0.8 0.27 rpy=0.0  0.0 -0.57 -> xyz=-3 0.8 0.27 rpy=0.0  0.0 -0.4939

File: boot3_description/urdf/boot.xacro (robot description, xacro)
@@ -8,4 +8,10 @@
   <!-- parameters that can be configured -->
   <xacro:include filename="$(find boot3_description)/config/param.xacro" />
+  <!-- hoe vanuit launch file te kiezen?  -->
+  <xacro:property name="reconnectloops" value='yes'/>
+  <xacro:if value="${reconnectloops == 'yes'}">
+    <!-- Set some joints to fixed when recreating the kinematic loops again -->
+    <xacro:property name="sliding_type" value="fixed" />
+  </xacro:if>
   <joint name="prism" type="prismatic">
     <parent link="world"/>
@@ -88,5 +94,5 @@
     <limit effort="101.0" lower="-0.4" upper="0.4" velocity="1.0"/>
   </joint>
-  <joint name="sliding" type="fixed">  <!-- tijdelijk -->
+  <joint name="sliding" type="${sliding_type}">  <!-- prismatic -->
     <parent link="skiff"/>
     <child link="seat"/>
@@ -120,5 +126,5 @@
     <limit effort="101.0" lower="-1.6" upper="0" velocity="1.0"/>
   </joint>
-  <joint name="hip2" type="fixed">   <!-- tijdelijk -->
+  <joint name="hip2" type="revolute">   <!-- tijdelijk -->
     <parent link="seat"/>
     <child link="back_low"/>
@@ -128,5 +134,5 @@
     <limit effort="1000.0" lower="-1.0" upper="1.0" velocity="1.0"/>
   </joint>
-  <joint name="back_lh" type="fixed">  <!-- tijdelijk -->
+  <joint name="back_lh" type="revolute">  <!-- tijdelijk -->
     <parent link="back_low"/>
     <child link="back_high"/>
@@ -176,5 +182,5 @@
     <origin rpy="0 0 ${handle_left_j2}" xyz="0 0.0 0.0"/>
     <dynamics damping="0.005" />
-    <axis xyz="0  0 1"/>
+    <axis xyz="0 0 1"/>
     <limit effort="101.0" lower="-1" upper="1" velocity="1.0"/>
   </joint>
@@ -246,6 +252,6 @@
     <parent link="left_elbow_theta_link"/>
     <child link="arm_l_upper"/>
-    <origin rpy="1.0 0.0  0.0" xyz="-0.0 0.0  0.0"/>
-    <axis xyz="${elbow_xx_l} 0 0" />
+    <origin rpy="${elbow_xx_l} 0.0  0.0" xyz="-0.0 0.0  0.0"/>
+    <axis xyz="1 0 0" />
     <dynamics damping="0.5" />
     <limit effort="101.0" lower="-0.7" upper="2.0" velocity="1.0"/>
@@ -371,5 +377,5 @@
     <origin rpy="0 0 ${handle_right_j2}" xyz="0 0.0 0.0"/>
     <dynamics damping="0.005" />
-    <axis xyz="0  0 1"/>
+    <axis xyz="0 0 1"/>
     <limit effort="101.0" lower="-1" upper="1" velocity="1.0"/>
   </joint>
@@ -451,5 +457,5 @@
     <child link="right_shoulder_psi_link"/>
     <origin rpy="${pi} ${shoulder_theta_r} 0" xyz="0.35 0.0 0.0"/>
-    <axis xyz="0 1 0" />
+    <axis xyz="0 -1 0" />
     <dynamics damping="0.5" />
     <limit effort="101.0" lower="-1.5" upper="1.0" velocity="1.0"/>
@@ -472,5 +478,5 @@
     <child link="right_shoulder_xx_link" />
     <origin rpy="${shoulder_psi_r} 0.0 0.0" xyz="0.0 0.0   0.0"/>
-    <axis xyz="1 0 0" />
+    <axis xyz="-1 0 0" />
     <dynamics damping="0.005" />
     <limit effort="101.0" lower="-1.5" upper="1.5" velocity="1.0"/>
@@ -493,5 +499,5 @@
     <child link="shoulder_right" />
     <origin rpy="0.0 ${pi}  ${shoulder_r}" xyz="0.0 -0.0   0.0"/>
-    <axis xyz="0 0 1" />
+    <axis xyz="0 0 -1" />
     <dynamics damping="0.005" />
     <limit effort="101.0" lower="-1.0" upper="0.5" velocity="1.0"/>

Commit message: Configuration seems to work!

File: boot3_description/config/param.xacro (robot description, xacro)
@@ -17,28 +17,26 @@
 <!-- Initial position of links that might change-->
 <xacro:property name="starboard_rowlock" value="-0.4939"/>
-<xacro:property name="port_rowlock" value="0.61"/>
-<xacro:property name="starboard_oar" value="-0.1459"/>
-<xacro:property name="port_oar" value="0.13"/>
+<xacro:property name="port_rowlock" value="0.4939"/>
+<xacro:property name="starboard_oar" value="-0.1458"/>
+<xacro:property name="port_oar" value="0.1359"/>
 <xacro:property name="hip2" value="0.329"/>
 <xacro:property name="back_lh" value="0.011"/>
-<xacro:property name="handle_left_j1" value="0.1427"/>
-<xacro:property name="handle_left_j2" value="0.0808"/>
-<xacro:property name="handle_left_j3" value="-0.0491"/>
-<xacro:property name="elbow_left" value="-1.9209"/>
-<xacro:property name="elbow_theta_l" value="-0.0007"/>
-<xacro:property name="elbow_xx_l" value="0.9758"/>
-<xacro:property name="shoulder_theta_l" value="0.5443"/>
-<xacro:property name="shoulder_psi_l" value="-0.0209"/>
-<xacro:property name="shoulder_l" value="0.1487"/>
-<xacro:property name="handle_right_j1" value="-0.07"/>
-<xacro:property name="handle_right_j2" value="-0.08"/>
-<xacro:property name="handle_right_j3" value="0.1"/>
-<xacro:property name="elbow_right" value="1.8"/>
-<xacro:property name="elbow_theta_r" value="-0.02"/>
-<xacro:property name="elbow_xx_r" value="0.7"/>
-<xacro:property name="shoulder_theta_r" value="-0.62"/>
-<xacro:property name="shoulder_psi_r" value="3.42"/>
-<xacro:property name="shoulder_r" value="0.0"/>
-<!-- Some joints have to change when creating the kinematic loops -->
-<xacro:property name="sliding_type" value="prismatic"/>
+<xacro:property name="handle_left_j1" value="0.1425"/>
+<xacro:property name="handle_left_j2" value="0.0807"/>
+<xacro:property name="handle_left_j3" value="-0.0503"/>
+<xacro:property name="elbow_left" value="-1.9207"/>
+<xacro:property name="elbow_theta_l" value="0.0003"/>
+<xacro:property name="elbow_xx_l" value="0.9796"/>
+<xacro:property name="shoulder_theta_l" value="0.5435"/>
+<xacro:property name="shoulder_psi_l" value="-0.0182"/>
+<xacro:property name="shoulder_l" value="0.1516"/>
+<xacro:property name="handle_right_j1" value="0.0496"/>
+<xacro:property name="handle_right_j2" value="0.0074"/>
+<xacro:property name="handle_right_j3" value="0.0084"/>
+<xacro:property name="elbow_right" value="1.2894"/>
+<xacro:property name="elbow_theta_r" value="0.0288"/>
+<xacro:property name="elbow_xx_r" value="-0.2775"/>
+<xacro:property name="shoulder_theta_r" value="-.7384"/>
+<xacro:property name="shoulder_psi_r" value="3.7462"/>
+<xacro:property name="shoulder_r" value="0.5698"/>
 </robot>

File: boot3_description/urdf/boot.urdf (robot description, URDF)
Before this commit: robot myboat, 41 links, 40 joints
Joints:
- joint Rdummy_2: origin xyz=0.0 -0.1 0.0 rpy=3.14159265359 -1.57079632679  0.0 -> xyz=0.0 -0.1 0.0 rpy=3.14159265359 0  0.0
- joint elbow_right: origin xyz=-0.4 0.0 0.0 rpy=3.14159265359 0 4.74209265359 -> xyz=-0.4 0.0 0.0 rpy=0 0 1.8
- joint elbow_theta_r: origin xyz=0.0 0.0  0.0 rpy=0.0 0.0259  0.0 -> xyz=0.0 0.0  0.0 rpy=0.0 -0.02  0.0
- joint elbow_xx_r: axis 1 0 0 -> -1 0 0; origin xyz=0.0 0.0  0.0 rpy=0.8072 0.0  0.0 -> xyz=0.0 0.0  0.0 rpy=0.7 0.0  0.0
- joint handle_right_j1: origin xyz=0 0.0 -0.87 rpy=-0.0377 0 1.57079632679 -> xyz=0 0.0 -0.87 rpy=0.07 0 1.57079632679
- joint handle_right_j2: origin xyz=0 0.0 0.0 rpy=0 0 -0.0843 -> xyz=0 0.0 0.0 rpy=0 0 -0.08
- joint handle_right_j3: axis 0 1 0 -> 0 -1 0; origin xyz=0 0.0 0.0 rpy=3.14159265359 0.231 0 -> xyz=0 0.0 0.0 rpy=0 0.638 0
- joint hip2: type revolute -> fixed
- joint port_oar: limit lower=0.0 upper=0.4 effort=101.0 velocity=1.0 -> lower=-0.1 upper=0.4 effort=101.0 velocity=1.0
- joint port_rowlock: origin xyz=-3 -0.8 0.25 rpy=0.0  0.0 0.5857 -> xyz=-3 -0.8 0.25 rpy=0.0  0.0 0.4939; type revolute -> fixed
- joint shoulder_psi_r: axis -1 0 0 -> 1 0 0; origin xyz=0.0 0.0   0.0 rpy=3.3329 0.0 0.0 -> xyz=0.0 0.0   0.0 rpy=3.42 0.0 0.0
- joint shoulder_r: axis 0 0 -1 -> 0 0 1; origin xyz=0.0 -0.0   0.0 rpy=0.0 3.14159265359  -0.0077 -> xyz=0.0 -0.0   0.0 rpy=0.0 0  0.0
- joint shoulder_theta_r: origin xyz=0.35 0.0 0.0 rpy=3.14159265359 -0.8444 0 -> xyz=0.35 0.0 0.0 rpy=3.14159265359 -0.62 0
- joint starboard_rowlock: type revolute -> fixed

File: boot3_description/urdf/boot.xacro (robot description, xacro)
@@ -1,5 +1,22 @@
 <?xml version="1.0" ?>
 <robot name="myboat"  xmlns:xacro="http://www.ros.org/wiki/xacro">
-  <!-- Constants for robot dimensions -->
+  <!-- Set some joints to fixed when recreating the kinematic loops again -->
+  <xacro:arg name="reconnectloops" default="true" />
+  <xacro:if value="$(arg reconnectloops)">
+    <xacro:property name="sliding_type" value="fixed" />
+    <xacro:property name="hip2_type" value="fixed" />
+    <xacro:property name="starboard_rowlock_type" value="fixed" />
+    <xacro:property name="port_rowlock_type" value="fixed" />
+    <xacro:property name="starboard_oar_type" value="fixed" />
+    <xacro:property name="port_oar_type" value="fixed" />
+  </xacro:if>
+  <xacro:unless value="$(arg reconnectloops)">
+    <xacro:property name="sliding_type" value="prismatic" />
+    <xacro:property name="hip2_type" value="revolute" />
+    <xacro:property name="starboard_rowlock_type" value="revolute" />
+    <xacro:property name="port_rowlock_type" value="revolute" />
+    <xacro:property name="starboard_oar_type" value="revolute" />
+    <xacro:property name="port_oar_type" value="revolute" />
+  </xacro:unless>
   <!-- Import all Gazebo-customization elements, including Gazebo colors -->
   <xacro:include filename="$(find boot3_description)/urdf/boot.gazebo" />
@@ -8,10 +25,4 @@
   <!-- parameters that can be configured -->
   <xacro:include filename="$(find boot3_description)/config/param.xacro" />
-  <!-- hoe vanuit launch file te kiezen?  -->
-  <xacro:property name="reconnectloops" value='yes'/>
-  <xacro:if value="${reconnectloops == 'yes'}">
-    <!-- Set some joints to fixed when recreating the kinematic loops again -->
-    <xacro:property name="sliding_type" value="fixed" />
-  </xacro:if>
   <joint name="prism" type="prismatic">
     <parent link="world"/>
@@ -38,5 +49,5 @@
     <limit effort="101.0" lower="-1" upper="1" velocity="1.0"/>
   </joint>
-  <joint name="starboard_rowlock" type="revolute">
+  <joint name="starboard_rowlock" type="${starboard_rowlock_type}">
     <parent link="skiff"/>
     <child link="starboard_rowlock_l"/>
@@ -46,5 +57,5 @@
     <limit effort="101.0" lower="-0.4" upper="1.4" velocity="1.0"/>
   </joint>
-  <joint name="port_rowlock" type="revolute">
+  <joint name="port_rowlock" type="${port_rowlock_type}">
     <parent link="skiff"/>
     <child link="port_rowlock_l"/>
@@ -54,5 +65,5 @@
     <limit effort="101.0" lower="-1.4" upper="1.4" velocity="1.0"/>
   </joint>
-  <joint name="starboard_oar" type="revolute">
+  <joint name="starboard_oar" type="${starboard_oar_type}">
     <parent link="starboard_rowlock_l"/>
     <child link="starboard_oar_l"/>
@@ -62,5 +73,5 @@
     <limit effort="101.0" lower="-0.4" upper="0.1" velocity="1.0"/>
   </joint>
-  <joint name="port_oar" type="revolute">
+  <joint name="port_oar" type="${port_oar_type}">
     <parent link="port_rowlock_l"/>
     <child link="port_oar_l"/>
@@ -68,5 +79,5 @@
     <dynamics damping="0.005" />
     <axis xyz="0 1 0"/>
-    <limit effort="101.0" lower="0.0" upper="0.4" velocity="1.0"/>
+    <limit effort="101.0" lower="-0.1" upper="0.4" velocity="1.0"/>
   </joint>
   <joint name="starboard_blade" type="revolute">
@@ -126,5 +137,5 @@
     <limit effort="101.0" lower="-1.6" upper="0" velocity="1.0"/>
   </joint>
-  <joint name="hip2" type="revolute">   <!-- tijdelijk -->
+  <joint name="hip2" type="${hip2_type}">
     <parent link="seat"/>
     <child link="back_low"/>
@@ -134,5 +145,5 @@
     <limit effort="1000.0" lower="-1.0" upper="1.0" velocity="1.0"/>
   </joint>
-  <joint name="back_lh" type="revolute">  <!-- tijdelijk -->
+  <joint name="back_lh" type="revolute">
     <parent link="back_low"/>
     <child link="back_high"/>
@@ -354,5 +365,5 @@
     <parent link="port_oar_l"/>
     <child link="handle_right_l1"/>
-    <origin rpy="${handle_right_j1} 0 ${pi/2}" xyz="0 0.0 -${inner}"/>
+    <origin rpy="${-1*handle_right_j1} 0 ${pi/2}" xyz="0 0.0 -${inner}"/>
     <dynamics damping="0.005" />
     <axis xyz="-1 0 0"/>
@@ -396,7 +407,7 @@
     <parent link="handle_right_l2"/>
     <child link="arm_r_lower"/>
-    <origin rpy="${pi} ${handle_right_j3} 0" xyz="0 0.0 0.0"/>
-    <dynamics damping="0.005" />
-    <axis xyz="0 1 0"/>
+    <origin rpy="0 ${-1*handle_right_j3} 0" xyz="0 0.0 0.0"/>
+    <dynamics damping="0.005" />
+    <axis xyz="0 -1 0"/>
     <limit effort="101.0" lower="-1" upper="1" velocity="1.0"/>
   </joint>
@@ -405,5 +416,5 @@
     <parent link="arm_r_lower"/>
     <child link="right_elbow_psi_link"/>
-    <origin rpy="${pi} 0 ${pi+elbow_right}" xyz="-0.4 0.0 0.0"/>
+    <origin rpy="0 0 ${elbow_right}" xyz="-0.4 0.0 0.0"/>
     <dynamics damping="0.5" />
     <axis xyz="0 0 1"/>
@@ -447,6 +458,6 @@
     <parent link="right_elbow_theta_link"/>
     <child link="arm_r_upper"/>
-    <origin rpy="${elbow_xx_r} 0.0  0.0" xyz="0.0 0.0  0.0"/>
-    <axis xyz="1 0 0" />
+    <origin rpy="${-1*elbow_xx_r} 0.0  0.0" xyz="0.0 0.0  0.0"/>
+    <axis xyz="-1 0 0" />
     <dynamics damping="0.5" />
     <limit effort="101.0" lower="-1.0" upper="2.0" velocity="1.0"/>
@@ -456,5 +467,5 @@
     <parent link="arm_r_upper"/>
     <child link="right_shoulder_psi_link"/>
-    <origin rpy="${pi} ${shoulder_theta_r} 0" xyz="0.35 0.0 0.0"/>
+    <origin rpy="${pi} ${-1*shoulder_theta_r} 0" xyz="0.35 0.0 0.0"/>
     <axis xyz="0 -1 0" />
     <dynamics damping="0.5" />
@@ -478,5 +489,5 @@
     <child link="right_shoulder_xx_link" />
     <origin rpy="${shoulder_psi_r} 0.0 0.0" xyz="0.0 0.0   0.0"/>
-    <axis xyz="-1 0 0" />
+    <axis xyz="1 0 0" />
     <dynamics damping="0.005" />
     <limit effort="101.0" lower="-1.5" upper="1.5" velocity="1.0"/>
@@ -498,6 +509,6 @@
     <parent link="right_shoulder_xx_link" />
     <child link="shoulder_right" />
-    <origin rpy="0.0 ${pi}  ${shoulder_r}" xyz="0.0 -0.0   0.0"/>
-    <axis xyz="0 0 -1" />
+    <origin rpy="0.0 0  ${shoulder_r}" xyz="0.0 -0.0   0.0"/>
+    <axis xyz="0 0 1" />
     <dynamics damping="0.005" />
     <limit effort="101.0" lower="-1.0" upper="0.5" velocity="1.0"/>
@@ -506,5 +517,5 @@
     <parent link="shoulder_right"/>
     <child link="Rdummy_link_2"/>
-    <origin rpy="${pi} -${pi/2}  0.0" xyz="0.0 -0.1 0.0"/>
+    <origin rpy="${pi} 0  0.0" xyz="0.0 -0.1 0.0"/>
     <dynamics damping="0.005" />
     <limit effort="101.0" lower="-1.0" upper="1.0" velocity="1.0"/>
