Commit message: Add video of failure

File: boot3_description/urdf/boot.urdf (robot description, URDF)
Before this commit: robot myboat, 31 links, 30 joints
Links:
- link port_oar_l: geometry collision cylinder length=2.27 radius=0.02; visual cylinder length=2.87 radius=0.02
- link skiff: mass ${15 + weight} -> 85
- link starboard_oar_l: geometry collision cylinder length=2.27 radius=0.02; visual cylinder length=2.87 radius=0.02
Joints:
- joint dummy_2: origin xyz=-0.15 0.0 0.0 rpy=${pi/2} ${pi}  0.0 -> xyz=-0.15 0.0 0.0 rpy=1.57079632679 3.14159265359  0.0
- joint fp_ll: limit lower=0.0 upper=${pi/2} effort=1000.0 velocity=1.0 -> lower=0.0 upper=1.57079632679 effort=1000.0 velocity=1.0
- joint handle_left_j1: origin xyz=0 0.0 ${inner} rpy=0.209 0 ${pi/2} -> xyz=0 0.0 0.87 rpy=0.209 0 1.57079632679
- joint hip2: origin xyz=0.0 0.0   0.1 rpy=0  -${pi/2+0.34} 0.0 -> xyz=0.0 0.0   0.1 rpy=0  -1.91079632679 0.0
- joint port_blade: origin xyz=0.0 0.0   ${outer} rpy=0.0  0 0.0 -> xyz=0.0 0.0   2.0 rpy=0.0  0 0.0
- joint port_oar: origin xyz=0.0 0.0   0.02 rpy=0.0  ${pi/2} -${pi/2} -> xyz=0.0 0.0   0.02 rpy=0.0  1.57079632679 -1.57079632679
- joint port_rowlock: origin xyz=-3 -${span/2} 0.4 rpy=0.0  0.0 0.0 -> xyz=-3 -0.8 0.4 rpy=0.0  0.0 0.0
- joint rev1: origin xyz=0.0 0 -0.2 rpy=0 ${pi/2} 0 -> xyz=0.0 0 -0.2 rpy=0 1.57079632679 0
- joint rev2: origin xyz=0.0 0.0 0.4 rpy=${pi} ${pi/2} 0 -> xyz=0.0 0.0 0.4 rpy=3.14159265359 1.57079632679 0
- joint shoulder_r: origin xyz=0.0 -0.2   0.0 rpy=0.0 ${pi}  0.0 -> xyz=0.0 -0.2   0.0 rpy=0.0 3.14159265359  0.0
- joint starboard_blade: origin xyz=0.0 0.0   -${outer} rpy=0 0  0.0 -> xyz=0.0 0.0   -2.0 rpy=0 0  0.0
- joint starboard_oar: origin xyz=0.0 0.0   0.02 rpy=0.0  ${pi/2-0.13} -${pi/2} -> xyz=0.0 0.0   0.02 rpy=0.0  1.44079632679 -1.57079632679
- joint starboard_rowlock: origin xyz=-3 ${span} 0.42 rpy=0.0  0.0 -0.61 -> xyz=-3 1.6 0.42 rpy=0.0  0.0 -0.61

Commit message: removed plugin form sdf-file

File: boot3_description/urdf/boot.urdf (robot description, URDF)
Before this commit: robot myboat, 31 links, 30 joints
Joints:
- joint fp_ll: origin xyz=0.0 0.0   0.0 rpy=0.0  0.0998 0.0 -> xyz=0.0 0.0   0.0 rpy=0.0  0.1001675 0.0
- joint hip1: origin xyz=0.0 0.0   0.1 rpy=0  0.0998 0.0 -> xyz=0.0 0.0   0.1 rpy=0  0.1001675 0.0
- joint port_oar: origin xyz=0.0 0.0   0.02 rpy=0.0  1.57079632679 -1.57079632679 -> xyz=0.0 0.0   0.02 rpy=0.0  1.70079632679 -1.57079632679
- joint port_rowlock: origin xyz=-3 -0.8 0.4 rpy=0.0  0.0 0.0 -> xyz=-3 -0.8 0.4 rpy=0.0  0.0 0.61
- joint shoulder_iets: type revolute -> fixed
- joint sk_fp: type revolute -> fixed
- joint sliding: origin xyz=-3.495 0.0 0.2 rpy=0 0 0 -> xyz=-3.49514 0.0 0.2 rpy=0 0 0

Commit message: Simplified model

File: boot3_description/urdf/boot.urdf (robot description, URDF)
Before this commit: robot myboat, 31 links, 30 joints
Links:
- removed link arm_l_lower_2
- removed link dummy_link_2
- removed link handle_left_l1
- removed link handle_left_l2
- removed link l1
- removed link l2
- removed link port_blade_l
- removed link port_oar_l
- removed link port_rowlock_l
- removed link skiff
- removed link starboard_blade_l
- removed link starboard_oar_l
- removed link starboard_rowlock_l
Joints:
- removed joint dummy_2
- removed joint handle_left_j1
- removed joint handle_left_j2
- removed joint handle_left_j3
- removed joint port_blade
- removed joint port_oar
- removed joint port_rowlock
- removed joint prism
- removed joint rev1
- removed joint rev2
- removed joint starboard_blade
- removed joint starboard_oar
- removed joint starboard_rowlock
- joint sk_fp: parent skiff -> world
- joint sliding: parent skiff -> world

File: boot3_description/urdf/boot.xacro (robot description, xacro)
@@ -8,79 +8,7 @@
   <!-- parameters that can be configured -->
   <xacro:include filename="$(find boot3_description)/config/param.xacro" />
-  <joint name="prism" type="fixed">  <!-- prismatic -->
-    <parent link="world"/>
-    <child link="l1"/>
-    <origin xyz="0 0 0.25" rpy="0 0 0"/>
-    <dynamics damping="0.005" />
-    <axis xyz="1 0 0"/>
-    <limit effort="101.0" lower="0" upper="1000" velocity="0.5"/>
-  </joint>
-  <joint name="rev1" type="fixed">
-    <parent link="l1"/>
-    <child link="l2"/>
-    <origin xyz="0.0 0 -0.2" rpy="0 ${pi/2} 0"/>
-    <dynamics damping="0.005" />
-    <axis xyz="0 1 0"/>
-    <limit effort="101.0" lower="-1" upper="1" velocity="1.0"/>
-  </joint>
-  <joint name="rev2" type="fixed">
-    <parent link="l2"/>
-    <child link="skiff"/>
-    <origin xyz="0.0 0.0 0.4" rpy="${pi} ${pi/2} 0"/>
-    <dynamics damping="0.005" />
-    <axis xyz="0 1 0"/>
-    <limit effort="101.0" lower="-1" upper="1" velocity="1.0"/>
-  </joint>
-  <joint name="starboard_rowlock" type="fixed">
-    <parent link="skiff"/>
-    <child link="starboard_rowlock_l"/>
-    <origin rpy="0.0  0.0 -0.61" xyz="-3 ${span} 0.42"/>   <!-- span/2  -->
-    <dynamics damping="0.005" />
-    <axis xyz="0 0 1"/>
-    <limit effort="101.0" lower="-0.4" upper="1.4" velocity="1.0"/>
-  </joint>
-  <joint name="port_rowlock" type="fixed">
-    <parent link="skiff"/>
-    <child link="port_rowlock_l"/>
-    <origin rpy="0.0  0.0 0.61" xyz="-3 -${span/2} 0.4"/>
-    <dynamics damping="0.005" />
-    <axis xyz="0 0 1"/>
-    <limit effort="101.0" lower="-1.4" upper="1.4" velocity="1.0"/>
-  </joint>
-  <joint name="starboard_oar" type="fixed">
-    <parent link="starboard_rowlock_l"/>
-    <child link="starboard_oar_l"/>
-    <origin rpy="0.0  ${pi/2-0.13} -${pi/2}" xyz="0.0 0.0   0.02"/>
-    <dynamics damping="0.005" />
-    <axis xyz="0 1 0"/>
-    <limit effort="101.0" lower="-0.4" upper="0.1" velocity="1.0"/>
-  </joint>
-  <joint name="port_oar" type="fixed">
-    <parent link="port_rowlock_l"/>
-    <child link="port_oar_l"/>
-    <origin rpy="0.0  ${pi/2+0.13} -${pi/2}" xyz="0.0 0.0   0.02"/>
-    <dynamics damping="0.005" />
-    <axis xyz="0 1 0"/>
-    <limit effort="101.0" lower="0.0" upper="0.4" velocity="1.0"/>
-  </joint>
-  <joint name="starboard_blade" type="fixed">
-    <parent link="starboard_oar_l"/>
-    <child link="starboard_blade_l"/>
-    <origin rpy="0 0  0.0" xyz="0.0 0.0   -${outer}"/>
-    <dynamics damping="0.005" />
-    <axis xyz="0 1 0"/>
-    <limit effort="101.0" lower="-0.4" upper="0.4" velocity="1.0"/>
-  </joint>
-  <joint name="port_blade" type="fixed">
-    <parent link="port_oar_l"/>
-    <child link="port_blade_l"/>
-    <origin rpy="0.0  0 0.0" xyz="0.0 0.0   ${outer}"/>
-    <dynamics damping="0.005" />
-    <axis xyz="0 1 0"/>
-    <limit effort="101.0" lower="-0.4" upper="0.4" velocity="1.0"/>
-  </joint>
   <!-- Rower joints -->
   <joint name="sk_fp" type="fixed">
-    <parent link="skiff"/>
+    <parent link="world"/>
     <child link="footplate"/>
     <origin rpy="0.0  0 0.0" xyz="-2.5 0.0  0.2"/>
@@ -89,5 +17,5 @@
   </joint>
   <joint name="sliding" type="prismatic">
-    <parent link="skiff"/>
+    <parent link="world"/>
     <child link="seat"/>
     <origin rpy="0 0 0" xyz="-3.49514 0.0 0.2"/>
@@ -194,33 +122,4 @@
     <limit effort="100.0" lower="-2.0" upper="1.0" velocity="1.0"/>
   </joint>
-  <!-- 2D joint right shoulder -->
-  <joint name="shoulder_r" type="fixed" >
-    <parent link="shoulder_link" />
-    <child link="right_shoulder_psi_link" />
-    <origin rpy="0.0 ${pi}  0.0" xyz="0.0 -0.2   0.0"/>
-    <axis xyz="0 0 1" />
-    <dynamics damping="0.005" />
-    <limit effort="101.0" lower="-1.0" upper="0.5" velocity="1.0"/>
-  </joint>
-  <link name="right_shoulder_psi_link">
-    <inertial>
-      <mass value="0.01"/>
-      <origin rpy="0 0 0" xyz="0 0.0 0.0"/>
-      <inertia ixx="0.000000167" ixy="0" ixz="0" iyy="0.000000167" iyz="0" izz="0.000000167"/>
-    </inertial>
-    <visual>
-      <origin rpy="0 0 0" xyz="0.0 0.0 0.0"/>
-      <geometry>
-        <box size="0.01 0.01 0.01"/>
-      </geometry>
-    </visual>
-  </link>
-  <joint name="RShoulderTheta" type="fixed" >
-    <parent link="right_shoulder_psi_link"/>
-    <child link="arm_r_upper"/>
-    <axis xyz="0 1 0" />
-    <dynamics damping="0.005" />
-    <limit effort="101.0" lower="-1.5" upper="1.0" velocity="1.0"/>
-  </joint>
   <!-- 2D joint left elbow -->
   <joint name="LElbowTheta" type="fixed" >
@@ -274,243 +173,6 @@
     </visual>
   </link>
-  <joint name="dummy_2" type="fixed">
-    <parent link="arm_l_lower_2"/>
-    <child link="dummy_link_2"/>
-    <origin rpy="${pi/2} ${pi}  0.0" xyz="-0.15 0.0 0.0"/>
-    <dynamics damping="0.005" />
-    <limit effort="101.0" lower="-1.0" upper="1.0" velocity="1.0"/>
-  </joint>
-  <link name="dummy_link_2">
-    <inertial>
-      <mass value="0.01"/>
-      <origin rpy="0 0 0" xyz="0 0.0 0.0"/>
-      <inertia ixx="0.000000167" ixy="0" ixz="0" iyy="0.000000167" iyz="0" izz="0.000000167"/>
-    </inertial>
-    <visual>
-      <origin rpy="0 0 0" xyz="0.0 0.0 0.0"/>
-      <geometry>
-        <box size="0.01 0.01 0.01"/>
-      </geometry>
-    </visual>
-  </link>
-  <!-- 3D handle joint -->
-  <joint name="handle_left_j1" type="fixed">
-    <parent link="starboard_oar_l"/>
-    <child link="handle_left_l1"/>
-    <origin rpy="0.209 0 ${pi/2}" xyz="0 0.0 ${inner}"/>
-    <dynamics damping="0.005" />
-    <axis xyz="1 0 0"/>
-    <limit effort="101.0" lower="-0.2" upper="0.2" velocity="1.0"/>
-  </joint>
-  <link name="handle_left_l1">
-    <inertial>
-      <mass value="0.01"/>
-      <origin rpy="0 0 0" xyz="0 0.0 0.0"/>
-      <inertia ixx="0.000000167" ixy="0" ixz="0" iyy="0.000000167" iyz="0" izz="0.000000167"/>
-    </inertial>
-    <visual>
-      <origin rpy="0 0 0" xyz="0.0 0.0 0.0"/>
-      <geometry>
-        <box size="0.01 0.01 0.01"/>
-      </geometry>
-    </visual>
-  </link>
-  <joint name="handle_left_j2" type="fixed">
-    <parent link="handle_left_l1"/>
-    <child link="handle_left_l2"/>
-    <origin rpy="0 0 0.06" xyz="0 0.0 0.0"/>
-    <dynamics damping="0.005" />
-    <axis xyz="0  0 1"/>
-    <limit effort="101.0" lower="-0.2" upper="0.2" velocity="1.0"/>
-  </joint>
-  <link name="handle_left_l2">
-    <inertial>
-      <mass value="0.01"/>
-      <origin rpy="0 0 0" xyz="0 0.0 0.0"/>
-      <inertia ixx="0.000000167" ixy="0" ixz="0" iyy="0.000000167" iyz="0" izz="0.000000167"/>
-    </inertial>
-    <visual>
-      <origin rpy="0 0 0" xyz="0.0 0.0 0.0"/>
-      <geometry>
-        <box size="0.01 0.01 0.01"/>
-      </geometry>
-    </visual>
-  </link>
-  <joint name="handle_left_j3" type="fixed">
-    <parent link="handle_left_l2"/>
-    <child link="arm_l_lower_2"/>
-    <origin rpy="0 -0.16 0" xyz="0 0.0 0.0"/>
-    <dynamics damping="0.005" />
-    <axis xyz="0 1 0"/>
-    <limit effort="101.0" lower="-0.2" upper="0.2" velocity="1.0"/>
-  </joint>
-  <joint name="head_joint" type="fixed">
-    <parent link="shoulder_link"/>
-    <child link="head"/>
-    <origin rpy="0  0.0 0.0" xyz="0.2 0.0   0.0"/>
-  </joint>
   <!-- Boat links -->
   <link name="world"/>
-  <link name="l1">
-    <inertial>
-      <mass value="0.01"/>
-      <origin rpy="0 0 0" xyz="0 0.0 -0.1"/>
-      <inertia ixx="0.000033" ixy="0" ixz="0" iyy="0.000033" iyz="0" izz="0.000000167"/>
-    </inertial>
-    <visual>
-      <origin rpy="0 0 0" xyz="0.0 0.0 -0.1"/>
-      <geometry>
-        <box size="0.01 0.01 0.20"/>
-      </geometry>
-    </visual>
-  </link>
-  <link name="l2">
-    <inertial>
-      <mass value="0.01"/>
-      <origin rpy="0 0 0" xyz="0 0.0 0.2"/>
-      <inertia ixx="0.000133" ixy="0" ixz="0" iyy="0.000133" iyz="0" izz="0.000000167"/>
-    </inertial>
-    <visual>
-      <origin rpy="0 0 0" xyz="0.0 0.0 0.2"/>
-      <geometry>
-        <box size="0.01 0.01 0.40"/>
-      </geometry>
-    </visual>
-  </link>
-  <link name="skiff">
-    <inertial>
-      <mass value="${15 + weight}"/>   <!-- boat plus roeier -->
-      <origin rpy="0 0 0" xyz="-3 0.0 0.05"/>
-      <inertia ixx="3.2" ixy="0" ixz="0" iyy="225" iyz="0" izz="228"/>   <!-- weight= 60 -->
-    </inertial>
-    <collision>
-      <origin rpy="0 0 0" xyz="-3 0.0   0.05"/>
-      <geometry>
-        <box size="6.0 0.7 0.2"/>
-      </geometry>
-    </collision>
-    <visual>
-      <!-- should be a nice skull shape including riggers-->
-      <origin rpy="0 0 0" xyz="-3 0.0   0.05"/>
-      <geometry>
-        <box size="6.0 0.7 0.2"/>
-      </geometry>
-    </visual>
-  </link>
-  <link name="starboard_rowlock_l">
-    <inertial>
-      <mass value="0.1"/>
-      <origin rpy="0 0 0" xyz="0.0 0.0 0.0"/>
-      <inertia ixx="0.000017" ixy="0" ixz="0" iyy="0.000017" iyz="0" izz="0.000007"/>
-    </inertial>
-    <collision>
-      <origin rpy="0 0 0" xyz="0.0 0.0   0.0"/>
-      <geometry>
-        <box size="0.02 0.02 0.04"/>
-      </geometry>
-    </collision>
-    <visual>
-      <origin rpy="0 0 0" xyz="0.0 0.0   0.0"/>
-      <geometry>
-        <box size="0.02 0.02 0.04"/>
-      </geometry>
-    </visual>
-  </link>
-  <link name="port_rowlock_l">
-    <inertial>
-      <mass value="0.1"/>
-      <origin rpy="0 0 0" xyz="0.0 0.0 0.0"/>
-      <inertia ixx="0.000017" ixy="0" ixz="0" iyy="0.000017" iyz="0" izz="0.000007"/>
-    </inertial>
-    <collision>
-      <origin rpy="0 0 0" xyz="0.0 0.0   0.0"/>
-      <geometry>
-        <box size="0.02 0.02 0.04"/>
-      </geometry>
-    </collision>
-    <visual>
-      <origin rpy="0 0 0" xyz="0.0 0.0   0.0"/>
-      <geometry>
-        <box size="0.02 0.02 0.04"/>
-      </geometry>
-    </visual>
-  </link>
-  <link name="starboard_oar_l">
-    <inertial>
-      <mass value="1.0"/>
-      <origin rpy="0 0 0" xyz="0 0 -${(outer-inner)/2}"/>
-      <inertia ixx="0.6" ixy="0" ixz="0" iyy="0.6" iyz="0" izz="0.001"/>
-    </inertial>
-    <collision>
-      <origin rpy="0 0 0" xyz="0   0   -${(outer-inner)/2}"/>
-      <geometry>
-        <cylinder length="${inner+outer -0.6}" radius="0.02"/>
-      </geometry>
-    </collision>
-    <visual>
-      <origin rpy="0 0 0" xyz="0   0.0   -${(outer-inner)/2}"/>
-      <geometry>
-        <cylinder length="${inner+outer}" radius="0.02"/>
-      </geometry>
-    </visual>
-  </link>
-  <link name="port_oar_l">
-    <inertial>
-      <mass value="1.0"/>
-      <origin rpy="0 0 0" xyz="0 0 ${(outer-inner)/2}"/>
-      <inertia ixx="0.6" ixy="0" ixz="0" iyy="0.6" iyz="0" izz="0.001"/>
-    </inertial>
-    <collision>
-      <origin rpy="0 0 0" xyz="0   0   ${(outer-inner)/2}"/>
-      <geometry>
-        <cylinder length="${inner+outer-0.6}" radius="0.02"/>
-	<!-- -0.6 to prevent collissions  -->
-      </geometry>
-    </collision>
-    <visual>
-      <origin rpy="0 0 0" xyz="0   0   ${(outer-inner)/2}"/>
-      <geometry>
-        <cylinder length="${inner+outer}" radius="0.02"/>
-      </geometry>
-    </visual>
-  </link>
-  <link name="starboard_blade_l">
-    <inertial>
-      <mass value="1.0"/>
-      <origin rpy="0 -1.4 0" xyz="0.02 0 -0.02"/>
-      <inertia ixx="0.0009" ixy="0" ixz="0" iyy="0.0034" iyz="0" izz="0.004"/>
-    </inertial>
-    <collision>
-      <origin rpy="0 -1.4 0" xyz="0.02    0   -0.02"/>
-      <geometry>
-        <box size="0.2 0.1 0.03"/>
-      </geometry>
-    </collision>
-    <visual>
-      <origin rpy="0 -1.4 0" xyz="0.02    0   -0.02"/>
-      <geometry>
-        <box size="0.2 0.1 0.03"/>
-      </geometry>
-    </visual>
-  </link>
-  <link name="port_blade_l">
-    <inertial>
-      <mass value="1.0"/>
-      <origin rpy="0 1.4 0" xyz="0.02 0 -0.02"/>
-      <inertia ixx="0.0009" ixy="0" ixz="0" iyy="0.0034" iyz="0" izz="0.004"/>
-    </inertial>
-    <collision>
-      <origin rpy="0 1.4 0" xyz="0.02    0   -0.02"/>
-      <geometry>
-        <box size="0.2 0.1 0.03"/>
-      </geometry>
-    </collision>
-    <visual>
-      <origin rpy="0 1.4 0" xyz="0.02    0.0  -0.02"/>
-      <geometry>
-        <box size="0.2 0.1 0.03"/>
-      </geometry>
-    </visual>
-  </link>
   <!-- Rower links -->
   <link name="footplate">
@@ -675,23 +337,4 @@
     </visual>
   </link>
-  <link name="arm_r_upper">
-    <inertial>
-      <mass value="1.0"/>
-      <origin rpy="0 0 0" xyz="0.175 0.0 0.0"/>
-      <inertia ixx="0.004" ixy="0" ixz="0" iyy="0.01" iyz="0" izz="0.01"/>
-    </inertial>
-    <collision>
-      <origin rpy="0 0 0" xyz="0.175 0.0   0.0"/>
-      <geometry>
-        <box size="0.35 0.05 0.05"/>
-      </geometry>
-    </collision>
-    <visual>
-      <origin rpy="0 0 0" xyz="0.175 0.0   0.0"/>
-      <geometry>
-        <box size="0.35 0.05 0.05"/>
-      </geometry>
-    </visual>
-  </link>
   <!-- lower arm in two to create a kinematic loop in gazebo -->
   <link name="arm_l_lower_1">
@@ -708,99 +351,5 @@
     </visual>
   </link>
-  <link name="arm_l_lower_2">
-    <inertial>
-      <mass value="1.0"/>
-      <origin rpy="0 0 0" xyz="-0.075 0.0 0.0"/>
-      <inertia ixx="0.004" ixy="0" ixz="0" iyy="0.002" iyz="0" izz="0.002"/>
-    </inertial>
-    <collision>
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
Commit message: Updated boot.sdf

File: boot3_description/urdf/boot.urdf (robot description, URDF)
Before this commit: robot myboat, 18 links, 17 joints
Links:
- removed link arm_r_upper
- removed link head
- removed link right_shoulder_psi_link
Joints:
- removed joint RShoulderTheta
- removed joint head_joint
- removed joint shoulder_r
