Commit message: Link parameters added

File: boot3_description/urdf/boot.urdf (robot description, URDF)
Before this commit: robot myboat, 39 links, 38 joints
Links:
- removed link arm_l_lower_1
- removed link arm_l_lower_2
- removed link arm_r_lower_1
- removed link arm_r_lower_2
- added link arm_l_lower, mass 1.0; collision box size=0.40 0.05 0.05; visual box size=0.40 0.05 0.05
- added link arm_r_lower, mass 1.0; collision box size=0.40 0.05 0.05; visual box size=0.40 0.05 0.05
- added link left_elbow_theta_link, mass 0.01; visual box size=0.01 0.01 0.01
- added link right_elbow_theta_link, mass 0.01; visual box size=0.01 0.01 0.01
- added link shoulder_left, mass 1.0; collision box size=0.05 0.1 0.05; visual box size=0.05 0.1 0.05
- added link shoulder_right, mass 1.0; collision box size=0.05 0.1 0.05; visual box size=0.05 0.1 0.05
- link port_oar_l: geometry collision cylinder length=2.27 radius=0.02; visual cylinder length=2.87 radius=0.02
- link shoulder_link: geometry collision box size=0.05 0.2 0.05; visual box size=0.05 0.2 0.05
- link skiff: mass ${15 + weight} -> 85
- link starboard_oar_l: geometry collision cylinder length=2.27 radius=0.02; visual cylinder length=2.87 radius=0.02
Joints:
- added joint elbow_xx_l: type revolute, parent left_elbow_theta_link, child arm_l_upper, origin xyz=-0.0 0.0  0.0 rpy=1.0 0.0  0.0, axis 1.0 0 0, limit lower=-0.7 upper=2.0 effort=101.0 velocity=1.0
- added joint elbow_xx_r: type revolute, parent right_elbow_theta_link, child arm_r_upper, origin xyz=0.0 0.0  0.0 rpy=0.7 0.0  0.0, axis 1 0 0, limit lower=-1.0 upper=2.0 effort=101.0 velocity=1.0
- joint Ldummy_1: origin xyz=-0.2 0.0 0.0 rpy=0 0 0.0 -> xyz=0.0 0.1 0.0 rpy=0 0 0.0; parent arm_l_lower_1 -> shoulder_link
- joint Ldummy_2: origin xyz=-0.15 0.0 0.0 rpy=${pi/2} ${pi}  0.0 -> xyz=0.0 0.1 0.0 rpy=0 0 3.14159265359 ; parent arm_l_lower_2 -> shoulder_left
- joint Rdummy_1: origin xyz=-0.2 0.0 0.0 rpy=0 0 0.0 -> xyz=0.0 -0.1 0.0 rpy=0 0 0.0; parent arm_r_lower_1 -> shoulder_link
- joint Rdummy_2: origin xyz=-0.15 0.0 0.0 rpy=${pi/2} ${pi}  0.0 -> xyz=0.0 -0.1 0.0 rpy=3.14159265359 -1.57079632679  0.0; parent arm_r_lower_2 -> shoulder_right
- joint elbow_left: child arm_l_lower_1 -> left_elbow_psi_link; origin xyz=0 0.0 0.0 rpy=0 0 -0.127 -> xyz=-0.4 0.0 0.0 rpy=0 0 -2.0; parent left_elbow_psi_link -> arm_l_lower
- joint elbow_right: child arm_r_lower_1 -> right_elbow_psi_link; origin xyz=0 0.0 0.0 rpy=0 0 -0.127 -> xyz=-0.4 0.0 0.0 rpy=3.14159265359 0 4.94159265359; parent right_elbow_psi_link -> arm_r_lower
- joint elbow_theta_l: child left_elbow_psi_link -> left_elbow_theta_link; origin xyz=-0.35 0.0  0.0 rpy=0.0 -1.90  0.0 -> xyz=-0.0 0.0  0.0 rpy=0.0 0.0  0.0; parent arm_l_upper -> left_elbow_psi_link
- joint elbow_theta_r: child right_elbow_psi_link -> right_elbow_theta_link; origin xyz=0.35 0.0  0.0 rpy=0.0 -${pi+1.9 }  0.0 -> xyz=0.0 0.0  0.0 rpy=0.0 -0.02  0.0; parent arm_r_upper -> right_elbow_psi_link
- joint fp_ll: limit lower=0.0 upper=${pi/2} effort=101.0 velocity=1.0 -> lower=0.0 upper=1.57079632679 effort=101.0 velocity=1.0
- joint handle_left_j1: origin xyz=0 0.0 ${inner} rpy=0.209 0 ${pi/2} -> xyz=0 0.0 0.87 rpy=0.13 0 1.57079632679
- joint handle_left_j2: origin xyz=0 0.0 0.0 rpy=0 0 0.06 -> xyz=0 0.0 0.0 rpy=0 0 0.0
- joint handle_left_j3: child arm_l_lower_2 -> arm_l_lower; origin xyz=0 0.0 0.0 rpy=0 -0.16 0 -> xyz=0 0.0 0.0 rpy=0 0.04 0
- joint handle_right_j1: origin xyz=0 0.0 -${inner} rpy=-0.23 0 ${pi/2} -> xyz=0 0.0 -0.87 rpy=-0.07 0 1.57079632679
- joint handle_right_j2: origin xyz=0 0.0 0.0 rpy=0 0 -0.02 -> xyz=0 0.0 0.0 rpy=0 0 -0.08
- joint handle_right_j3: child arm_r_lower_2 -> arm_r_lower; origin xyz=0 0.0 0.0 rpy=${pi} 0.1 0 -> xyz=0 0.0 0.0 rpy=3.14159265359 0.1 0
- joint hip2: origin xyz=0.0 0.0   0.1 rpy=0  -${pi/2+0.329} 0.0 -> xyz=0.0 0.0   0.1 rpy=0  -1.89979632679 0.0
- joint port_blade: origin xyz=0.0 0.0   ${outer} rpy=0.0  0 0.0 -> xyz=0.0 0.0   2.0 rpy=0.0  0 0.0
- joint port_oar: origin xyz=0.0 0.0   0.02 rpy=0.0  ${pi/2+0.13} -${pi/2} -> xyz=0.0 0.0   0.02 rpy=0.0  1.70079632679 -1.57079632679
- joint port_rowlock: origin xyz=-3 -${span/2} 0.25 rpy=0.0  0.0 0.61 -> xyz=-3 -0.8 0.25 rpy=0.0  0.0 0.61
- joint rev1: origin xyz=0.0 0 -0.2 rpy=0 ${pi/2} 0 -> xyz=0.0 0 -0.2 rpy=0 1.57079632679 0
- joint rev2: origin xyz=0.0 0.0 0.4 rpy=${pi} ${pi/2} 0 -> xyz=0.0 0.0 0.4 rpy=3.14159265359 1.57079632679 0
- joint shoulder_l: child left_shoulder_xx_link -> shoulder_left; limit lower=-1.5 upper=0.5 effort=101.0 velocity=1.0 -> lower=-1.5 upper=1.5 effort=101.0 velocity=1.0; origin xyz=0.0 0.2   0.0 rpy=0.0 0.0 0.18 -> xyz=0.0 0.0   0.0 rpy=0.0 0.0 0.16; parent shoulder_link -> left_shoulder_xx_link
- joint shoulder_psi_l: child left_shoulder_psi_link -> left_shoulder_xx_link; origin xyz=0.0 0.0   0.0 rpy=-0.84 0.0 0.0 -> xyz=0.0 0.0   0.0 rpy=0.0 0.0 0.0; parent left_shoulder_xx_link -> left_shoulder_psi_link
- joint shoulder_psi_r: child right_shoulder_psi_link -> right_shoulder_xx_link; origin xyz=0.0 0.0   0.0 rpy=2.47 0.0 0.0 -> xyz=0.0 0.0   0.0 rpy=3.42 0.0 0.0; parent right_shoulder_xx_link -> right_shoulder_psi_link
- joint shoulder_r: child right_shoulder_xx_link -> shoulder_right; origin xyz=0.0 -0.2   0.0 rpy=0.0 ${pi}  -0.0 -> xyz=0.0 -0.0   0.0 rpy=0.0 3.14159265359  0.0; parent shoulder_link -> right_shoulder_xx_link
- joint shoulder_theta_l: child arm_l_upper -> left_shoulder_psi_link; origin xyz=0 0.0 0.0 rpy=0 0.655 0 -> xyz=-0.35 0.0 0.0 rpy=0 0.37 0; parent left_shoulder_psi_link -> arm_l_upper
- joint shoulder_theta_r: child arm_r_upper -> right_shoulder_psi_link; origin xyz=0 0.0 0.0 rpy=${pi} -0.62 0 -> xyz=0.35 0.0 0.0 rpy=3.14159265359 -0.62 0; parent right_shoulder_psi_link -> arm_r_upper
- joint starboard_blade: origin xyz=0.0 0.0   -${outer} rpy=0 0  0.0 -> xyz=0.0 0.0   -2.0 rpy=0 0  0.0
- joint starboard_oar: origin xyz=0.0 0.0   0.02 rpy=0.0  ${pi/2-0.13} -${pi/2} -> xyz=0.0 0.0   0.02 rpy=0.0  1.44079632679 -1.57079632679
- joint starboard_rowlock: origin xyz=-3 ${span/2} 0.27 rpy=0.0  0.0 -0.57 -> xyz=-3 0.8 0.27 rpy=0.0  0.0 -0.57

File: boot3_description/urdf/boot.xacro (robot description, xacro)
@@ -35,5 +35,5 @@
     <parent link="skiff"/>
     <child link="starboard_rowlock_l"/>
-    <origin rpy="0.0  0.0 -0.57" xyz="-3 ${span/2} 0.27"/>
+    <origin rpy="0.0  0.0 ${starboard_rowlock}" xyz="-3 ${span/2} 0.27"/>
     <dynamics damping="0.005" />
     <axis xyz="0 0 1"/>
@@ -43,5 +43,5 @@
     <parent link="skiff"/>
     <child link="port_rowlock_l"/>
-    <origin rpy="0.0  0.0 0.61" xyz="-3 -${span/2} 0.25"/>
+    <origin rpy="0.0  0.0 ${port_rowlock}" xyz="-3 -${span/2} 0.25"/>
     <dynamics damping="0.005" />
     <axis xyz="0 0 1"/>
@@ -51,5 +51,5 @@
     <parent link="starboard_rowlock_l"/>
     <child link="starboard_oar_l"/>
-    <origin rpy="0.0  ${pi/2-0.13} -${pi/2}" xyz="0.0 0.0   0.02"/>
+    <origin rpy="0.0  ${pi/2+starboard_oar} -${pi/2}" xyz="0.0 0.0   0.02"/>
     <dynamics damping="0.005" />
     <axis xyz="0 1 0"/>
@@ -59,5 +59,5 @@
     <parent link="port_rowlock_l"/>
     <child link="port_oar_l"/>
-    <origin rpy="0.0  ${pi/2+0.13} -${pi/2}" xyz="0.0 0.0   0.02"/>
+    <origin rpy="0.0  ${pi/2+port_oar} -${pi/2}" xyz="0.0 0.0   0.02"/>
     <dynamics damping="0.005" />
     <axis xyz="0 1 0"/>
@@ -123,5 +123,5 @@
     <parent link="seat"/>
     <child link="back_low"/>
-    <origin rpy="0  -${pi/2+0.329} 0.0" xyz="0.0 0.0   0.1"/>
+    <origin rpy="0  -${pi/2+hip2} 0.0" xyz="0.0 0.0   0.1"/>
     <dynamics damping="0.005" />
     <axis xyz="0 1 0"/>
@@ -131,5 +131,5 @@
     <parent link="back_low"/>
     <child link="back_high"/>
-    <origin rpy="0  0.011 0.0" xyz="0.25 0.0   0.0"/>
+    <origin rpy="0  ${back_lh} 0.0" xyz="0.25 0.0   0.0"/>
     <dynamics damping="0.5" />
     <axis xyz="0 1 0"/>
@@ -153,5 +153,5 @@
     <parent link="starboard_oar_l"/>
     <child link="handle_left_l1"/>
-    <origin rpy="0.13 0 ${pi/2}" xyz="0 0.0 ${inner}"/>
+    <origin rpy="${handle_left_j1} 0 ${pi/2}" xyz="0 0.0 ${inner}"/>
     <dynamics damping="0.005" />
     <axis xyz="1 0 0"/>
@@ -174,5 +174,5 @@
     <parent link="handle_left_l1"/>
     <child link="handle_left_l2"/>
-    <origin rpy="0 0 0.0" xyz="0 0.0 0.0"/>
+    <origin rpy="0 0 ${handle_left_j2}" xyz="0 0.0 0.0"/>
     <dynamics damping="0.005" />
     <axis xyz="0  0 1"/>
@@ -195,5 +195,5 @@
     <parent link="handle_left_l2"/>
     <child link="arm_l_lower"/>
-    <origin rpy="0 0.04 0" xyz="0 0.0 0.0"/>
+    <origin rpy="0 ${handle_left_j3} 0" xyz="0 0.0 0.0"/>
     <dynamics damping="0.005" />
     <axis xyz="0 1 0"/>
@@ -204,5 +204,5 @@
     <parent link="arm_l_lower"/>
     <child link="left_elbow_psi_link"/>
-    <origin rpy="0 0 -2.0" xyz="-0.4 0.0 0.0"/>
+    <origin rpy="0 0 ${elbow_left}" xyz="-0.4 0.0 0.0"/>
     <dynamics damping="0.5" />
     <axis xyz="0 0 1"/>
@@ -225,5 +225,5 @@
     <parent link="left_elbow_psi_link"/>
     <child link="left_elbow_theta_link"/>
-    <origin rpy="0.0 0.0  0.0" xyz="-0.0 0.0  0.0"/>
+    <origin rpy="0.0 ${elbow_theta_l}  0.0" xyz="-0.0 0.0  0.0"/>
     <axis xyz="0 1 0" />
     <dynamics damping="0.5" />
@@ -247,5 +247,5 @@
     <child link="arm_l_upper"/>
     <origin rpy="1.0 0.0  0.0" xyz="-0.0 0.0  0.0"/>
-    <axis xyz="1 0 0" />
+    <axis xyz="${elbow_xx_l} 0 0" />
     <dynamics damping="0.5" />
     <limit effort="101.0" lower="-0.7" upper="2.0" velocity="1.0"/>
@@ -255,5 +255,5 @@
     <parent link="arm_l_upper"/>
     <child link="left_shoulder_psi_link"/>
-    <origin rpy="0 0.37 0" xyz="-0.35 0.0 0.0"/>
+    <origin rpy="0 ${shoulder_theta_l} 0" xyz="-0.35 0.0 0.0"/>
     <axis xyz="0 1 0" />
     <dynamics damping="0.005" />
@@ -276,5 +276,5 @@
     <parent link="left_shoulder_psi_link" />
     <child link="left_shoulder_xx_link" />
-    <origin rpy="-0.0 0.0 0.0" xyz="0.0 0.0   0.0"/>
+    <origin rpy="${shoulder_psi_l} 0.0 0.0" xyz="0.0 0.0   0.0"/>
     <axis xyz="1 0 0" />
     <dynamics damping="0.005" />
@@ -297,5 +297,5 @@
     <parent link="left_shoulder_xx_link" />
     <child link="shoulder_left" />
-    <origin rpy="0.0 0.0 0.16" xyz="0.0 0.0   0.0"/>
+    <origin rpy="0.0 0.0 ${shoulder_l}" xyz="0.0 0.0   0.0"/>
     <axis xyz="0 0 1" />
     <dynamics damping="0.005" />
@@ -348,5 +348,5 @@
     <parent link="port_oar_l"/>
     <child link="handle_right_l1"/>
-    <origin rpy="-0.07 0 ${pi/2}" xyz="0 0.0 -${inner}"/>
+    <origin rpy="${handle_right_j1} 0 ${pi/2}" xyz="0 0.0 -${inner}"/>
     <dynamics damping="0.005" />
     <axis xyz="-1 0 0"/>
@@ -369,5 +369,5 @@
     <parent link="handle_right_l1"/>
     <child link="handle_right_l2"/>
-    <origin rpy="0 0 -0.08" xyz="0 0.0 0.0"/>
+    <origin rpy="0 0 ${handle_right_j2}" xyz="0 0.0 0.0"/>
     <dynamics damping="0.005" />
     <axis xyz="0  0 1"/>
@@ -390,5 +390,5 @@
     <parent link="handle_right_l2"/>
     <child link="arm_r_lower"/>
-    <origin rpy="${pi} 0.1 0" xyz="0 0.0 0.0"/>
+    <origin rpy="${pi} ${handle_right_j3} 0" xyz="0 0.0 0.0"/>
     <dynamics damping="0.005" />
     <axis xyz="0 1 0"/>
@@ -399,5 +399,5 @@
     <parent link="arm_r_lower"/>
     <child link="right_elbow_psi_link"/>
-    <origin rpy="${pi} 0 ${pi+1.8}" xyz="-0.4 0.0 0.0"/>
+    <origin rpy="${pi} 0 ${pi+elbow_right}" xyz="-0.4 0.0 0.0"/>
     <dynamics damping="0.5" />
     <axis xyz="0 0 1"/>
@@ -420,5 +420,5 @@
     <parent link="right_elbow_psi_link"/>
     <child link="right_elbow_theta_link"/>
-    <origin rpy="0.0 -0.02  0.0" xyz="0.0 0.0  0.0"/>
+    <origin rpy="0.0 ${elbow_theta_r}  0.0" xyz="0.0 0.0  0.0"/>
     <axis xyz="0 1 0" />
     <dynamics damping="0.5" />
@@ -441,5 +441,5 @@
     <parent link="right_elbow_theta_link"/>
     <child link="arm_r_upper"/>
-    <origin rpy="0.7 0.0  0.0" xyz="0.0 0.0  0.0"/>
+    <origin rpy="${elbow_xx_r} 0.0  0.0" xyz="0.0 0.0  0.0"/>
     <axis xyz="1 0 0" />
     <dynamics damping="0.5" />
@@ -450,5 +450,5 @@
     <parent link="arm_r_upper"/>
     <child link="right_shoulder_psi_link"/>
-    <origin rpy="${pi} -0.62 0" xyz="0.35 0.0 0.0"/>
+    <origin rpy="${pi} ${shoulder_theta_r} 0" xyz="0.35 0.0 0.0"/>
     <axis xyz="0 1 0" />
     <dynamics damping="0.5" />
@@ -471,5 +471,5 @@
     <parent link="right_shoulder_psi_link" />
     <child link="right_shoulder_xx_link" />
-    <origin rpy="3.42 0.0 0.0" xyz="0.0 0.0   0.0"/>
+    <origin rpy="${shoulder_psi_r} 0.0 0.0" xyz="0.0 0.0   0.0"/>
     <axis xyz="1 0 0" />
     <dynamics damping="0.005" />
@@ -492,5 +492,5 @@
     <parent link="right_shoulder_xx_link" />
     <child link="shoulder_right" />
-    <origin rpy="0.0 ${pi}  -0.0" xyz="0.0 -0.0   0.0"/>
+    <origin rpy="0.0 ${pi}  ${shoulder_r}" xyz="0.0 -0.0   0.0"/>
     <axis xyz="0 0 1" />
     <dynamics damping="0.005" />
@@ -557,5 +557,5 @@
       <mass value="0.01"/>
       <origin rpy="0 0 0" xyz="0 0.0 0.2"/>
-      <inertia ixx="0.000133" ixy="0" ixz="0" iyy="0.1=000133" iyz="0" izz="0.000000167"/>
+      <inertia ixx="0.000133" ixy="0" ixz="0" iyy="000133" iyz="0" izz="0.000000167"/>
     </inertial>
     <visual>
@@ -768,5 +768,5 @@
     </inertial>
     <collision>
-      <origin rpy="0 0 0" xyz="0.125.  0.0   0.0"/>
+      <origin rpy="0 0 0" xyz="0.125  0.0   0.0"/>
       <geometry>
         <box size="0.25 0.05 0.05"/>
@@ -806,5 +806,5 @@
     </inertial>
     <collision>
-      <origin rpy="0 0 0" xyz="0.125.  0.0   0.0"/>
+      <origin rpy="0 0 0" xyz="0.125  0.0   0.0"/>
       <geometry>
         <box size="0.25 0.1 0.05"/>
@@ -825,5 +825,5 @@
     </inertial>
     <collision>
-      <origin rpy="0 0 0" xyz="0.15.  0.0   0.0"/>
+      <origin rpy="0 0 0" xyz="0.15  0.0   0.0"/>
       <geometry>
         <box size="0.3 0.15 0.05"/>

Commit message: Stillwrong

File: boot3_description/urdf/boot.urdf (robot description, URDF)
Before this commit: robot myboat, 41 links, 40 joints
Joints:
- joint elbow_left: origin xyz=-0.4 0.0 0.0 rpy=0 0 -1.9209 -> xyz=-0.4 0.0 0.0 rpy=0 0 -1.9207
- joint elbow_right: origin xyz=-0.4 0.0 0.0 rpy=0 0 1.8 -> xyz=-0.4 0.0 0.0 rpy=0 0 1.2894
- joint elbow_theta_l: origin xyz=-0.0 0.0  0.0 rpy=0.0 -0.0007  0.0 -> xyz=-0.0 0.0  0.0 rpy=0.0 0.0003  0.0
- joint elbow_theta_r: origin xyz=0.0 0.0  0.0 rpy=0.0 -0.02  0.0 -> xyz=0.0 0.0  0.0 rpy=0.0 0.0288  0.0
- joint elbow_xx_l: origin xyz=-0.0 0.0  0.0 rpy=0.9758 0.0  0.0 -> xyz=-0.0 0.0  0.0 rpy=0.9796 0.0  0.0
- joint elbow_xx_r: origin xyz=0.0 0.0  0.0 rpy=0.7 0.0  0.0 -> xyz=0.0 0.0  0.0 rpy=0.2775 0.0  0.0
- joint handle_left_j1: origin xyz=0 0.0 0.87 rpy=0.1427 0 1.57079632679 -> xyz=0 0.0 0.87 rpy=0.1425 0 1.57079632679
- joint handle_left_j2: origin xyz=0 0.0 0.0 rpy=0 0 0.0808 -> xyz=0 0.0 0.0 rpy=0 0 0.0807
- joint handle_left_j3: origin xyz=0 0.0 0.0 rpy=0 -0.0491 0 -> xyz=0 0.0 0.0 rpy=0 -0.0503 0
- joint handle_right_j1: origin xyz=0 0.0 -0.87 rpy=0.07 0 1.57079632679 -> xyz=0 0.0 -0.87 rpy=-0.0496 0 1.57079632679
- joint handle_right_j2: origin xyz=0 0.0 0.0 rpy=0 0 -0.08 -> xyz=0 0.0 0.0 rpy=0 0 0.0074
- joint handle_right_j3: origin xyz=0 0.0 0.0 rpy=0 0.638 0 -> xyz=0 0.0 0.0 rpy=0 -0.0084 0
- joint hip2: type fixed -> revolute
- joint port_oar: origin xyz=0.0 0.0   0.02 rpy=0.0  1.70079632679 -1.57079632679 -> xyz=0.0 0.0   0.02 rpy=0.0  1.70669632679 -1.57079632679
- joint port_rowlock: type fixed -> revolute
- joint shoulder_l: origin xyz=0.0 0.0   0.0 rpy=0.0 0.0 0.1487 -> xyz=0.0 0.0   0.0 rpy=0.0 0.0 0.1516
- joint shoulder_psi_l: origin xyz=0.0 0.0   0.0 rpy=-0.0209 0.0 0.0 -> xyz=0.0 0.0   0.0 rpy=-0.0182 0.0 0.0
- joint shoulder_psi_r: origin xyz=0.0 0.0   0.0 rpy=3.42 0.0 0.0 -> xyz=0.0 0.0   0.0 rpy=3.7462 0.0 0.0
- joint shoulder_r: origin xyz=0.0 -0.0   0.0 rpy=0.0 0  0.0 -> xyz=0.0 -0.0   0.0 rpy=0.0 0  0.5698
- joint shoulder_theta_l: origin xyz=-0.35 0.0 0.0 rpy=0 0.5443 0 -> xyz=-0.35 0.0 0.0 rpy=0 0.5435 0
- joint shoulder_theta_r: origin xyz=0.35 0.0 0.0 rpy=3.14159265359 -0.62 0 -> xyz=0.35 0.0 0.0 rpy=3.14159265359 0.7384 0
- joint sliding: type fixed -> prismatic
- joint starboard_oar: origin xyz=0.0 0.0   0.02 rpy=0.0  1.42489632679 -1.57079632679 -> xyz=0.0 0.0   0.02 rpy=0.0  1.42499632679 -1.57079632679
- joint starboard_rowlock: type fixed -> revolute

File: boot3_description/urdf/boot.xacro (robot description, xacro)
@@ -2,5 +2,5 @@
 <robot name="myboat"  xmlns:xacro="http://www.ros.org/wiki/xacro">
   <!-- Set some joints to fixed when recreating the kinematic loops again -->
-  <xacro:arg name="reconnectloops" default="true" />
+  <xacro:arg name="reconnectloops" default="false" />
   <xacro:if value="$(arg reconnectloops)">
     <xacro:property name="sliding_type" value="fixed" />

Commit message: Added testboot variant

File: boot3_description/urdf/boot.urdf (robot description, URDF)
Before this commit: robot myboat, 41 links, 40 joints
Joints:
- joint shoulder_l: limit lower=-1.5 upper=1.5 effort=101.0 velocity=1.0 -> lower=-1.0 upper=1.0 effort=101.0 velocity=1.0
- joint shoulder_psi_l: limit lower=-1.5 upper=1.5 effort=101.0 velocity=1.0 -> lower=-1.0 upper=1.0 effort=101.0 velocity=1.0
- joint shoulder_psi_r: limit lower=-1.5 upper=1.5 effort=101.0 velocity=1.0 -> lower=-1.0 upper=1.0 effort=101.0 velocity=1.0
- joint shoulder_r: limit lower=-1.0 upper=0.5 effort=101.0 velocity=1.0 -> lower=-1.0 upper=1.0 effort=101.0 velocity=1.0
- joint shoulder_theta_l: limit lower=-2.0 upper=1.0 effort=101.0 velocity=1.0 -> lower=-1.0 upper=1.0 effort=101.0 velocity=1.0
- joint shoulder_theta_r: limit lower=-1.5 upper=1.0 effort=101.0 velocity=1.0 -> lower=-1.0 upper=1.0 effort=101.0 velocity=1.0

File: boot3_description/urdf/boot.xacro (robot description, xacro)
@@ -646,5 +646,5 @@
       <mass value="1.0"/>
       <origin rpy="0 0 0" xyz="0 0 -${(outer-inner)/2}"/>
-      <inertia ixx="0.6" ixy="0" ixz="0" iyy="0.6" iyz="0" izz="0.001"/>
+      <inertia ixx="0.6" ixy="0" ixz="0" iyy="0.6" iyz="0" izz="0.0002"/>
     </inertial>
     <collision>
@@ -665,5 +665,5 @@
       <mass value="1.0"/>
       <origin rpy="0 0 0" xyz="0 0 ${(outer-inner)/2}"/>
-      <inertia ixx="0.6" ixy="0" ixz="0" iyy="0.6" iyz="0" izz="0.001"/>
+      <inertia ixx="0.6" ixy="0" ixz="0" iyy="0.6" iyz="0" izz="0.0002"/>
     </inertial>
     <collision>
@@ -742,5 +742,5 @@
       <mass value="1.0"/>
       <origin rpy="0 0 0" xyz="-0.25 0.0 0.0"/>
-      <inertia ixx="0.001" ixy="0" ixz="0" iyy="0.0005" iyz="0" izz="0.001"/>
+      <inertia ixx="0.00041" ixy="0" ixz="0" iyy="0.021" iyz="0" izz="0.021"/>
     </inertial>
     <collision>
@@ -763,5 +763,5 @@
       <mass value="1.0"/>
       <origin rpy="0 0 0" xyz="-0.125 0.0 0.0"/>
-      <inertia ixx="0.001" ixy="0" ixz="0" iyy="0.0005" iyz="0" izz="0.001"/>
+      <inertia ixx="0.00041" ixy="0" ixz="0" iyy="0.0054" iyz="0" izz="0.0054"/>
     </inertial>
     <collision>
@@ -782,5 +782,5 @@
       <mass value="1.0"/>
       <origin rpy="0 0 0" xyz="0.125 0.0 0.0"/>
-      <inertia ixx="0.001" ixy="0" ixz="0" iyy="0.0005" iyz="0" izz="0.001"/>
+      <inertia ixx="0.00041" ixy="0" ixz="0" iyy="0.0054" iyz="0" izz="0.0054"/>
     </inertial>
     <collision>
@@ -820,5 +820,5 @@
       <mass value="10.0"/>
       <origin rpy="0 0 0" xyz="0.125 0.0 0.0"/>
-      <inertia ixx="0.01" ixy="0" ixz="0" iyy="0.077" iyz="0" izz="0.083"/>
+      <inertia ixx="0.01" ixy="0" ixz="0" iyy="0.054" iyz="0" izz="0.06"/>
     </inertial>
     <collision>
@@ -878,5 +878,5 @@
       <mass value="1.0"/>
       <origin rpy="0 0 0" xyz="0.0 0.05 0.0"/>
-      <inertia ixx="0.013" ixy="0" ixz="0" iyy="0.0004" iyz="0" izz="0.013"/>
+      <inertia ixx="0.001" ixy="0" ixz="0" iyy="0.0004" iyz="0" izz="0.001"/>
     </inertial>
     <collision>
@@ -897,5 +897,5 @@
       <mass value="1.0"/>
       <origin rpy="0 0 0" xyz="0.0 -0.05 0.0"/>
-      <inertia ixx="0.013" ixy="0" ixz="0" iyy="0.0004" iyz="0" izz="0.013"/>
+      <inertia ixx="0.001" ixy="0" ixz="0" iyy="0.0004" iyz="0" izz="0.001"/>
     </inertial>
     <collision>
@@ -916,5 +916,5 @@
       <mass value="1.0"/>
       <origin rpy="0 0 0" xyz="-0.175 0.0 0.0"/>
-      <inertia ixx="0.004" ixy="0" ixz="0" iyy="0.01" iyz="0" izz="0.01"/>
+      <inertia ixx="0.00041" ixy="0" ixz="0" iyy="0.01" iyz="0" izz="0.01"/>
     </inertial>
     <collision>
@@ -935,5 +935,5 @@
       <mass value="1.0"/>
       <origin rpy="0 0 0" xyz="-0.2 0.0 0.0"/>
-      <inertia ixx="0.0004" ixy="0" ixz="0" iyy="0.0035" iyz="0" izz="0.0035"/>
+      <inertia ixx="0.00041" ixy="0" ixz="0" iyy="0.0135" iyz="0" izz="0.0135"/>
     </inertial>
     <collision>
@@ -954,5 +954,5 @@
       <mass value="1.0"/>
       <origin rpy="0 0 0" xyz="0.175 0.0 0.0"/>
-      <inertia ixx="0.004" ixy="0" ixz="0" iyy="0.01" iyz="0" izz="0.01"/>
+      <inertia ixx="0.0004" ixy="0" ixz="0" iyy="0.01" iyz="0" izz="0.01"/>
     </inertial>
     <collision>
