Commit message: Connect rower to oar

File: boot3_description/urdf/boot.xacro (robot description, xacro)
@@ -13,5 +13,5 @@
     <origin xyz="0 0 0.25" rpy="0 0 0"/>
     <axis xyz="1 0 0"/>
-    <limit effort="1000.0" lower="-1000" upper="1000" velocity="0.5"/>
+    <limit effort="1000.0" lower="0" upper="1000" velocity="0.5"/>
   </joint>
   <joint name="rev1" type="revolute">
@@ -32,7 +32,7 @@
     <parent link="skiff"/>
     <child link="starboard_rowlock_l"/>
-    <origin rpy="0.0  0.0 0.0" xyz="-3 ${span/2} 0.42"/>
+    <origin rpy="0.0  0.0 -0.61" xyz="-3 ${span/2} 0.42"/>
     <axis xyz="0 0 1"/>
-    <limit effort="1000.0" lower="-1.4" upper="1.4" velocity="1.0"/>
+    <limit effort="1000.0" lower="-0.4" upper="1.4" velocity="1.0"/>
   </joint>
   <joint name="port_rowlock" type="revolute">
@@ -46,7 +46,7 @@
     <parent link="starboard_rowlock_l"/>
     <child link="starboard_oar_l"/>
-    <origin rpy="0.0  ${pi/2} -${pi/2}" xyz="0.0 0.0   0.02"/>
-    <axis xyz="0 1 0"/>
-    <limit effort="1000.0" lower="-0.4" upper="0.0" velocity="1.0"/>
+    <origin rpy="0.0  ${pi/2-0.13} -${pi/2}" xyz="0.0 0.0   0.02"/>
+    <axis xyz="0 1 0"/>
+    <limit effort="1000.0" lower="-0.4" upper="0.1" velocity="1.0"/>
   </joint>
   <joint name="port_oar" type="revolute">
@@ -71,4 +71,216 @@
     <limit effort="1000.0" lower="-0.4" upper="0.4" velocity="1.0"/>
   </joint>
+  <!-- Rower joints -->
+  <joint name="sk_fp" type="fixed">
+    <parent link="skiff"/>
+    <child link="footplate"/>
+    <origin rpy="0.0  0 0.0" xyz="-2.5 0.0  0.2"/>
+    <limit effort="1000.0" lower="-0.4" upper="0.4" velocity="1.0"/>
+  </joint>
+  <joint name="sliding" type="fixed">
+    <parent link="skiff"/>
+    <child link="seat"/>
+    <origin rpy="0 0 0" xyz="-3.495 0.0 0.2"/>
+    <axis xyz="1 0 0"/>
+    <limit effort="1000.0" lower="-0.1" upper="0.8" velocity="0.5"/>
+  </joint>
+  <joint name="fp_ll" type="revolute">
+    <parent link="footplate"/>
+    <child link="lowerleg"/>
+    <origin rpy="0.0  0.0998 0.0" xyz="0.0 0.0   0.0"/>
+    <axis xyz="0 1 0"/>
+    <limit effort="1000.0" lower="0.0" upper="${pi/2}" velocity="1.0"/>
+  </joint>
+  <joint name="knee" type="revolute">
+    <parent link="lowerleg"/>
+    <child link="upperleg_1"/>
+    <origin rpy="0.0  0 0.0" xyz="-0.5 0.0   0.0"/>
+    <axis xyz="0 1 0"/>
+    <limit effort="1000.0" lower="-2.5" upper="0" velocity="1.0"/>
+  </joint>
+  <joint name="hip1" type="revolute">
+    <parent link="seat"/>
+    <child link="upperleg_2"/>
+    <origin rpy="0  0.0998 0.0" xyz="0.0 0.0   0.1"/>
+    <axis xyz="0 1 0"/>
+    <limit effort="1000.0" lower="-2.5" upper="0" velocity="1.0"/>
+  </joint>
+  <joint name="hip2" type="revolute">
+    <parent link="seat"/>
+    <child link="back_low"/>
+    <origin rpy="0  -${pi/2+0.34} 0.0" xyz="0.0 0.0   0.1"/>
+    <axis xyz="0 1 0"/>
+    <limit effort="1000.0" lower="-1.0" upper="1.0" velocity="1.0"/>
+  </joint>
+  <joint name="back_lh" type="revolute">
+    <parent link="back_low"/>
+    <child link="back_high"/>
+    <origin rpy="0  0.0 0.0" xyz="0.3 0.0   0.0"/>
+    <axis xyz="0 1 0"/>
+    <limit effort="1000.0" lower="0.0" upper="0.5" velocity="1.0"/>
+  </joint>
+  <joint name="shoulder" type="fixed">
+    <parent link="back_high"/>
+    <child link="shoulder_link"/>
+    <origin rpy="0  0.0 0.0" xyz="0.3 0.0   0.0"/>
+    <limit effort="1000.0" lower="0.0" upper="0.5" velocity="1.0"/>
+  </joint>
+  <!-- 3D joint left shoulder -->
+  <joint name="shoulder_l" type="revolute" >
+    <parent link="shoulder_link" />
+    <child link="left_shoulder_xx_link" />
+    <origin rpy="0.0 0.0 0.13" xyz="0.0 0.2   0.0"/>
+    <axis xyz="0 0 1" />
+    <dynamics damping="0.005" />
+    <!--    <limit effort="1000.0" lower="-1.5" upper="0.5" velocity="1.0"/> -->
+    <limit effort="1000.0" lower="-0.1" upper="0.1" velocity="1.0"/>
+  </joint>
+  <link name="left_shoulder_xx_link">
+    <inertial>
+      <mass value="0.01"/>
+      <origin rpy="0 0 0" xyz="0 0.0 0.2"/>
+      <inertia ixx="0.006" ixy="0" ixz="0" iyy="0.1" iyz="0" izz="0.1"/>
+    </inertial>
+  </link>
+  <joint name="shoulder_iets" type="revolute" >
+    <parent link="left_shoulder_xx_link" />
+    <child link="left_shoulder_psi_link" />
+    <origin rpy="-0.803 0.0 0.0" xyz="0.0 0.0   0.0"/>
+    <axis xyz="1 0 0" />
+    <dynamics damping="0.005" />
+<!--    <limit effort="1000.0" lower="-1.5" upper="1.5" velocity="1.0"/> -->
+    <limit effort="1000.0" lower="-0.2" upper="0.2" velocity="1.0"/>
+  </joint>
+  <link name="left_shoulder_psi_link">
+    <inertial>
+      <mass value="0.01"/>
+      <origin rpy="0 0 0" xyz="0 0.0 0.2"/>
+      <inertia ixx="0.006" ixy="0" ixz="0" iyy="0.1" iyz="0" izz="0.1"/>
+    </inertial>
+  </link>
+  <joint name="LShoulderTheta" type="revolute" >
+    <parent link="left_shoulder_psi_link"/>
+    <child link="arm_l_upper"/>
+      <origin rpy="0 0.68 0" xyz="0 0.0 0.0"/>
+    <axis xyz="0 1 0" />
+    <dynamics damping="0.005" />
+<!--    <limit effort="1000.0" lower="-2.0" upper="1.0" velocity="1.0"/> -->
+    <limit effort="1000.0" lower="-0.2" upper="0.2" velocity="1.0"/>
+  </joint>
+  <!-- 2D joint right shoulder -->
+  <joint name="shoulder_r" type="revolute" >
+    <parent link="shoulder_link" />
+    <child link="right_shoulder_psi_link" />
+    <origin rpy="0.0 ${pi}  0.0" xyz="0.0 -0.2   0.0"/>
+    <axis xyz="0 0 1" />
+    <dynamics damping="0.005" />
+    <limit effort="1000.0" lower="-1.0" upper="0.5" velocity="1.0"/>
+  </joint>
+  <link name="right_shoulder_psi_link">
+    <inertial>
+      <mass value="0.01"/>
+      <origin rpy="0 0 0" xyz="0 0.0 0.2"/>
+      <inertia ixx="0.006" ixy="0" ixz="0" iyy="0.1" iyz="0" izz="0.1"/>
+    </inertial>
+  </link>
+  <joint name="RShoulderTheta" type="revolute" >
+    <parent link="right_shoulder_psi_link"/>
+    <child link="arm_r_upper"/>
+    <axis xyz="0 1 0" />
+    <dynamics damping="0.005" />
+    <limit effort="1000.0" lower="-1.5" upper="1.0" velocity="1.0"/>
+  </joint>
+  <!-- 2D joint left elbow -->
+  <joint name="LElbowTheta" type="revolute" >
+    <parent link="arm_l_upper"/>
+    <child link="left_elbow_psi_link"/>
+    <origin rpy="0.0 -1.94  0.0" xyz="-0.35 0.0  0.0"/>
+    <axis xyz="0 1 0" />
+    <dynamics damping="0.005" />
+    <limit effort="1000.0" lower="-0.7" upper="2.0" velocity="1.0"/>
+  </joint>
+  <link name="left_elbow_psi_link">
+    <inertial>
+      <mass value="0.01"/>
+      <origin rpy="0 0 0" xyz="0 0.0 0.0"/>
+      <inertia ixx="0.006" ixy="0" ixz="0" iyy="0.1" iyz="0" izz="0.1"/>
+    </inertial>
+  </link>
+  <joint name="elbow_left" type="revolute">
+    <parent link="left_elbow_psi_link"/>
+    <child link="arm_l_lower_1"/>
+    <origin rpy="0 0 -0.09" xyz="0 0.0 0.0"/>
+    <axis xyz="0 0 1"/>
+    <limit effort="1000.0" lower="-1.0" upper="1.0" velocity="1.0"/>
+  </joint>
+  <!-- hoe kom ik aan de andere kant van arm_lower_1 en 2 ?  -->
+  <joint name="dummy_1" type="fixed">
+    <parent link="arm_l_lower_1"/>
+    <child link="dummy_link_1"/>
+    <origin rpy="0 0 0.0" xyz="-0.2 0.0 0.0"/>
+    <limit effort="1000.0" lower="-1.0" upper="1.0" velocity="1.0"/>
+  </joint>
+  <link name="dummy_link_1">
+    <inertial>
+      <mass value="0.01"/>
+      <origin rpy="0 0 0" xyz="0.0 0.0 0.0"/>
+      <inertia ixx="0.006" ixy="0" ixz="0" iyy="0.1" iyz="0" izz="0.1"/>
+    </inertial>
+  </link>
+  <joint name="dummy_2" type="fixed">
+    <parent link="arm_l_lower_2"/>
+    <child link="dummy_link_2"/>
+    <origin rpy="${pi/2} ${pi}  0.0" xyz="-0.15 0.0 0.0"/>
+    <limit effort="1000.0" lower="-1.0" upper="1.0" velocity="1.0"/>
+  </joint>
+  <link name="dummy_link_2">
+    <inertial>
+      <mass value="0.01"/>
+      <origin rpy="0 0 0" xyz="0.0 0.0 0.0"/>
+      <inertia ixx="0.006" ixy="0" ixz="0" iyy="0.1" iyz="0" izz="0.1"/>
+    </inertial>
+  </link>
+  <!-- 3D handle joint -->
+  <joint name="handle_left_j1" type="revolute">
+    <parent link="starboard_oar_l"/>
+    <child link="handle_left_l1"/>
+    <origin rpy="0.209 0 ${pi/2}" xyz="0 0.0 ${inner}"/>
+    <axis xyz="1 0 0"/>
+    <limit effort="1000.0" lower="-0.2" upper="0.2" velocity="1.0"/>
+  </joint>
+  <link name="handle_left_l1">
+    <inertial>
+      <mass value="0.01"/>
+      <origin rpy="0 0 0" xyz="0 0.0 0.0"/>
+      <inertia ixx="0.006" ixy="0" ixz="0" iyy="0.1" iyz="0" izz="0.1"/>
+    </inertial>
+  </link>
+  <joint name="handle_left_j2" type="revolute">
+    <parent link="handle_left_l1"/>
+    <child link="handle_left_l2"/>
+    <origin rpy="0 0 0.06" xyz="0 0.0 0.0"/>
+    <axis xyz="0  0 1"/>
+    <limit effort="1000.0" lower="-0.2" upper="0.2" velocity="1.0"/>
+  </joint>
+  <link name="handle_left_l2">
+    <inertial>
+      <mass value="0.01"/>
+      <origin rpy="0 0 0" xyz="0 0.0 0.0"/>
+      <inertia ixx="0.006" ixy="0" ixz="0" iyy="0.1" iyz="0" izz="0.1"/>
+    </inertial>
+  </link>
+  <joint name="handle_left_j3" type="revolute">
+    <parent link="handle_left_l2"/>
+    <child link="arm_l_lower_2"/>
+    <origin rpy="0 -0.16 0" xyz="0 0.0 0.0"/>
+    <axis xyz="0 1 0"/>
+    <limit effort="1000.0" lower="-0.2" upper="0.2" velocity="1.0"/>
+  </joint>
+  <joint name="head_joint" type="fixed">
+    <parent link="shoulder_link"/>
+    <child link="head"/>
+    <origin rpy="0  0.0 0.0" xyz="0.2 0.0   0.0"/>
+  </joint>
+  <!-- Boat links -->
   <link name="world"/>
   <link name="l1">
@@ -233,4 +445,257 @@
     </visual>
   </link>
+  <!-- Rower links -->
+  <link name="footplate">
+    <inertial>
+      <mass value="0.1"/>
+      <origin rpy="0 0 0" xyz="0 0.0 0.0"/>
+      <inertia ixx="0.001" ixy="0" ixz="0" iyy="0.0005" iyz="0" izz="0.001"/>
+    </inertial>
+    <collision>
+      <origin rpy="0 0 0" xyz="0 0.0   0.0"/>
+      <geometry>
+        <box size="0.1 0.3 0.1"/>
+      </geometry>
+    </collision>
+    <visual>
+      <origin rpy="0 0 0" xyz="0  0.0   0.0"/>
+      <geometry>
+        <box size="0.1 0.3 0.1"/>
+      </geometry>
+    </visual>
+  </link>
+  <link name="lowerleg">
+    <inertial>
+      <mass value="1.0"/>
+      <origin rpy="0 0 0" xyz="-0.25 0.0 0.0"/>
+      <inertia ixx="0.001" ixy="0" ixz="0" iyy="0.0005" iyz="0" izz="0.001"/>
+    </inertial>
+    <collision>
+      <origin rpy="0 0 0" xyz="-0.25 0.0   0.0"/>
+      <geometry>
+        <box size="0.5 0.05 0.05"/>
+      </geometry>
+    </collision>
+    <visual>
+      <origin rpy="0 0 0" xyz="-0.25 0.0   0.0"/>
+      <geometry>
+        <box size="0.5 0.05 0.05"/>
+      </geometry>
+    </visual>
+  </link>
+  <!-- upperleg split into two parts to avoid a kinematic loop in the urdf
+       the loop will be close in gazebo -->
+  <link name="upperleg_1">
+    <inertial>
+      <mass value="1.0"/>
+      <origin rpy="0 0 0" xyz="-0.125 0.0 0.0"/>
+      <inertia ixx="0.001" ixy="0" ixz="0" iyy="0.0005" iyz="0" izz="0.001"/>
+    </inertial>
+    <collision>
+      <origin rpy="0 0 0" xyz="-0.125  0.0   0.0"/>
+      <geometry>
+        <box size="0.25 0.05 0.05"/>
+      </geometry>
+    </collision>
+    <visual>
+      <origin rpy="0 0 0" xyz="-0.125   0.0   0.0"/>
+      <geometry>
+        <box size="0.25 0.05 0.05"/>
+      </geometry>
+    </visual>
+  </link>
+  <link name="upperleg_2">
+    <inertial>
+      <mass value="1.0"/>
+      <origin rpy="0 0 0" xyz="0.125 0.0 0.0"/>
+      <inertia ixx="0.001" ixy="0" ixz="0" iyy="0.0005" iyz="0" izz="0.001"/>
+    </inertial>
+    <collision>
+      <origin rpy="0 0 0" xyz="0.125.  0.0   0.0"/>
+      <geometry>
+        <box size="0.25 0.05 0.05"/>
+      </geometry>
+    </collision>
+    <visual>
+      <origin rpy="0 0 0" xyz="0.125 0.0   0.0"/>
+      <geometry>
+        <box size="0.25 0.05 0.05"/>
+      </geometry>
+    </visual>
+  </link>
+  <link name="seat">
+    <inertial>
+      <mass value="0.1"/>
+      <origin rpy="0 0 0" xyz="0.0 0.0 0.0"/>
+      <inertia ixx="0.001" ixy="0" ixz="0" iyy="0.0005" iyz="0" izz="0.001"/>
+    </inertial>
+    <collision>
+      <origin rpy="0 0 0" xyz="0.0 0.0   0.0"/>
+      <geometry>
+        <box size="0.1 0.3 0.1"/>
+      </geometry>
+    </collision>
+    <visual>
+      <origin rpy="0 0 0" xyz="0.0 0.0   0.0"/>
+      <geometry>
+        <box size="0.1 0.3 0.1"/>
+      </geometry>
+    </visual>
+  </link>
+  <link name="back_low">
+    <inertial>
+      <mass value="10.0"/>
+      <origin rpy="0 0 0" xyz="0.15 0.0 0.0"/>
+      <inertia ixx="0.001" ixy="0" ixz="0" iyy="0.0005" iyz="0" izz="0.001"/>
+    </inertial>
+    <collision>
+      <origin rpy="0 0 0" xyz="0.15.  0.0   0.0"/>
+      <geometry>
+        <box size="0.3 0.1 0.05"/>
+      </geometry>
+    </collision>
+    <visual>
+      <origin rpy="0 0 0" xyz="0.15 0.0   0.0"/>
+      <geometry>
+        <box size="0.3 0.1 0.05"/>
+      </geometry>
+    </visual>
+  </link>
+  <link name="back_high">
+    <inertial>
+      <mass value="10.0"/>
+      <origin rpy="0 0 0" xyz="0.15 0.0 0.0"/>
+      <inertia ixx="0.001" ixy="0" ixz="0" iyy="0.0005" iyz="0" izz="0.001"/>
+    </inertial>
+    <collision>
+      <origin rpy="0 0 0" xyz="0.15.  0.0   0.0"/>
+      <geometry>
+        <box size="0.3 0.15 0.05"/>
+      </geometry>
+    </collision>
+    <visual>
+      <origin rpy="0 0 0" xyz="0.15 0.0   0.0"/>
+      <geometry>
+        <box size="0.3 0.15 0.05"/>
+      </geometry>
+    </visual>
+  </link>
+  <link name="shoulder_link">
+    <inertial>
+      <mass value="1.0"/>
+      <origin rpy="0 0 0" xyz="0.0 0.0 0.0"/>
+      <inertia ixx="0.001" ixy="0" ixz="0" iyy="0.0005" iyz="0" izz="0.001"/>
+    </inertial>
+    <collision>
+      <origin rpy="0 0 0" xyz="0.0  0.0   0.0"/>
+      <geometry>
+        <box size="0.05 0.4 0.05"/>
+      </geometry>
+    </collision>
+    <visual>
+      <origin rpy="0 0 0" xyz="0.0 0.0   0.0"/>
+      <geometry>
+        <box size="0.05 0.4 0.05"/>
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
Commit message: some tuning

File: boot3_description/urdf/boot.xacro (robot description, xacro)
@@ -78,5 +78,5 @@
     <limit effort="1000.0" lower="-0.4" upper="0.4" velocity="1.0"/>
   </joint>
-  <joint name="sliding" type="fixed">
+  <joint name="sliding" type="prismatic">
     <parent link="skiff"/>
     <child link="seat"/>
@@ -762,3 +762,57 @@
     </actuator>
   </transmission>
+  <transmission name="tran8">
+    <type>transmission_interface/SimpleTransmission</type>
+    <joint name="hip1">
+      <hardwareInterface>hardware_interface/EffortJointInterface</hardwareInterface>
+    </joint>
+    <actuator name="motor8">
+      <mechanicalReduction>1</mechanicalReduction>
+    </actuator>
+  </transmission>
+  <transmission name="tran9">
+    <type>transmission_interface/SimpleTransmission</type>
+    <joint name="hip2">
+      <hardwareInterface>hardware_interface/EffortJointInterface</hardwareInterface>
+    </joint>
+    <actuator name="motor9">
+      <mechanicalReduction>1</mechanicalReduction>
+    </actuator>
+  </transmission>
+  <transmission name="tran10">
+    <type>transmission_interface/SimpleTransmission</type>
+    <joint name="back_lh">
+      <hardwareInterface>hardware_interface/EffortJointInterface</hardwareInterface>
+    </joint>
+    <actuator name="motor10">
+      <mechanicalReduction>1</mechanicalReduction>
+    </actuator>
+  </transmission>
+  <transmission name="tran11">
+    <type>transmission_interface/SimpleTransmission</type>
+    <joint name="shoulder_l">
+      <hardwareInterface>hardware_interface/EffortJointInterface</hardwareInterface>
+    </joint>
+    <actuator name="motor11">
+      <mechanicalReduction>1</mechanicalReduction>
+    </actuator>
+  </transmission>
+  <transmission name="tran12">
+    <type>transmission_interface/SimpleTransmission</type>
+    <joint name="shoulder_iets">
+      <hardwareInterface>hardware_interface/EffortJointInterface</hardwareInterface>
+    </joint>
+    <actuator name="motor12">
+      <mechanicalReduction>1</mechanicalReduction>
+    </actuator>
+  </transmission>
+  <transmission name="tran13">
+    <type>transmission_interface/SimpleTransmission</type>
+    <joint name="LShoulderTheta">
+      <hardwareInterface>hardware_interface/EffortJointInterface</hardwareInterface>
+    </joint>
+    <actuator name="motor13">
+      <mechanicalReduction>1</mechanicalReduction>
+    </actuator>
+  </transmission>
 </robot>

Commit message: disconnect arm

File: boot3_description/urdf/boot.xacro (robot description, xacro)
@@ -8,5 +8,5 @@
   <!-- parameters that can be configured -->
   <xacro:include filename="$(find boot3_description)/config/param.xacro" />
-  <joint name="prism" type="prismatic">
+  <joint name="prism" type="fixed">  <!-- prismatic -->
     <parent link="world"/>
     <child link="l1"/>
@@ -97,5 +97,5 @@
     <origin rpy="0.0  0 0.0" xyz="-0.5 0.0   0.0"/>
     <axis xyz="0 1 0"/>
-    <limit effort="1000.0" lower="-2.5" upper="0" velocity="1.0"/>
+    <limit effort="10000.0" lower="-3.1" upper="0" velocity="1.0"/>
   </joint>
   <joint name="hip1" type="revolute">
@@ -104,5 +104,5 @@
     <origin rpy="0  0.0998 0.0" xyz="0.0 0.0   0.1"/>
     <axis xyz="0 1 0"/>
-    <limit effort="1000.0" lower="-2.5" upper="0" velocity="1.0"/>
+    <limit effort="1000.0" lower="-1.6" upper="0" velocity="1.0"/>
   </joint>
   <joint name="hip2" type="revolute">
@@ -111,5 +111,5 @@
     <origin rpy="0  -${pi/2+0.34} 0.0" xyz="0.0 0.0   0.1"/>
     <axis xyz="0 1 0"/>
-    <limit effort="1000.0" lower="-1.0" upper="1.0" velocity="1.0"/>
+    <limit effort="10000.0" lower="-1.0" upper="1.0" velocity="1.0"/>
   </joint>
   <joint name="back_lh" type="revolute">
