Commit message: updated xacro

File: boot3_description/urdf/boot.xacro (robot description, xacro)
@@ -12,4 +12,5 @@
     <child link="l1"/>
     <origin xyz="0 0 0.25" rpy="0 0 0"/>
+    <dynamics damping="0.005" />
     <axis xyz="1 0 0"/>
     <limit effort="1000.0" lower="0" upper="1000" velocity="0.5"/>
@@ -19,4 +20,5 @@
     <child link="l2"/>
     <origin xyz="0.0 0 -0.2" rpy="0 ${pi/2} 0"/>
+    <dynamics damping="0.005" />
     <axis xyz="0 1 0"/>
     <limit effort="1000.0" lower="-1" upper="1" velocity="1.0"/>
@@ -26,4 +28,5 @@
     <child link="skiff"/>
     <origin xyz="0.0 0.0 0.4" rpy="${pi} ${pi/2} 0"/>
+    <dynamics damping="0.005" />
     <axis xyz="0 1 0"/>
     <limit effort="1000.0" lower="-1" upper="1" velocity="1.0"/>
@@ -33,4 +36,5 @@
     <child link="starboard_rowlock_l"/>
     <origin rpy="0.0  0.0 -0.61" xyz="-3 ${span/2} 0.42"/>
+    <dynamics damping="0.005" />
     <axis xyz="0 0 1"/>
     <limit effort="1000.0" lower="-0.4" upper="1.4" velocity="1.0"/>
@@ -40,4 +44,5 @@
     <child link="port_rowlock_l"/>
     <origin rpy="0.0  0.0 0.0" xyz="-3 -${span/2} 0.4"/>
+    <dynamics damping="0.005" />
     <axis xyz="0 0 1"/>
     <limit effort="1000.0" lower="-1.4" upper="1.4" velocity="1.0"/>
@@ -47,4 +52,5 @@
     <child link="starboard_oar_l"/>
     <origin rpy="0.0  ${pi/2-0.13} -${pi/2}" xyz="0.0 0.0   0.02"/>
+    <dynamics damping="0.005" />
     <axis xyz="0 1 0"/>
     <limit effort="1000.0" lower="-0.4" upper="0.1" velocity="1.0"/>
@@ -54,4 +60,5 @@
     <child link="port_oar_l"/>
     <origin rpy="0.0  ${pi/2} -${pi/2}" xyz="0.0 0.0   0.02"/>
+    <dynamics damping="0.005" />
     <axis xyz="0 1 0"/>
     <limit effort="1000.0" lower="0.0" upper="0.4" velocity="1.0"/>
@@ -61,4 +68,5 @@
     <child link="starboard_blade_l"/>
     <origin rpy="0 0  0.0" xyz="0.0 0.0   -${outer}"/>
+    <dynamics damping="0.005" />
     <axis xyz="0 1 0"/>
     <limit effort="1000.0" lower="-0.4" upper="0.4" velocity="1.0"/>
@@ -68,4 +76,5 @@
     <child link="port_blade_l"/>
     <origin rpy="0.0  0 0.0" xyz="0.0 0.0   ${outer}"/>
+    <dynamics damping="0.005" />
     <axis xyz="0 1 0"/>
     <limit effort="1000.0" lower="-0.4" upper="0.4" velocity="1.0"/>
@@ -76,4 +85,5 @@
     <child link="footplate"/>
     <origin rpy="0.0  0 0.0" xyz="-2.5 0.0  0.2"/>
+    <dynamics damping="0.005" />
     <limit effort="1000.0" lower="-0.4" upper="0.4" velocity="1.0"/>
   </joint>
@@ -82,4 +92,5 @@
     <child link="seat"/>
     <origin rpy="0 0 0" xyz="-3.495 0.0 0.2"/>
+    <dynamics damping="0.005" />
     <axis xyz="1 0 0"/>
     <limit effort="1000.0" lower="-0.1" upper="0.8" velocity="0.5"/>
@@ -89,4 +100,5 @@
     <child link="lowerleg"/>
     <origin rpy="0.0  0.0998 0.0" xyz="0.0 0.0   0.0"/>
+    <dynamics damping="0.005" />
     <axis xyz="0 1 0"/>
     <limit effort="1000.0" lower="0.0" upper="${pi/2}" velocity="1.0"/>
@@ -96,4 +108,5 @@
     <child link="upperleg_1"/>
     <origin rpy="0.0  0 0.0" xyz="-0.5 0.0   0.0"/>
+    <dynamics damping="0.005" />
     <axis xyz="0 1 0"/>
     <limit effort="10000.0" lower="-3.1" upper="0" velocity="1.0"/>
@@ -103,4 +116,5 @@
     <child link="upperleg_2"/>
     <origin rpy="0  0.0998 0.0" xyz="0.0 0.0   0.1"/>
+    <dynamics damping="0.005" />
     <axis xyz="0 1 0"/>
     <limit effort="1000.0" lower="-1.6" upper="0" velocity="1.0"/>
@@ -110,4 +124,5 @@
     <child link="back_low"/>
     <origin rpy="0  -${pi/2+0.34} 0.0" xyz="0.0 0.0   0.1"/>
+    <dynamics damping="0.005" />
     <axis xyz="0 1 0"/>
     <limit effort="10000.0" lower="-1.0" upper="1.0" velocity="1.0"/>
@@ -117,4 +132,5 @@
     <child link="back_high"/>
     <origin rpy="0  0.0 0.0" xyz="0.3 0.0   0.0"/>
+    <dynamics damping="0.005" />
     <axis xyz="0 1 0"/>
     <limit effort="1000.0" lower="0.0" upper="0.5" velocity="1.0"/>
@@ -124,4 +140,5 @@
     <child link="shoulder_link"/>
     <origin rpy="0  0.0 0.0" xyz="0.3 0.0   0.0"/>
+    <dynamics damping="0.005" />
     <limit effort="1000.0" lower="0.0" upper="0.5" velocity="1.0"/>
   </joint>
@@ -139,7 +156,13 @@
     <inertial>
       <mass value="0.01"/>
-      <origin rpy="0 0 0" xyz="0 0.0 0.2"/>
-      <inertia ixx="0.006" ixy="0" ixz="0" iyy="0.1" iyz="0" izz="0.1"/>
-    </inertial>
+      <origin rpy="0 0 0" xyz="0 0.0 0.0"/>
+      <inertia ixx="0.000000167" ixy="0" ixz="0" iyy="0.000000167" iyz="0" izz="0.000000167"/>
+    </inertial>
+    <visual>
+      <origin rpy="0 0 0" xyz="0.0 0.0 0.0"/>
+      <geometry>
+        <box size="0.01 0.01 0.01"/>
+      </geometry>
+    </visual>
   </link>
   <joint name="shoulder_iets" type="revolute" >
@@ -155,7 +178,13 @@
     <inertial>
       <mass value="0.01"/>
-      <origin rpy="0 0 0" xyz="0 0.0 0.2"/>
-      <inertia ixx="0.006" ixy="0" ixz="0" iyy="0.1" iyz="0" izz="0.1"/>
-    </inertial>
+      <origin rpy="0 0 0" xyz="0 0.0 0.0"/>
+      <inertia ixx="0.000000167" ixy="0" ixz="0" iyy="0.000000167" iyz="0" izz="0.000000167"/>
+    </inertial>
+    <visual>
+      <origin rpy="0 0 0" xyz="0.0 0.0 0.0"/>
+      <geometry>
+        <box size="0.01 0.01 0.01"/>
+      </geometry>
+    </visual>
   </link>
   <joint name="LShoulderTheta" type="revolute" >
@@ -180,7 +209,13 @@
     <inertial>
       <mass value="0.01"/>
-      <origin rpy="0 0 0" xyz="0 0.0 0.2"/>
-      <inertia ixx="0.006" ixy="0" ixz="0" iyy="0.1" iyz="0" izz="0.1"/>
-    </inertial>
+      <origin rpy="0 0 0" xyz="0 0.0 0.0"/>
+      <inertia ixx="0.000000167" ixy="0" ixz="0" iyy="0.000000167" iyz="0" izz="0.000000167"/>
+    </inertial>
+    <visual>
+      <origin rpy="0 0 0" xyz="0.0 0.0 0.0"/>
+      <geometry>
+        <box size="0.01 0.01 0.01"/>
+      </geometry>
+    </visual>
   </link>
   <joint name="RShoulderTheta" type="revolute" >
@@ -204,6 +239,12 @@
       <mass value="0.01"/>
       <origin rpy="0 0 0" xyz="0 0.0 0.0"/>
-      <inertia ixx="0.006" ixy="0" ixz="0" iyy="0.1" iyz="0" izz="0.1"/>
-    </inertial>
+      <inertia ixx="0.000000167" ixy="0" ixz="0" iyy="0.000000167" iyz="0" izz="0.000000167"/>
+    </inertial>
+    <visual>
+      <origin rpy="0 0 0" xyz="0.0 0.0 0.0"/>
+      <geometry>
+        <box size="0.01 0.01 0.01"/>
+      </geometry>
+    </visual>
   </link>
   <joint name="elbow_left" type="revolute">
@@ -211,4 +252,5 @@
     <child link="arm_l_lower_1"/>
     <origin rpy="0 0 -0.09" xyz="0 0.0 0.0"/>
+    <dynamics damping="0.005" />
     <axis xyz="0 0 1"/>
     <limit effort="1000.0" lower="-1.0" upper="1.0" velocity="1.0"/>
@@ -219,4 +261,5 @@
     <child link="dummy_link_1"/>
     <origin rpy="0 0 0.0" xyz="-0.2 0.0 0.0"/>
+    <dynamics damping="0.005" />
     <limit effort="1000.0" lower="-1.0" upper="1.0" velocity="1.0"/>
   </joint>
@@ -224,7 +267,13 @@
     <inertial>
       <mass value="0.01"/>
-      <origin rpy="0 0 0" xyz="0.0 0.0 0.0"/>
-      <inertia ixx="0.006" ixy="0" ixz="0" iyy="0.1" iyz="0" izz="0.1"/>
-    </inertial>
+      <origin rpy="0 0 0" xyz="0 0.0 0.0"/>
+      <inertia ixx="0.000000167" ixy="0" ixz="0" iyy="0.000000167" iyz="0" izz="0.000000167"/>
+    </inertial>
+    <visual>
+      <origin rpy="0 0 0" xyz="0.0 0.0 0.0"/>
+      <geometry>
+        <box size="0.01 0.01 0.01"/>
+      </geometry>
+    </visual>
   </link>
   <joint name="dummy_2" type="fixed">
@@ -232,4 +281,5 @@
     <child link="dummy_link_2"/>
     <origin rpy="${pi/2} ${pi}  0.0" xyz="-0.15 0.0 0.0"/>
+    <dynamics damping="0.005" />
     <limit effort="1000.0" lower="-1.0" upper="1.0" velocity="1.0"/>
   </joint>
@@ -237,7 +287,13 @@
     <inertial>
       <mass value="0.01"/>
-      <origin rpy="0 0 0" xyz="0.0 0.0 0.0"/>
-      <inertia ixx="0.006" ixy="0" ixz="0" iyy="0.1" iyz="0" izz="0.1"/>
-    </inertial>
+      <origin rpy="0 0 0" xyz="0 0.0 0.0"/>
+      <inertia ixx="0.000000167" ixy="0" ixz="0" iyy="0.000000167" iyz="0" izz="0.000000167"/>
+    </inertial>
+    <visual>
+      <origin rpy="0 0 0" xyz="0.0 0.0 0.0"/>
+      <geometry>
+        <box size="0.01 0.01 0.01"/>
+      </geometry>
+    </visual>
   </link>
   <!-- 3D handle joint -->
@@ -246,4 +302,5 @@
     <child link="handle_left_l1"/>
     <origin rpy="0.209 0 ${pi/2}" xyz="0 0.0 ${inner}"/>
+    <dynamics damping="0.005" />
     <axis xyz="1 0 0"/>
     <limit effort="1000.0" lower="-0.2" upper="0.2" velocity="1.0"/>
@@ -253,6 +310,12 @@
       <mass value="0.01"/>
       <origin rpy="0 0 0" xyz="0 0.0 0.0"/>
-      <inertia ixx="0.006" ixy="0" ixz="0" iyy="0.1" iyz="0" izz="0.1"/>
-    </inertial>
+      <inertia ixx="0.000000167" ixy="0" ixz="0" iyy="0.000000167" iyz="0" izz="0.000000167"/>
+    </inertial>
+    <visual>
+      <origin rpy="0 0 0" xyz="0.0 0.0 0.0"/>
+      <geometry>
+        <box size="0.01 0.01 0.01"/>
+      </geometry>
+    </visual>
   </link>
   <joint name="handle_left_j2" type="revolute">
@@ -260,4 +323,5 @@
     <child link="handle_left_l2"/>
     <origin rpy="0 0 0.06" xyz="0 0.0 0.0"/>
+    <dynamics damping="0.005" />
     <axis xyz="0  0 1"/>
     <limit effort="1000.0" lower="-0.2" upper="0.2" velocity="1.0"/>
@@ -267,6 +331,12 @@
       <mass value="0.01"/>
       <origin rpy="0 0 0" xyz="0 0.0 0.0"/>
-      <inertia ixx="0.006" ixy="0" ixz="0" iyy="0.1" iyz="0" izz="0.1"/>
-    </inertial>
+      <inertia ixx="0.000000167" ixy="0" ixz="0" iyy="0.000000167" iyz="0" izz="0.000000167"/>
+    </inertial>
+    <visual>
+      <origin rpy="0 0 0" xyz="0.0 0.0 0.0"/>
+      <geometry>
+        <box size="0.01 0.01 0.01"/>
+      </geometry>
+    </visual>
   </link>
   <joint name="handle_left_j3" type="revolute">
@@ -274,4 +344,5 @@
     <child link="arm_l_lower_2"/>
     <origin rpy="0 -0.16 0" xyz="0 0.0 0.0"/>
+    <dynamics damping="0.005" />
     <axis xyz="0 1 0"/>
     <limit effort="1000.0" lower="-0.2" upper="0.2" velocity="1.0"/>
@@ -288,5 +359,5 @@
       <mass value="0.01"/>
       <origin rpy="0 0 0" xyz="0 0.0 -0.1"/>
-      <inertia ixx="0.006" ixy="0" ixz="0" iyy="0.1" iyz="0" izz="0.1"/>
+      <inertia ixx="0.000033" ixy="0" ixz="0" iyy="0.000033" iyz="0" izz="0.000000167"/>
     </inertial>
     <visual>
@@ -301,5 +372,5 @@
       <mass value="0.01"/>
       <origin rpy="0 0 0" xyz="0 0.0 0.2"/>
-      <inertia ixx="0.006" ixy="0" ixz="0" iyy="0.1" iyz="0" izz="0.1"/>
+      <inertia ixx="0.000133" ixy="0" ixz="0" iyy="0.1=000133" iyz="0" izz="0.000000167"/>
     </inertial>
     <visual>
@@ -314,5 +385,5 @@
       <mass value="${15 + weight}"/>   <!-- boat plus roeier -->
       <origin rpy="0 0 0" xyz="-3 0.0 0.05"/>
-      <inertia ixx="3.2" ixy="0" ixz="0" iyy="54.2" iyz="0" izz="57"/>
+      <inertia ixx="3.2" ixy="0" ixz="0" iyy="225" iyz="0" izz="228"/>   <!-- weight= 60 -->
 <!--      <inertia ixx="0.6" ixy="0" ixz="0" iyy="11" iyz="0" izz="11.8"/>  -->
     </inertial>
@@ -450,5 +521,5 @@
       <mass value="0.1"/>
       <origin rpy="0 0 0" xyz="0 0.0 0.0"/>
-      <inertia ixx="0.001" ixy="0" ixz="0" iyy="0.0005" iyz="0" izz="0.001"/>
+      <inertia ixx="0.0008" ixy="0" ixz="0" iyy="0.000166" iyz="0" izz="0.0008"/>
     </inertial>
     <collision>
@@ -547,5 +618,5 @@
       <mass value="10.0"/>
       <origin rpy="0 0 0" xyz="0.15 0.0 0.0"/>
-      <inertia ixx="0.001" ixy="0" ixz="0" iyy="0.0005" iyz="0" izz="0.001"/>
+      <inertia ixx="0.01" ixy="0" ixz="0" iyy="0.077" iyz="0" izz="0.083"/>
     </inertial>
     <collision>
@@ -585,5 +656,5 @@
       <mass value="1.0"/>
       <origin rpy="0 0 0" xyz="0.0 0.0 0.0"/>
-      <inertia ixx="0.001" ixy="0" ixz="0" iyy="0.0005" iyz="0" izz="0.001"/>
+      <inertia ixx="0.013" ixy="0" ixz="0" iyy="0.0004" iyz="0" izz="0.013"/>
     </inertial>
     <collision>
@@ -604,5 +675,5 @@
       <mass value="1.0"/>
       <origin rpy="0 0 0" xyz="-0.175 0.0 0.0"/>
-      <inertia ixx="0.001" ixy="0" ixz="0" iyy="0.0005" iyz="0" izz="0.001"/>
+      <inertia ixx="0.004" ixy="0" ixz="0" iyy="0.01" iyz="0" izz="0.01"/>
     </inertial>
     <collision>
@@ -624,5 +695,5 @@
       <mass value="1.0"/>
       <origin rpy="0 0 0" xyz="0.175 0.0 0.0"/>
-      <inertia ixx="0.001" ixy="0" ixz="0" iyy="0.0005" iyz="0" izz="0.001"/>
+      <inertia ixx="0.004" ixy="0" ixz="0" iyy="0.01" iyz="0" izz="0.01"/>
     </inertial>
     <collision>
@@ -644,5 +715,5 @@
       <mass value="1.0"/>
       <origin rpy="0 0 0" xyz="-0.1 0.0 0.0"/>
-      <inertia ixx="0.001" ixy="0" ixz="0" iyy="0.0005" iyz="0" izz="0.001"/>
+      <inertia ixx="0.0004" ixy="0" ixz="0" iyy="0.0035" iyz="0" izz="0.0035"/>
     </inertial>
     <collision>
@@ -663,5 +734,5 @@
       <mass value="1.0"/>
       <origin rpy="0 0 0" xyz="-0.075 0.0 0.0"/>
-      <inertia ixx="0.001" ixy="0" ixz="0" iyy="0.0005" iyz="0" izz="0.001"/>
+      <inertia ixx="0.004" ixy="0" ixz="0" iyy="0.002" iyz="0" izz="0.002"/>
     </inertial>
     <collision>
@@ -682,5 +753,5 @@
       <mass value="5.0"/>
       <origin rpy="0 0 0" xyz="-0.1 0.0 0.0"/>
-      <inertia ixx="0.001" ixy="0" ixz="0" iyy="0.0005" iyz="0" izz="0.001"/>
+      <inertia ixx="0.0128" ixy="0" ixz="0" iyy="0.0128" iyz="0" izz="0.0128"/>
     </inertial>
     <collision>

Commit message: reduce limits

File: boot3_description/urdf/boot.xacro (robot description, xacro)
@@ -14,5 +14,5 @@
     <dynamics damping="0.005" />
     <axis xyz="1 0 0"/>
-    <limit effort="1000.0" lower="0" upper="1000" velocity="0.5"/>
+    <limit effort="101.0" lower="0" upper="1000" velocity="0.5"/>
   </joint>
   <joint name="rev1" type="revolute">
@@ -22,5 +22,5 @@
     <dynamics damping="0.005" />
     <axis xyz="0 1 0"/>
-    <limit effort="1000.0" lower="-1" upper="1" velocity="1.0"/>
+    <limit effort="101.0" lower="-1" upper="1" velocity="1.0"/>
   </joint>
   <joint name="rev2" type="revolute">
@@ -30,5 +30,5 @@
     <dynamics damping="0.005" />
     <axis xyz="0 1 0"/>
-    <limit effort="1000.0" lower="-1" upper="1" velocity="1.0"/>
+    <limit effort="101.0" lower="-1" upper="1" velocity="1.0"/>
   </joint>
   <joint name="starboard_rowlock" type="revolute">
@@ -38,5 +38,5 @@
     <dynamics damping="0.005" />
     <axis xyz="0 0 1"/>
-    <limit effort="1000.0" lower="-0.4" upper="1.4" velocity="1.0"/>
+    <limit effort="101.0" lower="-0.4" upper="1.4" velocity="1.0"/>
   </joint>
   <joint name="port_rowlock" type="revolute">
@@ -46,5 +46,5 @@
     <dynamics damping="0.005" />
     <axis xyz="0 0 1"/>
-    <limit effort="1000.0" lower="-1.4" upper="1.4" velocity="1.0"/>
+    <limit effort="101.0" lower="-1.4" upper="1.4" velocity="1.0"/>
   </joint>
   <joint name="starboard_oar" type="revolute">
@@ -54,5 +54,5 @@
     <dynamics damping="0.005" />
     <axis xyz="0 1 0"/>
-    <limit effort="1000.0" lower="-0.4" upper="0.1" velocity="1.0"/>
+    <limit effort="101.0" lower="-0.4" upper="0.1" velocity="1.0"/>
   </joint>
   <joint name="port_oar" type="revolute">
@@ -62,5 +62,5 @@
     <dynamics damping="0.005" />
     <axis xyz="0 1 0"/>
-    <limit effort="1000.0" lower="0.0" upper="0.4" velocity="1.0"/>
+    <limit effort="101.0" lower="0.0" upper="0.4" velocity="1.0"/>
   </joint>
   <joint name="starboard_blade" type="revolute">
@@ -70,5 +70,5 @@
     <dynamics damping="0.005" />
     <axis xyz="0 1 0"/>
-    <limit effort="1000.0" lower="-0.4" upper="0.4" velocity="1.0"/>
+    <limit effort="101.0" lower="-0.4" upper="0.4" velocity="1.0"/>
   </joint>
   <joint name="port_blade" type="revolute">
@@ -78,5 +78,5 @@
     <dynamics damping="0.005" />
     <axis xyz="0 1 0"/>
-    <limit effort="1000.0" lower="-0.4" upper="0.4" velocity="1.0"/>
+    <limit effort="101.0" lower="-0.4" upper="0.4" velocity="1.0"/>
   </joint>
   <!-- Rower joints -->
@@ -86,5 +86,5 @@
     <origin rpy="0.0  0 0.0" xyz="-2.5 0.0  0.2"/>
     <dynamics damping="0.005" />
-    <limit effort="1000.0" lower="-0.4" upper="0.4" velocity="1.0"/>
+    <limit effort="101.0" lower="-0.4" upper="0.4" velocity="1.0"/>
   </joint>
   <joint name="sliding" type="prismatic">
@@ -94,5 +94,5 @@
     <dynamics damping="0.005" />
     <axis xyz="1 0 0"/>
-    <limit effort="1000.0" lower="-0.1" upper="0.8" velocity="0.5"/>
+    <limit effort="101.0" lower="-0.1" upper="0.8" velocity="0.5"/>
   </joint>
   <joint name="fp_ll" type="revolute">
@@ -102,5 +102,5 @@
     <dynamics damping="0.005" />
     <axis xyz="0 1 0"/>
-    <limit effort="1000.0" lower="0.0" upper="${pi/2}" velocity="1.0"/>
+    <limit effort="101.0" lower="0.0" upper="${pi/2}" velocity="1.0"/>
   </joint>
   <joint name="knee" type="revolute">
@@ -110,5 +110,5 @@
     <dynamics damping="0.005" />
     <axis xyz="0 1 0"/>
-    <limit effort="10000.0" lower="-3.1" upper="0" velocity="1.0"/>
+    <limit effort="1000.0" lower="-3.1" upper="0" velocity="1.0"/>
   </joint>
   <joint name="hip1" type="revolute">
@@ -118,5 +118,5 @@
     <dynamics damping="0.005" />
     <axis xyz="0 1 0"/>
-    <limit effort="1000.0" lower="-1.6" upper="0" velocity="1.0"/>
+    <limit effort="101.0" lower="-1.6" upper="0" velocity="1.0"/>
   </joint>
   <joint name="hip2" type="revolute">
@@ -126,5 +126,5 @@
     <dynamics damping="0.005" />
     <axis xyz="0 1 0"/>
-    <limit effort="10000.0" lower="-1.0" upper="1.0" velocity="1.0"/>
+    <limit effort="1000.0" lower="-1.0" upper="1.0" velocity="1.0"/>
   </joint>
   <joint name="back_lh" type="revolute">
@@ -134,5 +134,5 @@
     <dynamics damping="0.005" />
     <axis xyz="0 1 0"/>
-    <limit effort="1000.0" lower="0.0" upper="0.5" velocity="1.0"/>
+    <limit effort="101.0" lower="0.0" upper="0.5" velocity="1.0"/>
   </joint>
   <joint name="shoulder" type="fixed">
@@ -141,5 +141,5 @@
     <origin rpy="0  0.0 0.0" xyz="0.3 0.0   0.0"/>
     <dynamics damping="0.005" />
-    <limit effort="1000.0" lower="0.0" upper="0.5" velocity="1.0"/>
+    <limit effort="101.0" lower="0.0" upper="0.5" velocity="1.0"/>
   </joint>
   <!-- 3D joint left shoulder -->
@@ -150,6 +150,6 @@
     <axis xyz="0 0 1" />
     <dynamics damping="0.005" />
-    <!--    <limit effort="1000.0" lower="-1.5" upper="0.5" velocity="1.0"/> -->
-    <limit effort="1000.0" lower="-0.1" upper="0.1" velocity="1.0"/>
+    <!--    <limit effort="101.0" lower="-1.5" upper="0.5" velocity="1.0"/> -->
+    <limit effort="101.0" lower="-0.1" upper="0.1" velocity="1.0"/>
   </joint>
   <link name="left_shoulder_xx_link">
@@ -172,6 +172,6 @@
     <axis xyz="1 0 0" />
     <dynamics damping="0.005" />
-<!--    <limit effort="1000.0" lower="-1.5" upper="1.5" velocity="1.0"/> -->
-    <limit effort="1000.0" lower="-0.2" upper="0.2" velocity="1.0"/>
+<!--    <limit effort="101.0" lower="-1.5" upper="1.5" velocity="1.0"/> -->
+    <limit effort="101.0" lower="-0.2" upper="0.2" velocity="1.0"/>
   </joint>
   <link name="left_shoulder_psi_link">
@@ -194,6 +194,6 @@
     <axis xyz="0 1 0" />
     <dynamics damping="0.005" />
-<!--    <limit effort="1000.0" lower="-2.0" upper="1.0" velocity="1.0"/> -->
-    <limit effort="1000.0" lower="-0.2" upper="0.2" velocity="1.0"/>
+<!--    <limit effort="101.0" lower="-2.0" upper="1.0" velocity="1.0"/> -->
+    <limit effort="101.0" lower="-0.2" upper="0.2" velocity="1.0"/>
   </joint>
   <!-- 2D joint right shoulder -->
@@ -204,5 +204,5 @@
     <axis xyz="0 0 1" />
     <dynamics damping="0.005" />
-    <limit effort="1000.0" lower="-1.0" upper="0.5" velocity="1.0"/>
+    <limit effort="101.0" lower="-1.0" upper="0.5" velocity="1.0"/>
   </joint>
   <link name="right_shoulder_psi_link">
@@ -224,5 +224,5 @@
     <axis xyz="0 1 0" />
     <dynamics damping="0.005" />
-    <limit effort="1000.0" lower="-1.5" upper="1.0" velocity="1.0"/>
+    <limit effort="101.0" lower="-1.5" upper="1.0" velocity="1.0"/>
   </joint>
   <!-- 2D joint left elbow -->
@@ -233,5 +233,5 @@
     <axis xyz="0 1 0" />
     <dynamics damping="0.005" />
-    <limit effort="1000.0" lower="-0.7" upper="2.0" velocity="1.0"/>
+    <limit effort="101.0" lower="-0.7" upper="2.0" velocity="1.0"/>
   </joint>
   <link name="left_elbow_psi_link">
@@ -254,5 +254,5 @@
     <dynamics damping="0.005" />
     <axis xyz="0 0 1"/>
-    <limit effort="1000.0" lower="-1.0" upper="1.0" velocity="1.0"/>
+    <limit effort="101.0" lower="-1.0" upper="1.0" velocity="1.0"/>
   </joint>
   <!-- hoe kom ik aan de andere kant van arm_lower_1 en 2 ?  -->
@@ -262,5 +262,5 @@
     <origin rpy="0 0 0.0" xyz="-0.2 0.0 0.0"/>
     <dynamics damping="0.005" />
-    <limit effort="1000.0" lower="-1.0" upper="1.0" velocity="1.0"/>
+    <limit effort="101.0" lower="-1.0" upper="1.0" velocity="1.0"/>
   </joint>
   <link name="dummy_link_1">
@@ -282,5 +282,5 @@
     <origin rpy="${pi/2} ${pi}  0.0" xyz="-0.15 0.0 0.0"/>
     <dynamics damping="0.005" />
-    <limit effort="1000.0" lower="-1.0" upper="1.0" velocity="1.0"/>
+    <limit effort="101.0" lower="-1.0" upper="1.0" velocity="1.0"/>
   </joint>
   <link name="dummy_link_2">
@@ -304,5 +304,5 @@
     <dynamics damping="0.005" />
     <axis xyz="1 0 0"/>
-    <limit effort="1000.0" lower="-0.2" upper="0.2" velocity="1.0"/>
+    <limit effort="101.0" lower="-0.2" upper="0.2" velocity="1.0"/>
   </joint>
   <link name="handle_left_l1">
@@ -325,5 +325,5 @@
     <dynamics damping="0.005" />
     <axis xyz="0  0 1"/>
-    <limit effort="1000.0" lower="-0.2" upper="0.2" velocity="1.0"/>
+    <limit effort="101.0" lower="-0.2" upper="0.2" velocity="1.0"/>
   </joint>
   <link name="handle_left_l2">
@@ -346,5 +346,5 @@
     <dynamics damping="0.005" />
     <axis xyz="0 1 0"/>
-    <limit effort="1000.0" lower="-0.2" upper="0.2" velocity="1.0"/>
+    <limit effort="101.0" lower="-0.2" upper="0.2" velocity="1.0"/>
   </joint>
   <joint name="head_joint" type="fixed">
