Commit message: updated xacro's

File: boot3_description/urdf/boot.xacro (robot description, xacro)
@@ -35,5 +35,5 @@
     <parent link="skiff"/>
     <child link="starboard_rowlock_l"/>
-    <origin rpy="0.0  0.0 -0.61" xyz="-3 ${span} 0.42"/>
+    <origin rpy="0.0  0.0 -0.61" xyz="-3 ${span} 0.42"/>   <!-- span/2  -->
     <dynamics damping="0.005" />
     <axis xyz="0 0 1"/>
@@ -43,5 +43,5 @@
     <parent link="skiff"/>
     <child link="port_rowlock_l"/>
-    <origin rpy="0.0  0.0 0.0" xyz="-3 -${span/2} 0.4"/>
+    <origin rpy="0.0  0.0 0.61" xyz="-3 -${span/2} 0.4"/>
     <dynamics damping="0.005" />
     <axis xyz="0 0 1"/>
@@ -59,5 +59,5 @@
     <parent link="port_rowlock_l"/>
     <child link="port_oar_l"/>
-    <origin rpy="0.0  ${pi/2} -${pi/2}" xyz="0.0 0.0   0.02"/>
+    <origin rpy="0.0  ${pi/2+0.13} -${pi/2}" xyz="0.0 0.0   0.02"/>
     <dynamics damping="0.005" />
     <axis xyz="0 1 0"/>
@@ -81,5 +81,5 @@
   </joint>
   <!-- Rower joints -->
-  <joint name="sk_fp" type="revolute">
+  <joint name="sk_fp" type="fixed">
     <parent link="skiff"/>
     <child link="footplate"/>
@@ -91,5 +91,5 @@
     <parent link="skiff"/>
     <child link="seat"/>
-    <origin rpy="0 0 0" xyz="-3.495 0.0 0.2"/>
+    <origin rpy="0 0 0" xyz="-3.49514 0.0 0.2"/>
     <dynamics damping="0.005" />
     <axis xyz="1 0 0"/>
@@ -99,5 +99,5 @@
     <parent link="footplate"/>
     <child link="lowerleg"/>
-    <origin rpy="0.0  0.0998 0.0" xyz="0.0 0.0   0.0"/>
+    <origin rpy="0.0  0.1001675 0.0" xyz="0.0 0.0   0.0"/>
     <dynamics damping="0.005" />
     <axis xyz="0 1 0"/>
@@ -115,5 +115,5 @@
     <parent link="seat"/>
     <child link="upperleg_2"/>
-    <origin rpy="0  0.0998 0.0" xyz="0.0 0.0   0.1"/>
+    <origin rpy="0  0.1001675 0.0" xyz="0.0 0.0   0.1"/>
     <dynamics damping="0.005" />
     <axis xyz="0 1 0"/>
@@ -369,5 +369,5 @@
       <mass value="0.01"/>
       <origin rpy="0 0 0" xyz="0 0.0 0.2"/>
-      <inertia ixx="0.000133" ixy="0" ixz="0" iyy="0.1=000133" iyz="0" izz="0.000000167"/>
+      <inertia ixx="0.000133" ixy="0" ixz="0" iyy="0.000133" iyz="0" izz="0.000000167"/>
     </inertial>
     <visual>
@@ -383,5 +383,4 @@
       <origin rpy="0 0 0" xyz="-3 0.0 0.05"/>
       <inertia ixx="3.2" ixy="0" ixz="0" iyy="225" iyz="0" izz="228"/>   <!-- weight= 60 -->
-<!--      <inertia ixx="0.6" ixy="0" ixz="0" iyy="11" iyz="0" izz="11.8"/>  -->
     </inertial>
     <collision>
@@ -465,5 +464,6 @@
       <origin rpy="0 0 0" xyz="0   0   ${(outer-inner)/2}"/>
       <geometry>
-        <cylinder length="${inner+outer-0.6}" radius="0.02"/>  <!-- -0.6 to prevent collissions  -->
+        <cylinder length="${inner+outer-0.6}" radius="0.02"/>
+	<!-- -0.6 to prevent collissions  -->
       </geometry>
     </collision>

Commit message: tweek urdf

File: boot3_description/urdf/boot.xacro (robot description, xacro)
@@ -165,5 +165,5 @@
     </visual>
   </link>
-  <joint name="shoulder_iets" type="revolute" >
+  <joint name="shoulder_iets" type="fixed" >
     <parent link="left_shoulder_xx_link" />
     <child link="left_shoulder_psi_link" />
@@ -189,5 +189,5 @@
     <parent link="left_shoulder_psi_link"/>
     <child link="arm_l_upper"/>
-      <origin rpy="0 0.68 0" xyz="0 0.0 0.0"/>
+    <origin rpy="0 0.68 0" xyz="0 0.0 0.0"/>
     <axis xyz="0 1 0" />
     <dynamics damping="0.005" />
@@ -634,5 +634,5 @@
       <mass value="10.0"/>
       <origin rpy="0 0 0" xyz="0.15 0.0 0.0"/>
-      <inertia ixx="0.001" ixy="0" ixz="0" iyy="0.0005" iyz="0" izz="0.001"/>
+      <inertia ixx="0.02" ixy="0" ixz="0" iyy="0.077" iyz="0" izz="0.094"/>
     </inertial>
     <collision>
@@ -671,5 +671,4 @@
       <origin rpy="0 0 0" xyz="-0.175 0.0   0.0"/>
       <geometry>
-	fg
         <box size="0.35 0.05 0.05"/>
       </geometry>
@@ -840,23 +839,24 @@
     </actuator>
   </transmission>
+  <transmission name="tran11">
+    <type>transmission_interface/SimpleTransmission</type>
+    <joint name="shoulder_l">
+      <hardwareInterface>hardware_interface/EffortJointInterface</hardwareInterface>
+    </joint>
+    <actuator name="motor11">
+      <mechanicalReduction>1</mechanicalReduction>
+    </actuator>
+  </transmission>
+<!--
+  <transmission name="tran12">
+    <type>transmission_interface/SimpleTransmission</type>
+    <joint name="shoulder_iets">
+      <hardwareInterface>hardware_interface/EffortJointInterface</hardwareInterface>
+    </joint>
+    <actuator name="motor12">
+      <mechanicalReduction>1</mechanicalReduction>
+    </actuator>
+  </transmission>
 -->
-  <transmission name="tran11">
-    <type>transmission_interface/SimpleTransmission</type>
-    <joint name="shoulder_l">
-      <hardwareInterface>hardware_interface/EffortJointInterface</hardwareInterface>
-    </joint>
-    <actuator name="motor11">
-      <mechanicalReduction>1</mechanicalReduction>
-    </actuator>
-  </transmission>
-  <transmission name="tran12">
-    <type>transmission_interface/SimpleTransmission</type>
-    <joint name="shoulder_iets">
-      <hardwareInterface>hardware_interface/EffortJointInterface</hardwareInterface>
-    </joint>
-    <actuator name="motor12">
-      <mechanicalReduction>1</mechanicalReduction>
-    </actuator>
-  </transmission>
   <transmission name="tran13">
     <type>transmission_interface/SimpleTransmission</type>
@@ -868,4 +868,3 @@
     </actuator>
   </transmission>
--->
 </robot>

Commit message: more or less stable version, changed dynamics values

File: boot3_description/urdf/boot.xacro (robot description, xacro)
@@ -8,5 +8,5 @@
   <!-- parameters that can be configured -->
   <xacro:include filename="$(find boot3_description)/config/param.xacro" />
-  <joint name="prism" type="fixed">  <!-- prismatic -->
+  <joint name="prism" type="prismatic">  <!-- prismatic -->
     <parent link="world"/>
     <child link="l1"/>
@@ -16,5 +16,5 @@
     <limit effort="101.0" lower="0" upper="1000" velocity="0.5"/>
   </joint>
-  <joint name="rev1" type="fixed">
+  <joint name="rev1" type="revolute">
     <parent link="l1"/>
     <child link="l2"/>
@@ -24,5 +24,5 @@
     <limit effort="101.0" lower="-1" upper="1" velocity="1.0"/>
   </joint>
-  <joint name="rev2" type="fixed">
+  <joint name="rev2" type="revolute">
     <parent link="l2"/>
     <child link="skiff"/>
@@ -32,13 +32,13 @@
     <limit effort="101.0" lower="-1" upper="1" velocity="1.0"/>
   </joint>
-  <joint name="starboard_rowlock" type="fixed">
+  <joint name="starboard_rowlock" type="revolute">
     <parent link="skiff"/>
     <child link="starboard_rowlock_l"/>
-    <origin rpy="0.0  0.0 -0.61" xyz="-3 ${span} 0.42"/>   <!-- span/2  -->
+    <origin rpy="0.0  0.0 -0.57" xyz="-3 ${span/2} 0.42"/>
     <dynamics damping="0.005" />
     <axis xyz="0 0 1"/>
     <limit effort="101.0" lower="-0.4" upper="1.4" velocity="1.0"/>
   </joint>
-  <joint name="port_rowlock" type="fixed">
+  <joint name="port_rowlock" type="revolute">
     <parent link="skiff"/>
     <child link="port_rowlock_l"/>
@@ -48,5 +48,5 @@
     <limit effort="101.0" lower="-1.4" upper="1.4" velocity="1.0"/>
   </joint>
-  <joint name="starboard_oar" type="fixed">
+  <joint name="starboard_oar" type="revolute">
     <parent link="starboard_rowlock_l"/>
     <child link="starboard_oar_l"/>
@@ -56,5 +56,5 @@
     <limit effort="101.0" lower="-0.4" upper="0.1" velocity="1.0"/>
   </joint>
-  <joint name="port_oar" type="fixed">
+  <joint name="port_oar" type="revolute">
     <parent link="port_rowlock_l"/>
     <child link="port_oar_l"/>
@@ -64,5 +64,5 @@
     <limit effort="101.0" lower="0.0" upper="0.4" velocity="1.0"/>
   </joint>
-  <joint name="starboard_blade" type="fixed">
+  <joint name="starboard_blade" type="revolute">
     <parent link="starboard_oar_l"/>
     <child link="starboard_blade_l"/>
@@ -72,5 +72,5 @@
     <limit effort="101.0" lower="-0.4" upper="0.4" velocity="1.0"/>
   </joint>
-  <joint name="port_blade" type="fixed">
+  <joint name="port_blade" type="revolute">
     <parent link="port_oar_l"/>
     <child link="port_blade_l"/>
@@ -88,5 +88,5 @@
     <limit effort="101.0" lower="-0.4" upper="0.4" velocity="1.0"/>
   </joint>
-  <joint name="sliding" type="prismatic">
+  <joint name="sliding" type="prismatic">   <!-- prismatic -->
     <parent link="skiff"/>
     <child link="seat"/>
@@ -94,5 +94,5 @@
     <dynamics damping="0.005" />
     <axis xyz="1 0 0"/>
-    <limit effort="1000.0" lower="-0.1" upper="0.8" velocity="0.5"/>
+    <limit effort="101.0" lower="-0.1" upper="0.8" velocity="0.5"/>
   </joint>
   <joint name="fp_ll" type="revolute">
@@ -102,5 +102,5 @@
     <dynamics damping="0.005" />
     <axis xyz="0 1 0"/>
-    <limit effort="1000.0" lower="0.0" upper="${pi/2}" velocity="1.0"/>
+    <limit effort="101.0" lower="0.0" upper="${pi/2}" velocity="1.0"/>
   </joint>
   <joint name="knee" type="revolute">
@@ -110,5 +110,5 @@
     <dynamics damping="0.005" />
     <axis xyz="0 1 0"/>
-    <limit effort="100.0" lower="-3.1" upper="0" velocity="1.0"/>
+    <limit effort="1000.0" lower="-3.1" upper="0" velocity="1.0"/>
   </joint>
   <joint name="hip1" type="revolute">
@@ -118,21 +118,21 @@
     <dynamics damping="0.005" />
     <axis xyz="0 1 0"/>
-    <limit effort="100.0" lower="-1.6" upper="0" velocity="1.0"/>
+    <limit effort="101.0" lower="-1.6" upper="0" velocity="1.0"/>
   </joint>
   <joint name="hip2" type="revolute">
     <parent link="seat"/>
     <child link="back_low"/>
-    <origin rpy="0  -${pi/2+0.34} 0.0" xyz="0.0 0.0   0.1"/>
-    <dynamics damping="0.005" />
-    <axis xyz="0 1 0"/>
-    <limit effort="100.0" lower="-1.0" upper="1.0" velocity="1.0"/>
+    <origin rpy="0  -${pi/2+0.329} 0.0" xyz="0.0 0.0   0.1"/>
+    <dynamics damping="0.5" />
+    <axis xyz="0 1 0"/>
+    <limit effort="1000.0" lower="-1.0" upper="1.0" velocity="1.0"/>
   </joint>
   <joint name="back_lh" type="revolute">
     <parent link="back_low"/>
     <child link="back_high"/>
-    <origin rpy="0  0.0 0.0" xyz="0.3 0.0   0.0"/>
-    <dynamics damping="0.005" />
-    <axis xyz="0 1 0"/>
-    <limit effort="100.0" lower="0.0" upper="0.5" velocity="1.0"/>
+    <origin rpy="0  0.011 0.0" xyz="0.3 0.0   0.0"/>
+    <dynamics damping="0.5" />
+    <axis xyz="0 1 0"/>
+    <limit effort="101.0" lower="0.0" upper="0.5" velocity="1.0"/>
   </joint>
   <joint name="shoulder" type="fixed">
@@ -147,8 +147,9 @@
     <parent link="shoulder_link" />
     <child link="left_shoulder_xx_link" />
-    <origin rpy="0.0 0.0 0.13" xyz="0.0 0.2   0.0"/>
+    <origin rpy="0.0 0.0 0.18" xyz="0.0 0.2   0.0"/>
     <axis xyz="0 0 1" />
     <dynamics damping="0.005" />
-    <limit effort="100.0" lower="-1.5" upper="0.5" velocity="1.0"/>
+    <!--    <limit effort="101.0" lower="-1.5" upper="0.5" velocity="1.0"/> -->
+    <limit effort="101.0" lower="-0.1" upper="0.1" velocity="1.0"/>
   </joint>
   <link name="left_shoulder_xx_link">
@@ -165,11 +166,12 @@
     </visual>
   </link>
-  <joint name="shoulder_iets" type="fixed" >
+  <joint name="shoulder_iets" type="revolute" >
     <parent link="left_shoulder_xx_link" />
     <child link="left_shoulder_psi_link" />
-    <origin rpy="-0.803 0.0 0.0" xyz="0.0 0.0   0.0"/>
+    <origin rpy="-0.84 0.0 0.0" xyz="0.0 0.0   0.0"/>
     <axis xyz="1 0 0" />
     <dynamics damping="0.005" />
-    <limit effort="100.0" lower="-1.5" upper="1.5" velocity="1.0"/>
+<!--    <limit effort="101.0" lower="-1.5" upper="1.5" velocity="1.0"/> -->
+    <limit effort="101.0" lower="-0.2" upper="0.2" velocity="1.0"/>
   </joint>
   <link name="left_shoulder_psi_link">
@@ -189,16 +191,17 @@
     <parent link="left_shoulder_psi_link"/>
     <child link="arm_l_upper"/>
-    <origin rpy="0 0.68 0" xyz="0 0.0 0.0"/>
+    <origin rpy="0 0.655 0" xyz="0 0.0 0.0"/>
     <axis xyz="0 1 0" />
     <dynamics damping="0.005" />
-    <limit effort="100.0" lower="-2.0" upper="1.0" velocity="1.0"/>
+<!--    <limit effort="101.0" lower="-2.0" upper="1.0" velocity="1.0"/> -->
+    <limit effort="101.0" lower="-0.2" upper="0.2" velocity="1.0"/>
   </joint>
   <!-- 2D joint right shoulder -->
-  <joint name="shoulder_r" type="fixed" >
+  <joint name="shoulder_r" type="revolute" >
     <parent link="shoulder_link" />
     <child link="right_shoulder_psi_link" />
     <origin rpy="0.0 ${pi}  0.0" xyz="0.0 -0.2   0.0"/>
     <axis xyz="0 0 1" />
-    <dynamics damping="0.005" />
+    <dynamics damping="0.5" />
     <limit effort="101.0" lower="-1.0" upper="0.5" velocity="1.0"/>
   </joint>
@@ -216,18 +219,18 @@
     </visual>
   </link>
-  <joint name="RShoulderTheta" type="fixed" >
+  <joint name="RShoulderTheta" type="revolute" >
     <parent link="right_shoulder_psi_link"/>
     <child link="arm_r_upper"/>
     <axis xyz="0 1 0" />
-    <dynamics damping="0.005" />
+    <dynamics damping="0.5" />
     <limit effort="101.0" lower="-1.5" upper="1.0" velocity="1.0"/>
   </joint>
   <!-- 2D joint left elbow -->
-  <joint name="LElbowTheta" type="fixed" >
+  <joint name="LElbowTheta" type="revolute" >
     <parent link="arm_l_upper"/>
     <child link="left_elbow_psi_link"/>
-    <origin rpy="0.0 -1.94  0.0" xyz="-0.35 0.0  0.0"/>
+    <origin rpy="0.0 -1.90  0.0" xyz="-0.35 0.0  0.0"/>
     <axis xyz="0 1 0" />
-    <dynamics damping="0.005" />
+    <dynamics damping="0.5" />
     <limit effort="101.0" lower="-0.7" upper="2.0" velocity="1.0"/>
   </joint>
@@ -245,9 +248,9 @@
     </visual>
   </link>
-  <joint name="elbow_left" type="fixed">
+  <joint name="elbow_left" type="revolute">
     <parent link="left_elbow_psi_link"/>
     <child link="arm_l_lower_1"/>
-    <origin rpy="0 0 -0.09" xyz="0 0.0 0.0"/>
-    <dynamics damping="0.005" />
+    <origin rpy="0 0 -0.127" xyz="0 0.0 0.0"/>
+    <dynamics damping="0.5" />
     <axis xyz="0 0 1"/>
     <limit effort="101.0" lower="-1.0" upper="1.0" velocity="1.0"/>
@@ -295,5 +298,5 @@
   </link>
   <!-- 3D handle joint -->
-  <joint name="handle_left_j1" type="fixed">
+  <joint name="handle_left_j1" type="revolute">
     <parent link="starboard_oar_l"/>
     <child link="handle_left_l1"/>
@@ -316,5 +319,5 @@
     </visual>
   </link>
-  <joint name="handle_left_j2" type="fixed">
+  <joint name="handle_left_j2" type="revolute">
     <parent link="handle_left_l1"/>
     <child link="handle_left_l2"/>
@@ -337,5 +340,5 @@
     </visual>
   </link>
-  <joint name="handle_left_j3" type="fixed">
+  <joint name="handle_left_j3" type="revolute">
     <parent link="handle_left_l2"/>
     <child link="arm_l_lower_2"/>
@@ -369,5 +372,5 @@
       <mass value="0.01"/>
       <origin rpy="0 0 0" xyz="0 0.0 0.2"/>
-      <inertia ixx="0.000133" ixy="0" ixz="0" iyy="0.000133" iyz="0" izz="0.000000167"/>
+      <inertia ixx="0.000133" ixy="0" ixz="0" iyy="0.1=000133" iyz="0" izz="0.000000167"/>
     </inertial>
     <visual>
@@ -383,4 +386,5 @@
       <origin rpy="0 0 0" xyz="-3 0.0 0.05"/>
       <inertia ixx="3.2" ixy="0" ixz="0" iyy="225" iyz="0" izz="228"/>   <!-- weight= 60 -->
+<!--      <inertia ixx="0.6" ixy="0" ixz="0" iyy="11" iyz="0" izz="11.8"/>  -->
     </inertial>
     <collision>
@@ -464,6 +468,5 @@
       <origin rpy="0 0 0" xyz="0   0   ${(outer-inner)/2}"/>
       <geometry>
-        <cylinder length="${inner+outer-0.6}" radius="0.02"/>
-	<!-- -0.6 to prevent collissions  -->
+        <cylinder length="${inner+outer-0.6}" radius="0.02"/>  <!-- -0.6 to prevent collissions  -->
       </geometry>
     </collision>
@@ -655,4 +658,10 @@
       <inertia ixx="0.013" ixy="0" ixz="0" iyy="0.0004" iyz="0" izz="0.013"/>
     </inertial>
+    <collision>
+      <origin rpy="0 0 0" xyz="0.0  0.0   0.0"/>
+      <geometry>
+        <box size="0.05 0.4 0.05"/>
+      </geometry>
+    </collision>
     <visual>
       <origin rpy="0 0 0" xyz="0.0 0.0   0.0"/>
@@ -668,4 +677,10 @@
       <inertia ixx="0.004" ixy="0" ixz="0" iyy="0.01" iyz="0" izz="0.01"/>
     </inertial>
+    <collision>
+      <origin rpy="0 0 0" xyz="-0.175 0.0   0.0"/>
+      <geometry>
+        <box size="0.35 0.05 0.05"/>
+      </geometry>
+    </collision>
     <visual>
       <origin rpy="0 0 0" xyz="-0.175 0.0   0.0"/>
@@ -701,4 +716,10 @@
       <inertia ixx="0.0004" ixy="0" ixz="0" iyy="0.0035" iyz="0" izz="0.0035"/>
     </inertial>
+    <collision>
+      <origin rpy="0 0 0" xyz="-0.1 0.0   0.0"/>
+      <geometry>
+        <box size="0.20 0.05 0.05"/>
+      </geometry>
+    </collision>
     <visual>
       <origin rpy="0 0 0" xyz="-0.1 0.0   0.0"/>
@@ -747,5 +768,4 @@
   </link>
 <!-- Boat transmissions -->
-<!--
   <transmission name="tran1">
     <type>transmission_interface/SimpleTransmission</type>
@@ -792,5 +812,5 @@
       <mechanicalReduction>1</mechanicalReduction>
     </actuator>
-st  </transmission>
+  </transmission>
   <transmission name="tran6">
     <type>transmission_interface/SimpleTransmission</type>
@@ -802,5 +822,5 @@
     </actuator>
   </transmission>
--->
+  <!-- Rower transmissions -->
   <transmission name="tran7">
     <type>transmission_interface/SimpleTransmission</type>
@@ -848,5 +868,4 @@
     </actuator>
   </transmission>
-<!--
   <transmission name="tran12">
     <type>transmission_interface/SimpleTransmission</type>
@@ -858,5 +877,4 @@
     </actuator>
   </transmission>
--->
   <transmission name="tran13">
     <type>transmission_interface/SimpleTransmission</type>

Commit message: repair more

File: boot3_description/urdf/boot.xacro (robot description, xacro)
@@ -82,5 +82,5 @@
   <!-- Rower joints -->
   <joint name="sk_fp" type="fixed">
-    <parent link="world"/>
+    <parent link="skiff"/>
     <child link="footplate"/>
     <origin rpy="0.0  0 0.0" xyz="-2.5 0.0  0.2"/>
@@ -124,5 +124,5 @@
     <child link="back_low"/>
     <origin rpy="0  -${pi/2+0.329} 0.0" xyz="0.0 0.0   0.1"/>
-    <dynamics damping="0.5" />
+    <dynamics damping="0.005" />
     <axis xyz="0 1 0"/>
     <limit effort="1000.0" lower="-1.0" upper="1.0" velocity="1.0"/>
@@ -140,5 +140,5 @@
     <child link="shoulder_link"/>
     <origin rpy="0  0.0 0.0" xyz="0.3 0.0   0.0"/>
-    <dynamics damping="0.005" />
+    <dynamics damping="0.5" />
     <limit effort="101.0" lower="0.0" upper="0.5" velocity="1.0"/>
   </joint>
@@ -690,4 +690,23 @@
     </visual>
   </link>
+  <link name="arm_r_upper">
+    <inertial>
+      <mass value="1.0"/>
+      <origin rpy="0 0 0" xyz="0.175 0.0 0.0"/>
+      <inertia ixx="0.004" ixy="0" ixz="0" iyy="0.01" iyz="0" izz="0.01"/>
+    </inertial>
+    <collision>
+      <origin rpy="0 0 0" xyz="0.175 0.0   0.0"/>
+      <geometry>
+        <box size="0.35 0.05 0.05"/>
+      </geometry>
+    </collision>
+    <visual>
+      <origin rpy="0 0 0" xyz="0.175 0.0   0.0"/>
+      <geometry>
+        <box size="0.35 0.05 0.05"/>
+      </geometry>
+    </visual>
+  </link>
   <!-- lower arm in two to create a kinematic loop in gazebo -->
   <link name="arm_l_lower_1">
@@ -710,4 +729,42 @@
     </visual>
   </link>
+  <link name="arm_l_lower_2">
+    <inertial>
+      <mass value="1.0"/>
+      <origin rpy="0 0 0" xyz="-0.075 0.0 0.0"/>
+      <inertia ixx="0.004" ixy="0" ixz="0" iyy="0.002" iyz="0" izz="0.002"/>
+    </inertial>
+    <collision>
+      <origin rpy="0 0 0" xyz="-0.075 0.0   0.0"/>
+      <geometry>
+        <box size="0.15 0.05 0.05"/>
+      </geometry>
+    </collision>
+    <visual>
+      <origin rpy="0 0 0" xyz="-0.075 0.0   0.0"/>
+      <geometry>
+        <box size="0.15 0.05 0.05"/>
+      </geometry>
+    </visual>
+  </link>
+  <link name="head">
+    <inertial>
+      <mass value="5.0"/>
+      <origin rpy="0 0 0" xyz="-0.1 0.0 0.0"/>
+      <inertia ixx="0.0128" ixy="0" ixz="0" iyy="0.0128" iyz="0" izz="0.0128"/>
+    </inertial>
+    <collision>
+      <origin rpy="0 0 0" xyz="-0.1 0.0   0.0"/>
+      <geometry>
+        <sphere radius="0.08"/>
+      </geometry>
+    </collision>
+    <visual>
+      <origin rpy="0 0 0" xyz="-0.1 0.0   0.0"/>
+      <geometry>
+        <sphere radius="0.08"/>
+      </geometry>
+    </visual>
+  </link>
 <!-- Boat transmissions -->
   <transmission name="tran1">
