Commit message: Added testing dir

File: boot3_description/urdf/boot.xacro (robot description, xacro)
@@ -8,5 +8,5 @@
   <!-- parameters that can be configured -->
   <xacro:include filename="$(find boot3_description)/config/param.xacro" />
-  <joint name="prism" type="prismatic">  <!-- prismatic -->
+  <joint name="prism" type="prismatic">
     <parent link="world"/>
     <child link="l1"/>
@@ -88,5 +88,5 @@
     <limit effort="101.0" lower="-0.4" upper="0.4" velocity="1.0"/>
   </joint>
-  <joint name="sliding" type="prismatic">   <!-- prismatic -->
+  <joint name="sliding" type="fixed">
     <parent link="skiff"/>
     <child link="seat"/>
@@ -150,6 +150,5 @@
     <axis xyz="0 0 1" />
     <dynamics damping="0.005" />
-    <!--    <limit effort="101.0" lower="-1.5" upper="0.5" velocity="1.0"/> -->
-    <limit effort="101.0" lower="-0.1" upper="0.1" velocity="1.0"/>
+    <limit effort="101.0" lower="-1.5" upper="0.5" velocity="1.0"/>
   </joint>
   <link name="left_shoulder_xx_link">
@@ -166,5 +165,5 @@
     </visual>
   </link>
-  <joint name="shoulder_iets" type="revolute" >
+  <joint name="shoulder_psi_l" type="revolute" >
     <parent link="left_shoulder_xx_link" />
     <child link="left_shoulder_psi_link" />
@@ -172,6 +171,5 @@
     <axis xyz="1 0 0" />
     <dynamics damping="0.005" />
-<!--    <limit effort="101.0" lower="-1.5" upper="1.5" velocity="1.0"/> -->
-    <limit effort="101.0" lower="-0.2" upper="0.2" velocity="1.0"/>
+    <limit effort="101.0" lower="-1.5" upper="1.5" velocity="1.0"/>
   </joint>
   <link name="left_shoulder_psi_link">
@@ -194,15 +192,35 @@
     <axis xyz="0 1 0" />
     <dynamics damping="0.005" />
-<!--    <limit effort="101.0" lower="-2.0" upper="1.0" velocity="1.0"/> -->
-    <limit effort="101.0" lower="-0.2" upper="0.2" velocity="1.0"/>
-  </joint>
-  <!-- 2D joint right shoulder -->
+    <limit effort="101.0" lower="-2.0" upper="1.0" velocity="1.0"/>
+  </joint>
+  <!-- 3D joint right shoulder -->
   <joint name="shoulder_r" type="revolute" >
     <parent link="shoulder_link" />
+    <child link="right_shoulder_xx_link" />
+    <origin rpy="0.0 ${pi}  -0.0" xyz="0.0 -0.2   0.0"/>
+    <axis xyz="0 0 1" />
+    <dynamics damping="0.005" />
+    <limit effort="101.0" lower="-1.0" upper="0.5" velocity="1.0"/>
+  </joint>
+  <link name="right_shoulder_xx_link">
+    <inertial>
+      <mass value="0.01"/>
+      <origin rpy="0 0 0" xyz="0 0.0 0.0"/>
+      <inertia ixx="0.000000167" ixy="0" ixz="0" iyy="0.000000167" iyz="0" izz="0.000000167"/>
+    </inertial>
+    <visual>
+      <origin rpy="0 0 0" xyz="0.0 0.0 0.0"/>
+      <geometry>
+        <box size="0.01 0.01 0.01"/>
+      </geometry>
+    </visual>
+  </link>
+  <joint name="shoulder_psi_r" type="revolute" >
+    <parent link="right_shoulder_xx_link" />
     <child link="right_shoulder_psi_link" />
-    <origin rpy="0.0 ${pi}  0.0" xyz="0.0 -0.2   0.0"/>
-    <axis xyz="0 0 1" />
-    <dynamics damping="0.5" />
-    <limit effort="101.0" lower="-1.0" upper="0.5" velocity="1.0"/>
+    <origin rpy="2.47 0.0 0.0" xyz="0.0 0.0   0.0"/>
+    <axis xyz="1 0 0" />
+    <dynamics damping="0.005" />
+    <limit effort="101.0" lower="-1.5" upper="1.5" velocity="1.0"/>
   </joint>
   <link name="right_shoulder_psi_link">
@@ -222,4 +240,5 @@
     <parent link="right_shoulder_psi_link"/>
     <child link="arm_r_upper"/>
+    <origin rpy="${pi} -0.62 0" xyz="0 0.0 0.0"/>
     <axis xyz="0 1 0" />
     <dynamics damping="0.5" />
@@ -257,45 +276,45 @@
   </joint>
   <!-- hoe kom ik aan de andere kant van arm_lower_1 en 2 ?  -->
-  <joint name="dummy_1" type="fixed">
+  <joint name="Ldummy_1" type="fixed">
     <parent link="arm_l_lower_1"/>
-    <child link="dummy_link_1"/>
+    <child link="Ldummy_link_1"/>
     <origin rpy="0 0 0.0" xyz="-0.2 0.0 0.0"/>
     <dynamics damping="0.005" />
     <limit effort="101.0" lower="-1.0" upper="1.0" velocity="1.0"/>
   </joint>
-  <link name="dummy_link_1">
-    <inertial>
-      <mass value="0.01"/>
-      <origin rpy="0 0 0" xyz="0 0.0 0.0"/>
-      <inertia ixx="0.000000167" ixy="0" ixz="0" iyy="0.000000167" iyz="0" izz="0.000000167"/>
-    </inertial>
-    <visual>
-      <origin rpy="0 0 0" xyz="0.0 0.0 0.0"/>
-      <geometry>
-        <box size="0.01 0.01 0.01"/>
-      </geometry>
-    </visual>
-  </link>
-  <joint name="dummy_2" type="fixed">
+  <link name="Ldummy_link_1">
+    <inertial>
+      <mass value="0.01"/>
+      <origin rpy="0 0 0" xyz="0 0.0 0.0"/>
+      <inertia ixx="0.000000167" ixy="0" ixz="0" iyy="0.000000167" iyz="0" izz="0.000000167"/>
+    </inertial>
+    <visual>
+      <origin rpy="0 0 0" xyz="0.0 0.0 0.0"/>
+      <geometry>
+        <box size="0.01 0.01 0.01"/>
+      </geometry>
+    </visual>
+  </link>
+  <joint name="Ldummy_2" type="fixed">
     <parent link="arm_l_lower_2"/>
-    <child link="dummy_link_2"/>
+    <child link="Ldummy_link_2"/>
     <origin rpy="${pi/2} ${pi}  0.0" xyz="-0.15 0.0 0.0"/>
     <dynamics damping="0.005" />
     <limit effort="101.0" lower="-1.0" upper="1.0" velocity="1.0"/>
   </joint>
-  <link name="dummy_link_2">
-    <inertial>
-      <mass value="0.01"/>
-      <origin rpy="0 0 0" xyz="0 0.0 0.0"/>
-      <inertia ixx="0.000000167" ixy="0" ixz="0" iyy="0.000000167" iyz="0" izz="0.000000167"/>
-    </inertial>
-    <visual>
-      <origin rpy="0 0 0" xyz="0.0 0.0 0.0"/>
-      <geometry>
-        <box size="0.01 0.01 0.01"/>
-      </geometry>
-    </visual>
-  </link>
-  <!-- 3D handle joint -->
+  <link name="Ldummy_link_2">
+    <inertial>
+      <mass value="0.01"/>
+      <origin rpy="0 0 0" xyz="0 0.0 0.0"/>
+      <inertia ixx="0.000000167" ixy="0" ixz="0" iyy="0.000000167" iyz="0" izz="0.000000167"/>
+    </inertial>
+    <visual>
+      <origin rpy="0 0 0" xyz="0.0 0.0 0.0"/>
+      <geometry>
+        <box size="0.01 0.01 0.01"/>
+      </geometry>
+    </visual>
+  </link>
+  <!-- 3D handle joint left -->
   <joint name="handle_left_j1" type="revolute">
     <parent link="starboard_oar_l"/>
@@ -304,5 +323,5 @@
     <dynamics damping="0.005" />
     <axis xyz="1 0 0"/>
-    <limit effort="101.0" lower="-0.2" upper="0.2" velocity="1.0"/>
+    <limit effort="101.0" lower="-1" upper="1" velocity="1.0"/>
   </joint>
   <link name="handle_left_l1">
@@ -325,5 +344,5 @@
     <dynamics damping="0.005" />
     <axis xyz="0  0 1"/>
-    <limit effort="101.0" lower="-0.2" upper="0.2" velocity="1.0"/>
+    <limit effort="101.0" lower="-1" upper="1" velocity="1.0"/>
   </joint>
   <link name="handle_left_l2">
@@ -346,5 +365,127 @@
     <dynamics damping="0.005" />
     <axis xyz="0 1 0"/>
-    <limit effort="101.0" lower="-0.2" upper="0.2" velocity="1.0"/>
+    <limit effort="101.0" lower="-1" upper="1" velocity="1.0"/>
+  </joint>
+  <!-- 2D joint right elbow -->
+  <joint name="RElbowTheta" type="revolute" >
+    <parent link="arm_r_upper"/>
+    <child link="right_elbow_psi_link"/>
+    <origin rpy="0.0 -${pi+1.9 }  0.0" xyz="0.35 0.0  0.0"/>
+    <axis xyz="0 1 0" />
+    <dynamics damping="0.5" />
+    <limit effort="101.0" lower="-2.0" upper="1.0" velocity="1.0"/>
+  </joint>
+  <link name="right_elbow_psi_link">
+    <inertial>
+      <mass value="0.01"/>
+      <origin rpy="0 0 0" xyz="0 0.0 0.0"/>
+      <inertia ixx="0.000000167" ixy="0" ixz="0" iyy="0.000000167" iyz="0" izz="0.000000167"/>
+    </inertial>
+    <visual>
+      <origin rpy="0 0 0" xyz="0.0 0.0 0.0"/>
+      <geometry>
+        <box size="0.01 0.01 0.01"/>
+      </geometry>
+    </visual>
+  </link>
+  <joint name="elbow_right" type="revolute">
+    <parent link="right_elbow_psi_link"/>
+    <child link="arm_r_lower_1"/>
+    <origin rpy="0 0 -0.127" xyz="0 0.0 0.0"/>
+    <dynamics damping="0.5" />
+    <axis xyz="0 0 1"/>
+    <limit effort="101.0" lower="-1.0" upper="1.0" velocity="1.0"/>
+  </joint>
+  <!-- hoe kom ik aan de andere kant van arm_lower_1 en 2 ?  -->
+  <joint name="Rdummy_1" type="fixed">
+    <parent link="arm_r_lower_1"/>
+    <child link="Rdummy_link_1"/>
+    <origin rpy="0 0 0.0" xyz="-0.2 0.0 0.0"/>
+    <dynamics damping="0.005" />
+    <limit effort="101.0" lower="-1.0" upper="1.0" velocity="1.0"/>
+  </joint>
+  <link name="Rdummy_link_1">
+    <inertial>
+      <mass value="0.01"/>
+      <origin rpy="0 0 0" xyz="0 0.0 0.0"/>
+      <inertia ixx="0.000000167" ixy="0" ixz="0" iyy="0.000000167" iyz="0" izz="0.000000167"/>
+    </inertial>
+    <visual>
+      <origin rpy="0 0 0" xyz="0.0 0.0 0.0"/>
+      <geometry>
+        <box size="0.01 0.01 0.01"/>
+      </geometry>
+    </visual>
+  </link>
+  <joint name="Rdummy_2" type="fixed">
+    <parent link="arm_r_lower_2"/>
+    <child link="Rdummy_link_2"/>
+    <origin rpy="${pi/2} ${pi}  0.0" xyz="-0.15 0.0 0.0"/>
+    <dynamics damping="0.005" />
+    <limit effort="101.0" lower="-1.0" upper="1.0" velocity="1.0"/>
+  </joint>
+  <link name="Rdummy_link_2">
+    <inertial>
+      <mass value="0.01"/>
+      <origin rpy="0 0 0" xyz="0 0.0 0.0"/>
+      <inertia ixx="0.000000167" ixy="0" ixz="0" iyy="0.000000167" iyz="0" izz="0.000000167"/>
+    </inertial>
+    <visual>
+      <origin rpy="0 0 0" xyz="0.0 0.0 0.0"/>
+      <geometry>
+        <box size="0.01 0.01 0.01"/>
+      </geometry>
+    </visual>
+  </link>
+  <!-- 3D handle joint right-->
+  <joint name="handle_right_j1" type="revolute">
+    <parent link="port_oar_l"/>
+    <child link="handle_right_l1"/>
+    <origin rpy="-0.23 0 ${pi/2}" xyz="0 0.0 -${inner}"/>
+    <dynamics damping="0.005" />
+    <axis xyz="-1 0 0"/>
+    <limit effort="101.0" lower="-1" upper="1" velocity="1.0"/>
+  </joint>
+  <link name="handle_right_l1">
+    <inertial>
+      <mass value="0.01"/>
+      <origin rpy="0 0 0" xyz="0 0.0 0.0"/>
+      <inertia ixx="0.000000167" ixy="0" ixz="0" iyy="0.000000167" iyz="0" izz="0.000000167"/>
+    </inertial>
+    <visual>
+      <origin rpy="0 0 0" xyz="0.0 0.0 0.0"/>
+      <geometry>
+        <box size="0.01 0.01 0.01"/>
+      </geometry>
+    </visual>
+  </link>
+  <joint name="handle_right_j2" type="revolute">
+    <parent link="handle_right_l1"/>
+    <child link="handle_right_l2"/>
+    <origin rpy="0 0 -0.02" xyz="0 0.0 0.0"/>
+    <dynamics damping="0.005" />
+    <axis xyz="0  0 1"/>
+    <limit effort="101.0" lower="-1" upper="1" velocity="1.0"/>
+  </joint>
+  <link name="handle_right_l2">
+    <inertial>
+      <mass value="0.01"/>
+      <origin rpy="0 0 0" xyz="0 0.0 0.0"/>
+      <inertia ixx="0.000000167" ixy="0" ixz="0" iyy="0.000000167" iyz="0" izz="0.000000167"/>
+    </inertial>
+    <visual>
+      <origin rpy="0 0 0" xyz="0.0 0.0 0.0"/>
+      <geometry>
+        <box size="0.01 0.01 0.01"/>
+      </geometry>
+    </visual>
+  </link>
+  <joint name="handle_right_j3" type="revolute">
+    <parent link="handle_right_l2"/>
+    <child link="arm_r_lower_2"/>
+    <origin rpy="${pi} 0.1 0" xyz="0 0.0 0.0"/>
+    <dynamics damping="0.005" />
+    <axis xyz="0 1 0"/>
+    <limit effort="101.0" lower="-1" upper="1" velocity="1.0"/>
   </joint>
   <joint name="head_joint" type="fixed">
@@ -748,4 +889,43 @@
     </visual>
   </link>
+  <!-- lower arm in two to create a kinematic loop in gazebo -->
+  <link name="arm_r_lower_1">
+    <inertial>
+      <mass value="1.0"/>
+      <origin rpy="0 0 0" xyz="-0.1 0.0 0.0"/>
+      <inertia ixx="0.0004" ixy="0" ixz="0" iyy="0.0035" iyz="0" izz="0.0035"/>
+    </inertial>
+    <collision>
+      <origin rpy="0 0 0" xyz="-0.1 0.0   0.0"/>
+      <geometry>
+        <box size="0.20 0.05 0.05"/>
+      </geometry>
+    </collision>
+    <visual>
+      <origin rpy="0 0 0" xyz="-0.1 0.0   0.0"/>
+      <geometry>
+        <box size="0.20 0.05 0.05"/>
+      </geometry>
+    </visual>
+  </link>
+  <link name="arm_r_lower_2">
+    <inertial>
+      <mass value="1.0"/>
+      <origin rpy="0 0 0" xyz="-0.075 0.0 0.0"/>
+      <inertia ixx="0.004" ixy="0" ixz="0" iyy="0.002" iyz="0" izz="0.002"/>
+    </inertial>
+    <collision>
+      <origin rpy="0 0 0" xyz="-0.075 0.0   0.0"/>
+      <geometry>
+        <box size="0.15 0.05 0.05"/>
+      </geometry>
+    </collision>
+    <visual>
+      <origin rpy="0 0 0" xyz="-0.075 0.0   0.0"/>
+      <geometry>
+        <box size="0.15 0.05 0.05"/>
+      </geometry>
+    </visual>
+  </link>
   <link name="head">
     <inertial>
@@ -870,5 +1050,5 @@
   <transmission name="tran12">
     <type>transmission_interface/SimpleTransmission</type>
-    <joint name="shoulder_iets">
+    <joint name="shoulder_psi_l">
       <hardwareInterface>hardware_interface/EffortJointInterface</hardwareInterface>
     </joint>
@@ -886,3 +1066,12 @@
     </actuator>
   </transmission>
+  <transmission name="tran14">
+    <type>transmission_interface/SimpleTransmission</type>
+    <joint name="shoulder_psi_r">
+      <hardwareInterface>hardware_interface/EffortJointInterface</hardwareInterface>
+    </joint>
+    <actuator name="motor14">
+      <mechanicalReduction>1</mechanicalReduction>
+    </actuator>
+  </transmission>
 </robot>

Commit message: First complete version of boot!

File: boot3_description/urdf/boot.xacro (robot description, xacro)
@@ -88,5 +88,5 @@
     <limit effort="101.0" lower="-0.4" upper="0.4" velocity="1.0"/>
   </joint>
-  <joint name="sliding" type="fixed">
+  <joint name="sliding" type="prismatic">
     <parent link="skiff"/>
     <child link="seat"/>
@@ -186,5 +186,5 @@
     </visual>
   </link>
-  <joint name="LShoulderTheta" type="revolute" >
+  <joint name="shoulder_theta_l" type="revolute" >
     <parent link="left_shoulder_psi_link"/>
     <child link="arm_l_upper"/>
@@ -237,5 +237,5 @@
     </visual>
   </link>
-  <joint name="RShoulderTheta" type="revolute" >
+  <joint name="shoulder_theta_r" type="revolute" >
     <parent link="right_shoulder_psi_link"/>
     <child link="arm_r_upper"/>
@@ -246,5 +246,5 @@
   </joint>
   <!-- 2D joint left elbow -->
-  <joint name="LElbowTheta" type="revolute" >
+  <joint name="elbow_theta_l" type="revolute" >
     <parent link="arm_l_upper"/>
     <child link="left_elbow_psi_link"/>
@@ -368,5 +368,5 @@
   </joint>
   <!-- 2D joint right elbow -->
-  <joint name="RElbowTheta" type="revolute" >
+  <joint name="elbow_theta_r" type="revolute" >
     <parent link="arm_r_upper"/>
     <child link="right_elbow_psi_link"/>
@@ -1059,5 +1059,5 @@
   <transmission name="tran13">
     <type>transmission_interface/SimpleTransmission</type>
-    <joint name="LShoulderTheta">
+    <joint name="shoulder_theta_l">
       <hardwareInterface>hardware_interface/EffortJointInterface</hardwareInterface>
     </joint>
@@ -1068,8 +1068,116 @@
   <transmission name="tran14">
     <type>transmission_interface/SimpleTransmission</type>
+    <joint name="elbow_theta_l">
+      <hardwareInterface>hardware_interface/EffortJointInterface</hardwareInterface>
+    </joint>
+    <actuator name="motor14">
+      <mechanicalReduction>1</mechanicalReduction>
+    </actuator>
+  </transmission>
+  <transmission name="tran15">
+    <type>transmission_interface/SimpleTransmission</type>
+    <joint name="elbow_left">
+      <hardwareInterface>hardware_interface/EffortJointInterface</hardwareInterface>
+    </joint>
+    <actuator name="motor15">
+      <mechanicalReduction>1</mechanicalReduction>
+    </actuator>
+  </transmission>
+  <transmission name="tran16">
+    <type>transmission_interface/SimpleTransmission</type>
+    <joint name="handle_left_j1">
+      <hardwareInterface>hardware_interface/EffortJointInterface</hardwareInterface>
+    </joint>
+    <actuator name="motor16">
+      <mechanicalReduction>1</mechanicalReduction>
+    </actuator>
+  </transmission>
+  <transmission name="tran17">
+    <type>transmission_interface/SimpleTransmission</type>
+    <joint name="handle_left_j2">
+      <hardwareInterface>hardware_interface/EffortJointInterface</hardwareInterface>
+    </joint>
+    <actuator name="motor17">
+      <mechanicalReduction>1</mechanicalReduction>
+    </actuator>
+  </transmission>
+  <transmission name="tran18">
+    <type>transmission_interface/SimpleTransmission</type>
+    <joint name="handle_left_j3">
+      <hardwareInterface>hardware_interface/EffortJointInterface</hardwareInterface>
+    </joint>
+    <actuator name="motor18">
+      <mechanicalReduction>1</mechanicalReduction>
+    </actuator>
+  </transmission>
+  <transmission name="tran19">
+    <type>transmission_interface/SimpleTransmission</type>
+    <joint name="shoulder_r">
+      <hardwareInterface>hardware_interface/EffortJointInterface</hardwareInterface>
+    </joint>
+    <actuator name="motor19">
+      <mechanicalReduction>1</mechanicalReduction>
+    </actuator>
+  </transmission>
+  <transmission name="tran20">
+    <type>transmission_interface/SimpleTransmission</type>
     <joint name="shoulder_psi_r">
       <hardwareInterface>hardware_interface/EffortJointInterface</hardwareInterface>
     </joint>
-    <actuator name="motor14">
+    <actuator name="motor20">
+      <mechanicalReduction>1</mechanicalReduction>
+    </actuator>
+  </transmission>
+  <transmission name="tran21">
+    <type>transmission_interface/SimpleTransmission</type>
+    <joint name="shoulder_theta_r">
+      <hardwareInterface>hardware_interface/EffortJointInterface</hardwareInterface>
+    </joint>
+    <actuator name="motor21">
+      <mechanicalReduction>1</mechanicalReduction>
+    </actuator>
+  </transmission>
+  <transmission name="tran22">
+    <type>transmission_interface/SimpleTransmission</type>
+    <joint name="elbow_theta_r">
+      <hardwareInterface>hardware_interface/EffortJointInterface</hardwareInterface>
+    </joint>
+    <actuator name="motor22">
+      <mechanicalReduction>1</mechanicalReduction>
+    </actuator>
+  </transmission>
+  <transmission name="tran23">
+    <type>transmission_interface/SimpleTransmission</type>
+    <joint name="elbow_right">
+      <hardwareInterface>hardware_interface/EffortJointInterface</hardwareInterface>
+    </joint>
+    <actuator name="motor23">
+      <mechanicalReduction>1</mechanicalReduction>
+    </actuator>
+  </transmission>
+  <transmission name="tran24">
+    <type>transmission_interface/SimpleTransmission</type>
+    <joint name="handle_right_j1">
+      <hardwareInterface>hardware_interface/EffortJointInterface</hardwareInterface>
+    </joint>
+    <actuator name="motor24">
+      <mechanicalReduction>1</mechanicalReduction>
+    </actuator>
+  </transmission>
+  <transmission name="tran25">
+    <type>transmission_interface/SimpleTransmission</type>
+    <joint name="handle_right_j2">
+      <hardwareInterface>hardware_interface/EffortJointInterface</hardwareInterface>
+    </joint>
+    <actuator name="motor25">
+      <mechanicalReduction>1</mechanicalReduction>
+    </actuator>
+  </transmission>
+  <transmission name="tran26">
+    <type>transmission_interface/SimpleTransmission</type>
+    <joint name="handle_right_j3">
+      <hardwareInterface>hardware_interface/EffortJointInterface</hardwareInterface>
+    </joint>
+    <actuator name="motor26">
       <mechanicalReduction>1</mechanicalReduction>
     </actuator>
