Commit message: corrected joints

File: boot3_description/urdf/boot.xacro (robot description, xacro)
@@ -153,5 +153,5 @@
     <parent link="starboard_oar_l"/>
     <child link="handle_left_l1"/>
-    <origin rpy="0.209 0 ${pi/2}" xyz="0 0.0 ${inner}"/>
+    <origin rpy="0.13 0 ${pi/2}" xyz="0 0.0 ${inner}"/>
     <dynamics damping="0.005" />
     <axis xyz="1 0 0"/>
@@ -174,5 +174,5 @@
     <parent link="handle_left_l1"/>
     <child link="handle_left_l2"/>
-    <origin rpy="0 0 0.06" xyz="0 0.0 0.0"/>
+    <origin rpy="0 0 0.0" xyz="0 0.0 0.0"/>
     <dynamics damping="0.005" />
     <axis xyz="0  0 1"/>
@@ -195,5 +195,5 @@
     <parent link="handle_left_l2"/>
     <child link="arm_l_lower"/>
-    <origin rpy="0 -0.16 0" xyz="0 0.0 0.0"/>
+    <origin rpy="0 0.04 0" xyz="0 0.0 0.0"/>
     <dynamics damping="0.005" />
     <axis xyz="0 1 0"/>
@@ -246,5 +246,5 @@
     <parent link="left_elbow_theta_link"/>
     <child link="arm_l_upper"/>
-    <origin rpy="0.0 0.0  0.0" xyz="-0.0 0.0  0.0"/>
+    <origin rpy="1.0 0.0  0.0" xyz="-0.0 0.0  0.0"/>
     <axis xyz="1 0 0" />
     <dynamics damping="0.5" />
@@ -255,5 +255,5 @@
     <parent link="arm_l_upper"/>
     <child link="left_shoulder_psi_link"/>
-    <origin rpy="0 0.0 0" xyz="-0.35 0.0 0.0"/>
+    <origin rpy="0 0.37 0" xyz="-0.35 0.0 0.0"/>
     <axis xyz="0 1 0" />
     <dynamics damping="0.005" />
@@ -297,5 +297,5 @@
     <parent link="left_shoulder_xx_link" />
     <child link="shoulder_left" />
-    <origin rpy="0.0 0.0 0.0" xyz="0.0 0.0   0.0"/>
+    <origin rpy="0.0 0.0 0.16" xyz="0.0 0.0   0.0"/>
     <axis xyz="0 0 1" />
     <dynamics damping="0.005" />
@@ -305,5 +305,5 @@
     <parent link="shoulder_left"/>
     <child link="Ldummy_link_2"/>
-    <origin rpy="${pi/2} ${pi}  0.0" xyz="0.0 0.0 0.0"/>
+    <origin rpy="0 0 ${pi} " xyz="0.0 0.1 0.0"/>
     <dynamics damping="0.005" />
     <limit effort="101.0" lower="-1.0" upper="1.0" velocity="1.0"/>
@@ -326,5 +326,5 @@
     <parent link="shoulder_link"/>
     <child link="Ldummy_link_1"/>
-    <origin rpy="0 0 0.0" xyz="0.2 0.0 0.0"/>
+    <origin rpy="0 0 0.0" xyz="0.0 0.1 0.0"/>
     <dynamics damping="0.005" />
     <limit effort="101.0" lower="-1.0" upper="1.0" velocity="1.0"/>
@@ -348,5 +348,5 @@
     <parent link="port_oar_l"/>
     <child link="handle_right_l1"/>
-    <origin rpy="-0.23 0 ${pi/2}" xyz="0 0.0 -${inner}"/>
+    <origin rpy="-0.07 0 ${pi/2}" xyz="0 0.0 -${inner}"/>
     <dynamics damping="0.005" />
     <axis xyz="-1 0 0"/>
@@ -369,5 +369,5 @@
     <parent link="handle_right_l1"/>
     <child link="handle_right_l2"/>
-    <origin rpy="0 0 -0.02" xyz="0 0.0 0.0"/>
+    <origin rpy="0 0 -0.08" xyz="0 0.0 0.0"/>
     <dynamics damping="0.005" />
     <axis xyz="0  0 1"/>
@@ -399,5 +399,5 @@
     <parent link="arm_r_lower"/>
     <child link="right_elbow_psi_link"/>
-    <origin rpy="0 0 -0.127" xyz="-0.4 0.0 0.0"/>
+    <origin rpy="${pi} 0 ${pi+1.8}" xyz="-0.4 0.0 0.0"/>
     <dynamics damping="0.5" />
     <axis xyz="0 0 1"/>
@@ -420,5 +420,5 @@
     <parent link="right_elbow_psi_link"/>
     <child link="right_elbow_theta_link"/>
-    <origin rpy="0.0 -${pi+1.9 }  0.0" xyz="0.0 0.0  0.0"/>
+    <origin rpy="0.0 -0.02  0.0" xyz="0.0 0.0  0.0"/>
     <axis xyz="0 1 0" />
     <dynamics damping="0.5" />
@@ -441,8 +441,8 @@
     <parent link="right_elbow_theta_link"/>
     <child link="arm_r_upper"/>
-    <origin rpy="0.0 -${pi+1.9 }  0.0" xyz="0.0 0.0  0.0"/>
+    <origin rpy="0.7 0.0  0.0" xyz="0.0 0.0  0.0"/>
     <axis xyz="1 0 0" />
     <dynamics damping="0.5" />
-    <limit effort="101.0" lower="-2.0" upper="1.0" velocity="1.0"/>
+    <limit effort="101.0" lower="-1.0" upper="2.0" velocity="1.0"/>
   </joint>
   <!-- 3D joint right shoulder -->
@@ -450,5 +450,5 @@
     <parent link="arm_r_upper"/>
     <child link="right_shoulder_psi_link"/>
-    <origin rpy="${pi} -0.62 0" xyz="0 0.0 0.0"/>
+    <origin rpy="${pi} -0.62 0" xyz="0.35 0.0 0.0"/>
     <axis xyz="0 1 0" />
     <dynamics damping="0.5" />
@@ -471,5 +471,5 @@
     <parent link="right_shoulder_psi_link" />
     <child link="right_shoulder_xx_link" />
-    <origin rpy="2.47 0.0 0.0" xyz="0.0 0.0   0.0"/>
+    <origin rpy="3.42 0.0 0.0" xyz="0.0 0.0   0.0"/>
     <axis xyz="1 0 0" />
     <dynamics damping="0.005" />
@@ -492,5 +492,5 @@
     <parent link="right_shoulder_xx_link" />
     <child link="shoulder_right" />
-    <origin rpy="0.0 ${pi}  -0.0" xyz="0.0 -0.1   0.0"/>
+    <origin rpy="0.0 ${pi}  -0.0" xyz="0.0 -0.0   0.0"/>
     <axis xyz="0 0 1" />
     <dynamics damping="0.005" />
@@ -500,5 +500,5 @@
     <parent link="shoulder_right"/>
     <child link="Rdummy_link_2"/>
-    <origin rpy="${pi/2} ${pi}  0.0" xyz="-0.15 0.0 0.0"/>
+    <origin rpy="${pi} -${pi/2}  0.0" xyz="0.0 -0.1 0.0"/>
     <dynamics damping="0.005" />
     <limit effort="101.0" lower="-1.0" upper="1.0" velocity="1.0"/>
@@ -521,5 +521,5 @@
     <parent link="shoulder_link"/>
     <child link="Rdummy_link_1"/>
-    <origin rpy="0 0 0.0" xyz="-0.2 0.0 0.0"/>
+    <origin rpy="0 0 0.0" xyz="0.0 -0.1 0.0"/>
     <dynamics damping="0.005" />
     <limit effort="101.0" lower="-1.0" upper="1.0" velocity="1.0"/>
@@ -889,5 +889,5 @@
     </collision>
     <visual>
-      <origin rpy="0 0 0" xyz="0.0 -0.2   0.0"/>
+      <origin rpy="0 0 0" xyz="0.0 -0.05   0.0"/>
       <geometry>
         <box size="0.05 0.1 0.05"/>

Commit message: tweaked model

File: boot3_description/urdf/boot.xacro (robot description, xacro)
@@ -275,5 +275,5 @@
     <axis xyz="0 1 0" />
     <dynamics damping="0.005" />
-    <limit effort="101.0" lower="-2.0" upper="1.0" velocity="1.0"/>
+    <limit effort="101.0" lower="-1.0" upper="1.0" velocity="1.0"/>
   </joint>
   <link name="left_shoulder_psi_link">
@@ -296,5 +296,5 @@
     <axis xyz="1 0 0" />
     <dynamics damping="0.005" />
-    <limit effort="101.0" lower="-1.5" upper="1.5" velocity="1.0"/>
+    <limit effort="101.0" lower="-1.0" upper="1.0" velocity="1.0"/>
   </joint>
   <link name="left_shoulder_xx_link">
@@ -317,5 +317,5 @@
     <axis xyz="0 0 1" />
     <dynamics damping="0.005" />
-    <limit effort="101.0" lower="-1.5" upper="1.5" velocity="1.0"/>
+    <limit effort="101.0" lower="-1.0" upper="1.0" velocity="1.0"/>
   </joint>
   <joint name="Ldummy_2" type="fixed">
@@ -470,5 +470,5 @@
     <axis xyz="0 -1 0" />
     <dynamics damping="0.5" />
-    <limit effort="101.0" lower="-1.5" upper="1.0" velocity="1.0"/>
+    <limit effort="101.0" lower="-1.0" upper="1.0" velocity="1.0"/>
   </joint>
   <link name="right_shoulder_psi_link">
@@ -491,5 +491,5 @@
     <axis xyz="1 0 0" />
     <dynamics damping="0.005" />
-    <limit effort="101.0" lower="-1.5" upper="1.5" velocity="1.0"/>
+    <limit effort="101.0" lower="-1.0" upper="1.0" velocity="1.0"/>
   </joint>
   <link name="right_shoulder_xx_link">
@@ -512,5 +512,5 @@
     <axis xyz="0 0 1" />
     <dynamics damping="0.005" />
-    <limit effort="101.0" lower="-1.0" upper="0.5" velocity="1.0"/>
+    <limit effort="101.0" lower="-1.0" upper="1.0" velocity="1.0"/>
   </joint>
   <joint name="Rdummy_2" type="fixed">
@@ -877,9 +877,9 @@
     <inertial>
       <mass value="1.0"/>
-      <origin rpy="0 0 0" xyz="0.0 -0.2 0.0"/>
+      <origin rpy="0 0 0" xyz="0.0 0.05 0.0"/>
       <inertia ixx="0.013" ixy="0" ixz="0" iyy="0.0004" iyz="0" izz="0.013"/>
     </inertial>
     <collision>
-      <origin rpy="0 0 0" xyz="0.0  -0.2   0.0"/>
+      <origin rpy="0 0 0" xyz="0.0  0.05   0.0"/>
       <geometry>
         <box size="0.05 0.1 0.05"/>
@@ -896,9 +896,9 @@
     <inertial>
       <mass value="1.0"/>
-      <origin rpy="0 0 0" xyz="0.0 -0.2 0.0"/>
+      <origin rpy="0 0 0" xyz="0.0 -0.05 0.0"/>
       <inertia ixx="0.013" ixy="0" ixz="0" iyy="0.0004" iyz="0" izz="0.013"/>
     </inertial>
     <collision>
-      <origin rpy="0 0 0" xyz="0.0  -0.2   0.0"/>
+      <origin rpy="0 0 0" xyz="0.0  -0.05   0.0"/>
       <geometry>
         <box size="0.05 0.1 0.05"/>

File: testing/crash_boot.urdf (robot description, URDF)
Before this commit: robot myboat, 9 links, 8 joints
Links:
- link back_low: geometry visual box size=0.3 0.1 0.05

File: testing/crash_boot.xacro (robot description, xacro)
@@ -19,6 +19,5 @@
     <origin rpy="0 0 0" xyz="0.15 0.0   0.0"/>
     <geometry>
-      <mesh filename="model://myboot/meshes/hokuyo.dae" scale="10.0004 10.0004 10.0004"/>
-      <!--      <box size="0.3 0.1 0.05"/> -->
+      <box size="0.3 0.1 0.05"/>
     </geometry>
   </visual>
@@ -67,5 +66,5 @@
   <axis xyz="0 0 1" />
   <dynamics damping="0.5"  friction="0.1"/>
-  <limit effort="100.0" lower="-1.5" upper="0.5" velocity="1.0"/>
+  <limit effort="100.0" lower="-0.5" upper="0.5" velocity="1.0"/>
 </joint>
 <link name="left_shoulder_xx_link">
@@ -106,5 +105,5 @@
   <axis xyz="0 1 0" />
   <dynamics damping="0.5" friction="0.1" />
-  <limit effort="100.0" lower="-2.0" upper="1.0" velocity="1.0"/>
+  <limit effort="100.0" lower="-0.5" upper="0.5" velocity="1.0"/>
 </joint>
 <link name="arm_l_upper">

Commit message: small change

File: boot3_description/urdf/boot.xacro (robot description, xacro)
@@ -224,5 +224,5 @@
     <dynamics damping="0.5" />
     <axis xyz="0 0 1"/>
-    <limit effort="101.0" lower="-1.0" upper="1.0" velocity="1.0"/>
+    <limit effort="101.0" lower="-1.0" upper="2.0" velocity="1.0"/>
   </joint>
   <link name="left_elbow_psi_link">
@@ -973,5 +973,5 @@
       <mass value="1.0"/>
       <origin rpy="0 0 0" xyz="-0.2 0.0 0.0"/>
-      <inertia ixx="0.0004" ixy="0" ixz="0" iyy="0.0035" iyz="0" izz="0.0035"/>
+      <inertia ixx="0.00041" ixy="0" ixz="0" iyy="0.0135" iyz="0" izz="0.0135"/>
     </inertial>
     <collision>
@@ -1135,4 +1135,13 @@
     </actuator>
   </transmission>
+  <transmission name="tran28">
+    <type>transmission_interface/SimpleTransmission</type>
+    <joint name="elbow_xx_l">
+      <hardwareInterface>hardware_interface/EffortJointInterface</hardwareInterface>
+    </joint>
+    <actuator name="motor28">
+      <mechanicalReduction>1</mechanicalReduction>
+    </actuator>
+  </transmission>
   <transmission name="tran15">
     <type>transmission_interface/SimpleTransmission</type>
@@ -1207,4 +1216,13 @@
     </actuator>
   </transmission>
+  <transmission name="tran27">
+    <type>transmission_interface/SimpleTransmission</type>
+    <joint name="elbow_xx_r">
+      <hardwareInterface>hardware_interface/EffortJointInterface</hardwareInterface>
+    </joint>
+    <actuator name="motor27">
+      <mechanicalReduction>1</mechanicalReduction>
+    </actuator>
+  </transmission>
   <transmission name="tran23">
     <type>transmission_interface/SimpleTransmission</type>
