Commit message: Changed kinematic chain in boot4

File: boot4_description/config/param.xacro (robot description, xacro)
@@ -7,5 +7,5 @@
 <xacro:property name="span" value="1.6"/>
 <!-- oar -->
-<xacro:property name="inner" value="0.87"/>
+<xacro:property name="inner" value="0.87"/>  <!-- length inclusive 0.1 meter handle -->
 <xacro:property name="outer" value="2.00"/>
 <!--  rower -->
@@ -20,23 +20,23 @@
 <xacro:property name="starboard_oar" value="-0.1458"/>
 <xacro:property name="port_oar" value="0.1359"/>
-<xacro:property name="hip2" value="0.329"/>
-<xacro:property name="back_lh" value="0.011"/>
-<xacro:property name="handle_left_j1" value="0.1425"/>
-<xacro:property name="handle_left_j2" value="0.0807"/>
-<xacro:property name="handle_left_j3" value="-0.0503"/>
-<xacro:property name="elbow_left" value="-1.9207"/>
-<xacro:property name="elbow_theta_l" value="0.0003"/>
-<xacro:property name="elbow_xx_l" value="0.9796"/>
-<xacro:property name="shoulder_theta_l" value="0.5435"/>
-<xacro:property name="shoulder_psi_l" value="-0.0182"/>
-<xacro:property name="shoulder_l" value="0.1516"/>
-<xacro:property name="handle_right_j1" value="0.0496"/>
-<xacro:property name="handle_right_j2" value="0.0074"/>
-<xacro:property name="handle_right_j3" value="0.0084"/>
-<xacro:property name="elbow_right" value="1.2894"/>
-<xacro:property name="elbow_theta_r" value="0.0288"/>
-<xacro:property name="elbow_xx_r" value="-0.2775"/>
-<xacro:property name="shoulder_theta_r" value="-.7384"/>
-<xacro:property name="shoulder_psi_r" value="3.7462"/>
-<xacro:property name="shoulder_r" value="0.5698"/>
+<xacro:property name="hip2" value="-0.329"/>
+<xacro:property name="back_lh" value="0.0110"/>
+<xacro:property name="shoulder_l" value="-0.4209"/>
+<xacro:property name="shoulder_psi_l" value="0.1234"/>
+<xacro:property name="shoulder_theta_l" value="-0.3724"/>
+<xacro:property name="elbow_xx_l" value="0.1150"/>
+<xacro:property name="elbow_theta_l" value="0.1356"/>
+<xacro:property name="elbow_left" value="0.2445"/>
+<xacro:property name="handle_left_j3" value="0.0181"/>
+<xacro:property name="handle_left_j2" value="-0.0254"/>
+<xacro:property name="handle_left_j1" value="-0.0396"/>
+<xacro:property name="shoulder_r" value="-0.4208"/>
+<xacro:property name="shoulder_psi_r" value="0.1086"/>
+<xacro:property name="shoulder_theta_r" value="-0.3731"/>
+<xacro:property name="elbow_xx_r" value="0.0271"/>
+<xacro:property name="elbow_theta_r" value="0.1332"/>
+<xacro:property name="elbow_right" value="0.1927"/>
+<xacro:property name="handle_right_j3" value="0.0001"/>
+<xacro:property name="handle_right_j2" value="-0.0074"/>
+<xacro:property name="handle_right_j1" value="-0.1168"/>
 </robot>

File: boot4_description/urdf/boot.xacro (robot description, xacro)
@@ -4,4 +4,5 @@
   <xacro:arg name="reconnectloops" default="false" />
   <xacro:if value="$(arg reconnectloops)">
+    <xacro:property name="course_type" value="fixed" />
     <xacro:property name="sliding_type" value="fixed" />
     <xacro:property name="hip2_type" value="fixed" />
@@ -12,4 +13,5 @@
   </xacro:if>
   <xacro:unless value="$(arg reconnectloops)">
+    <xacro:property name="course_type" value="prismatic" />
     <xacro:property name="sliding_type" value="prismatic" />
     <xacro:property name="hip2_type" value="revolute" />
@@ -25,16 +27,16 @@
   <!-- parameters that can be configured -->
   <xacro:include filename="$(find boot4_description)/config/param.xacro" />
-  <joint name="prism" type="prismatic">
+  <joint name="the_course" type="${course_type}">
     <parent link="world"/>
     <child link="l1"/>
-    <origin xyz="0 0 0.25" rpy="0 0 0"/>
+    <origin xyz="0 0 0.0" rpy="0 0 0"/>
     <dynamics damping="0.005" />
     <axis xyz="1 0 0"/>
-    <limit effort="101.0" lower="0" upper="1000" velocity="0.5"/>
+    <limit effort="101.0" lower="0" upper="100" velocity="0.5"/>
   </joint>
   <joint name="rev1" type="revolute">
     <parent link="l1"/>
     <child link="l2"/>
-    <origin xyz="0.0 0 -0.2" rpy="0 ${pi/2} 0"/>
+    <origin xyz="0.0 0 0.05" rpy="0 ${pi/2} 0"/>
     <dynamics damping="0.005" />
     <axis xyz="0 1 0"/>
@@ -140,5 +142,5 @@
     <parent link="seat"/>
     <child link="back_low"/>
-    <origin rpy="0  -${pi/2+hip2} 0.0" xyz="0.0 0.0   0.1"/>
+    <origin rpy="0  -${pi/2-hip2} 0.0" xyz="0.0 0.0   0.1"/>
     <dynamics damping="0.005" />
     <axis xyz="0 1 0"/>
@@ -165,10 +167,133 @@
     <origin rpy="0  0.0 0.0" xyz="0.2 0.0   0.0"/>
   </joint>
-  <!-- Left branch from starboard_oar to shoulder_left -->
+  <!-- Left branch from shoulder_link to starboard_oar -->
+  <!-- 3D joint left shoulder -->
+  <joint name="shoulder_l" type="revolute" >
+    <parent link="shoulder_link" />
+    <child link="left_shoulder_xx_link" />
+    <origin rpy="0.0 ${-shoulder_l} 0.0" xyz="0.0 0.2   0.0"/>
+    <axis xyz="0 -1 0" />
+    <dynamics damping="0.005" />
+    <limit effort="101.0" lower="-1.0" upper="1.0" velocity="1.0"/>
+  </joint>
+  <link name="left_shoulder_xx_link">
+    <inertial>
+      <mass value="0.01"/>
+      <origin rpy="0 0 0" xyz="0 0.0 0.0"/>
+      <inertia ixx="0.000000167" ixy="0" ixz="0" iyy="0.000000167" iyz="0" izz="0.000000167"/>
+    </inertial>
+    <visual>
+      <origin rpy="0 0 0" xyz="0.0 0.0 0.0"/>
+      <geometry>
+        <box size="0.01 0.01 0.01"/>
+      </geometry>
+    </visual>
+  </link>
+  <joint name="shoulder_psi_l" type="revolute" >
+    <parent link="left_shoulder_xx_link" />
+    <child link="left_shoulder_psi_link" />
+    <origin rpy="0 0.0 ${-shoulder_psi_l}" xyz="0.0 0.0   0.0"/>
+    <axis xyz="0 0 -1" />
+    <dynamics damping="0.005" />
+    <limit effort="101.0" lower="-1.0" upper="1.0" velocity="1.0"/>
+  </joint>
+  <link name="left_shoulder_psi_link">
+    <inertial>
+      <mass value="0.01"/>
+      <origin rpy="0 0 0" xyz="0 0.0 0.0"/>
+      <inertia ixx="0.000000167" ixy="0" ixz="0" iyy="0.000000167" iyz="0" izz="0.000000167"/>
+    </inertial>
+    <visual>
+      <origin rpy="0 0 0" xyz="0.0 0.0 0.0"/>
+      <geometry>
+        <box size="0.01 0.01 0.01"/>
+      </geometry>
+    </visual>
+  </link>
+  <joint name="shoulder_theta_l" type="revolute" >
+    <parent link="left_shoulder_psi_link"/>
+    <child link="arm_l_upper"/>
+    <origin rpy="${shoulder_theta_l} 0 0" xyz="0.0 0.0 0.0"/>
+    <axis xyz="1 0 0" />
+    <dynamics damping="0.005" />
+    <limit effort="101.0" lower="-1.0" upper="1.0" velocity="1.0"/>
+  </joint>
+  <!-- 3D joint left elbow -->
+  <joint name="elbow_xx_l" type="revolute" >
+    <parent link="arm_l_upper"/>
+    <child link="left_elbow_theta_link"/>
+    <origin rpy=" ${pi} ${-(elbow_xx_l+pi/2)}  0.0" xyz="-0.3 0.0  0.0"/>
+    <axis xyz="0 1 0" />
+    <dynamics damping="0.5" />
+    <limit effort="101.0" lower="-${pi/2}" upper="${pi/2}" velocity="1.0"/>
+  </joint>
+  <link name="left_elbow_theta_link">
+    <inertial>
+      <mass value="0.01"/>
+      <origin rpy="0 0 0" xyz="0 0.0 0.0"/>
+      <inertia ixx="0.000000167" ixy="0" ixz="0" iyy="0.000000167" iyz="0" izz="0.000000167"/>
+    </inertial>
+    <visual>
+      <origin rpy="0 0 0" xyz="0.0 0.0 0.0"/>
+      <geometry>
+        <box size="0.01 0.01 0.01"/>
+      </geometry>
+    </visual>
+  </link>
+  <joint name="elbow_theta_l" type="revolute" >
+    <parent link="left_elbow_theta_link"/>
+    <child link="left_elbow_psi_link"/>
+    <origin rpy="0 0.0  ${-elbow_theta_l}" xyz="-0.0 0.0  0.0"/>
+    <axis xyz="0 0 -1" />
+    <dynamics damping="0.5" />
+    <limit effort="101.0" lower="-0.7" upper="2.0" velocity="1.0"/>
+  </joint>
+  <link name="left_elbow_psi_link">
+    <inertial>
+      <mass value="0.01"/>
+      <origin rpy="0 0 0" xyz="0 0.0 0.0"/>
+      <inertia ixx="0.000000167" ixy="0" ixz="0" iyy="0.000000167" iyz="0" izz="0.000000167"/>
+    </inertial>
+    <visual>
+      <origin rpy="0 0 0" xyz="0.0 0.0 0.0"/>
+      <geometry>
+        <box size="0.01 0.01 0.01"/>
+      </geometry>
+    </visual>
+  </link>
+  <joint name="elbow_left" type="revolute">
+    <parent link="left_elbow_psi_link"/>
+    <child link="arm_l_lower"/>
+    <origin rpy="${elbow_left} 0 0" xyz="-0.0 0.0 0.0"/>
+    <dynamics damping="0.5" />
+    <axis xyz="1 0 0"/>
+    <limit effort="101.0" lower="-1.0" upper="1.0" velocity="1.0"/>
+  </joint>
   <!-- 3D handle joint left -->
-  <joint name="handle_left_j1" type="revolute">
-    <parent link="starboard_oar_l"/>
+  <joint name="handle_left_j3" type="revolute">
+    <parent link="arm_l_lower"/>
+    <child link="handle_left_l2"/>
+    <origin rpy="${pi/2} ${handle_left_j3} 0" xyz="-0.35 0.0 0.0"/>
+    <dynamics damping="0.005" />
+    <axis xyz="0 1 0"/>
+    <limit effort="101.0" lower="-1" upper="1" velocity="1.0"/>
+  </joint>
+  <link name="handle_left_l2">
+    <inertial>
+      <mass value="0.01"/>
+      <origin rpy="0 0 0" xyz="0 0.0 0.0"/>
+      <inertia ixx="0.000000167" ixy="0" ixz="0" iyy="0.000000167" iyz="0" izz="0.000000167"/>
+    </inertial>
+    <visual>
+      <origin rpy="0 0 0" xyz="0.0 0.0 0.0"/>
+      <geometry>
+        <box size="0.01 0.01 0.01"/>
+      </geometry>
+    </visual>
+  </link>
+  <joint name="handle_left_j2" type="revolute">
+    <parent link="handle_left_l2"/>
     <child link="handle_left_l1"/>
-    <origin rpy="${handle_left_j1} 0 ${pi/2}" xyz="0 0.0 ${inner}"/>
+    <origin rpy="${handle_left_j2} 0 0" xyz="0 0.0 0.0"/>
     <dynamics damping="0.005" />
     <axis xyz="1 0 0"/>
@@ -188,182 +313,182 @@
     </visual>
   </link>
-  <joint name="handle_left_j2" type="revolute">
+  <joint name="handle_left_j1" type="revolute">
     <parent link="handle_left_l1"/>
-    <child link="handle_left_l2"/>
-    <origin rpy="0 0 ${handle_left_j2}" xyz="0 0.0 0.0"/>
+    <child link="starboard_handle_l"/>
+    <origin rpy="0 0 ${handle_left_j1}" xyz="0 0.0 0"/>
     <dynamics damping="0.005" />
     <axis xyz="0 0 1"/>
     <limit effort="101.0" lower="-1" upper="1" velocity="1.0"/>
   </joint>
-  <link name="handle_left_l2">
-    <inertial>
-      <mass value="0.01"/>
-      <origin rpy="0 0 0" xyz="0 0.0 0.0"/>
-      <inertia ixx="0.000000167" ixy="0" ixz="0" iyy="0.000000167" iyz="0" izz="0.000000167"/>
-    </inertial>
-    <visual>
-      <origin rpy="0 0 0" xyz="0.0 0.0 0.0"/>
-      <geometry>
-        <box size="0.01 0.01 0.01"/>
-      </geometry>
-    </visual>
-  </link>
-  <joint name="handle_left_j3" type="revolute">
-    <parent link="handle_left_l2"/>
-    <child link="arm_l_lower"/>
-    <origin rpy="0 ${handle_left_j3} 0" xyz="0 0.0 0.0"/>
-    <dynamics damping="0.005" />
-    <axis xyz="0 1 0"/>
-    <limit effort="101.0" lower="-1" upper="1" velocity="1.0"/>
-  </joint>
-  <!-- 3D joint left elbow -->
-  <joint name="elbow_left" type="revolute">
-    <parent link="arm_l_lower"/>
-    <child link="left_elbow_psi_link"/>
-    <origin rpy="0 0 ${elbow_left}" xyz="-0.4 0.0 0.0"/>
+  <joint name="Ldummy_2" type="fixed">
+    <parent link="starboard_handle_l"/>
+    <child link="Ldummy_link_2"/>
+    <origin rpy="0 0 0 " xyz="0.0 0.0 0.075"/>
+    <dynamics damping="0.005" />
+    <limit effort="101.0" lower="-1.0" upper="1.0" velocity="1.0"/>
+  </joint>
+  <link name="Ldummy_link_2">
+    <inertial>
+      <mass value="0.01"/>
+      <origin rpy="0 0 0" xyz="0 0.0 0.0"/>
+      <inertia ixx="0.000000167" ixy="0" ixz="0" iyy="0.000000167" iyz="0" izz="0.000000167"/>
+    </inertial>
+    <visual>
+      <origin rpy="0 0 0" xyz="0.0 0.0 0.0"/>
+      <geometry>
+        <box size="0.01 0.01 0.01"/>
+      </geometry>
+    </visual>
+  </link>
+  <!-- in gazebo here the joint that closes the left loop -->
+  <link name="Ldummy_link_1">
+    <inertial>
+      <mass value="0.01"/>
+      <origin rpy="0 0 0" xyz="0 0.0 0.0"/>
+      <inertia ixx="0.000000167" ixy="0" ixz="0" iyy="0.000000167" iyz="0" izz="0.000000167"/>
+    </inertial>
+    <visual>
+      <origin rpy="0 0 0" xyz="0.0 0.0 0.0"/>
+      <geometry>
+        <box size="0.01 0.01 0.01"/>
+      </geometry>
+    </visual>
+  </link>
+  <joint name="Ldummy_1" type="fixed">
+    <parent link="starboard_oar_l"/>
+    <child link="Ldummy_link_1"/>
+    <origin rpy="0 ${pi} ${pi/2}" xyz="0 0 ${inner-0.1} "/>
+    <dynamics damping="0.005" />
+    <limit effort="101.0" lower="-1.0" upper="1.0" velocity="1.0"/>
+  </joint>
+  <!-- Right branch from shoulder_link to port_handle -->
+  <!-- 3D joint right shoulder -->
+  <joint name="shoulder_r" type="revolute" >
+    <parent link="shoulder_link"/>
+    <child link="right_shoulder_xx_link" />
+    <origin rpy="0.0 ${-shoulder_r}  0" xyz="0.0 -0.2   0.0"/>
+    <axis xyz="0 -1 0" />
+    <dynamics damping="0.005" />
+    <limit effort="101.0" lower="-1.0" upper="1.0" velocity="1.0"/>
+  </joint>
+  <link name="right_shoulder_xx_link">
+    <inertial>
+      <mass value="0.01"/>
+      <origin rpy="0 0 0" xyz="0 0.0 0.0"/>
+      <inertia ixx="0.000000167" ixy="0" ixz="0" iyy="0.000000167" iyz="0" izz="0.000000167"/>
+    </inertial>
+    <visual>
+      <origin rpy="0 0 0" xyz="0.0 0.0 0.0"/>
+      <geometry>
+        <box size="0.01 0.01 0.01"/>
+      </geometry>
+    </visual>
+  </link>
+  <joint name="shoulder_psi_r" type="revolute" >
+    <parent link="right_shoulder_xx_link" />
+    <child link="right_shoulder_psi_link" />
+    <origin rpy="0 0.0 ${shoulder_psi_r}" xyz="0.0 0.0   0.0"/>
+    <axis xyz="0 0 1" />
+    <dynamics damping="0.005" />
+    <limit effort="101.0" lower="-1.0" upper="1.0" velocity="1.0"/>
+  </joint>
+  <link name="right_shoulder_psi_link">
+    <inertial>
+      <mass value="0.01"/>
+      <origin rpy="0 0 0" xyz="0 0.0 0.0"/>
+      <inertia ixx="0.000000167" ixy="0" ixz="0" iyy="0.000000167" iyz="0" izz="0.000000167"/>
+    </inertial>
+    <visual>
+      <origin rpy="0 0 0" xyz="0.0 0.0 0.0"/>
+      <geometry>
+        <box size="0.01 0.01 0.01"/>
+      </geometry>
+    </visual>
+  </link>
+  <joint name="shoulder_theta_r" type="revolute" >
+    <parent link="right_shoulder_psi_link"/>
+    <child link="arm_r_upper"/>
+    <origin rpy="${-shoulder_theta_r+pi} 0 0" xyz="0.0 0.0 0.0"/>
+    <axis xyz="-1 0 0" />
     <dynamics damping="0.5" />
-    <axis xyz="0 0 1"/>
     <limit effort="101.0" lower="-1.0" upper="1.0" velocity="1.0"/>
   </joint>
-  <link name="left_elbow_psi_link">
-    <inertial>
-      <mass value="0.01"/>
-      <origin rpy="0 0 0" xyz="0 0.0 0.0"/>
-      <inertia ixx="0.000000167" ixy="0" ixz="0" iyy="0.000000167" iyz="0" izz="0.000000167"/>
-    </inertial>
-    <visual>
-      <origin rpy="0 0 0" xyz="0.0 0.0 0.0"/>
-      <geometry>
-        <box size="0.01 0.01 0.01"/>
-      </geometry>
-    </visual>
-  </link>
-  <joint name="elbow_theta_l" type="revolute" >
-    <parent link="left_elbow_psi_link"/>
-    <child link="left_elbow_theta_link"/>
-    <origin rpy="0.0 ${elbow_theta_l}  0.0" xyz="-0.0 0.0  0.0"/>
+  <!-- 3D joint right elbow -->
+  <joint name="elbow_xx_r" type="revolute" >
+    <parent link="arm_r_upper"/>
+    <child link="right_elbow_theta_link"/>
+    <origin rpy="0 ${elbow_xx_r+pi/2}  0.0" xyz="-0.3 0.0  0.0"/>
     <axis xyz="0 1 0" />
     <dynamics damping="0.5" />
-    <limit effort="101.0" lower="-0.7" upper="2.0" velocity="1.0"/>
-  </joint>
-  <link name="left_elbow_theta_link">
-    <inertial>
-      <mass value="0.01"/>
-      <origin rpy="0 0 0" xyz="0 0.0 0.0"/>
-      <inertia ixx="0.000000167" ixy="0" ixz="0" iyy="0.000000167" iyz="0" izz="0.000000167"/>
-    </inertial>
-    <visual>
-      <origin rpy="0 0 0" xyz="0.0 0.0 0.0"/>
-      <geometry>
-        <box size="0.01 0.01 0.01"/>
-      </geometry>
-    </visual>
-  </link>
-  <joint name="elbow_xx_l" type="revolute" >
-    <parent link="left_elbow_theta_link"/>
-    <child link="arm_l_upper"/>
-    <origin rpy="${elbow_xx_l} 0.0  0.0" xyz="-0.0 0.0  0.0"/>
-    <axis xyz="1 0 0" />
+    <limit effort="101.0" lower="-${pi/2}" upper="${pi/2}" velocity="1.0"/>
+  </joint>
+  <link name="right_elbow_theta_link">
+    <inertial>
+      <mass value="0.01"/>
+      <origin rpy="0 0 0" xyz="0 0.0 0.0"/>
+      <inertia ixx="0.000000167" ixy="0" ixz="0" iyy="0.000000167" iyz="0" izz="0.000000167"/>
+    </inertial>
+    <visual>
+      <origin rpy="0 0 0" xyz="0.0 0.0 0.0"/>
+      <geometry>
+        <box size="0.01 0.01 0.01"/>
+      </geometry>
+    </visual>
+  </link>
+  <joint name="elbow_theta_r" type="revolute" >
+    <parent link="right_elbow_theta_link"/>
+    <child link="right_elbow_psi_link"/>
+    <origin rpy="0.0 0.0  ${elbow_theta_r}" xyz="0.0 0.0  0.0"/>
+    <axis xyz="0 0 1" />
     <dynamics damping="0.5" />
-    <limit effort="101.0" lower="-0.7" upper="2.0" velocity="1.0"/>
-  </joint>
-  <!-- 3D joint left shoulder -->
-  <joint name="shoulder_theta_l" type="revolute" >
-    <parent link="arm_l_upper"/>
-    <child link="left_shoulder_psi_link"/>
-    <origin rpy="0 ${shoulder_theta_l} 0" xyz="-0.35 0.0 0.0"/>
-    <axis xyz="0 1 0" />
-    <dynamics damping="0.005" />
+    <limit effort="101.0" lower="-2.0" upper="1.0" velocity="1.0"/>
+  </joint>
+  <link name="right_elbow_psi_link">
+    <inertial>
+      <mass value="0.01"/>
+      <origin rpy="0 0 0" xyz="0 0.0 0.0"/>
+      <inertia ixx="0.000000167" ixy="0" ixz="0" iyy="0.000000167" iyz="0" izz="0.000000167"/>
+    </inertial>
+    <visual>
+      <origin rpy="0 0 0" xyz="0.0 0.0 0.0"/>
+      <geometry>
+        <box size="0.01 0.01 0.01"/>
+      </geometry>
+    </visual>
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