Commit message: Completed first version of boot4

File: boot4_description/config/param.xacro (robot description, xacro)
@@ -18,6 +18,8 @@
 <xacro:property name="starboard_rowlock" value="-0.4939"/>
 <xacro:property name="port_rowlock" value="0.4939"/>
-<xacro:property name="starboard_oar" value="-0.1458"/>
-<xacro:property name="port_oar" value="0.1359"/>
+<xacro:property name="starboard_oar" value="-0.1258"/>
+<xacro:property name="port_oar" value="0.1159"/>
+<xacro:property name="starboard_blade" value="0.02"/>
+<xacro:property name="port_blade" value="0.0"/>
 <xacro:property name="hip2" value="-0.329"/>
 <xacro:property name="back_lh" value="0.0110"/>

File: boot4_description/urdf/boot.xacro (robot description, xacro)
@@ -86,5 +86,5 @@
     <parent link="starboard_oar_l"/>
     <child link="starboard_blade_l"/>
-    <origin rpy="0 0  0.0" xyz="0.0 0.0   -${outer}"/>
+    <origin rpy="0  ${starboard_blade}  0.0" xyz="0.0 0.0   -${outer}"/>
     <dynamics damping="0.005" />
     <axis xyz="0 1 0"/>
@@ -94,5 +94,5 @@
     <parent link="port_oar_l"/>
     <child link="port_blade_l"/>
-    <origin rpy="0.0  0 0.0" xyz="0.0 0.0   ${outer}"/>
+    <origin rpy="0.0  ${port_blade} 0.0" xyz="0.0 0.0   ${outer}"/>
     <dynamics damping="0.005" />
     <axis xyz="0 1 0"/>
@@ -179,7 +179,7 @@
   <link name="left_shoulder_xx_link">
     <inertial>
-      <mass value="0.01"/>
-      <origin rpy="0 0 0" xyz="0 0.0 0.0"/>
-      <inertia ixx="0.000000167" ixy="0" ixz="0" iyy="0.000000167" iyz="0" izz="0.000000167"/>
+      <mass value="1.0"/>
+      <origin rpy="0 0 0" xyz="0 0.0 0.0"/>
+      <inertia ixx="0.0000167" ixy="0" ixz="0" iyy="0.0000167" iyz="0" izz="0.0000167"/>
     </inertial>
     <visual>
@@ -200,7 +200,7 @@
   <link name="left_shoulder_psi_link">
     <inertial>
-      <mass value="0.01"/>
-      <origin rpy="0 0 0" xyz="0 0.0 0.0"/>
-      <inertia ixx="0.000000167" ixy="0" ixz="0" iyy="0.000000167" iyz="0" izz="0.000000167"/>
+      <mass value="1.0"/>
+      <origin rpy="0 0 0" xyz="0 0.0 0.0"/>
+      <inertia ixx="0.0000167" ixy="0" ixz="0" iyy="0.000167" iyz="0" izz="0.0000167"/>
     </inertial>
     <visual>
@@ -230,7 +230,7 @@
   <link name="left_elbow_theta_link">
     <inertial>
-      <mass value="0.01"/>
-      <origin rpy="0 0 0" xyz="0 0.0 0.0"/>
-      <inertia ixx="0.000000167" ixy="0" ixz="0" iyy="0.000000167" iyz="0" izz="0.000000167"/>
+      <mass value="1.0"/>
+      <origin rpy="0 0 0" xyz="0 0.0 0.0"/>
+      <inertia ixx="0.0000167" ixy="0" ixz="0" iyy="0.0000167" iyz="0" izz="0.0000167"/>
     </inertial>
     <visual>
@@ -251,7 +251,7 @@
   <link name="left_elbow_psi_link">
     <inertial>
-      <mass value="0.01"/>
-      <origin rpy="0 0 0" xyz="0 0.0 0.0"/>
-      <inertia ixx="0.000000167" ixy="0" ixz="0" iyy="0.000000167" iyz="0" izz="0.000000167"/>
+      <mass value="1.0"/>
+      <origin rpy="0 0 0" xyz="0 0.0 0.0"/>
+      <inertia ixx="0.0000167" ixy="0" ixz="0" iyy="0.0000167" iyz="0" izz="0.0000167"/>
     </inertial>
     <visual>
@@ -281,7 +281,7 @@
   <link name="handle_left_l2">
     <inertial>
-      <mass value="0.01"/>
-      <origin rpy="0 0 0" xyz="0 0.0 0.0"/>
-      <inertia ixx="0.000000167" ixy="0" ixz="0" iyy="0.000000167" iyz="0" izz="0.000000167"/>
+      <mass value="0.1"/>
+      <origin rpy="0 0 0" xyz="0 0.0 0.0"/>
+      <inertia ixx="0.00000167" ixy="0" ixz="0" iyy="0.00000167" iyz="0" izz="0.00000167"/>
     </inertial>
     <visual>
@@ -302,7 +302,7 @@
   <link name="handle_left_l1">
     <inertial>
-      <mass value="0.01"/>
-      <origin rpy="0 0 0" xyz="0 0.0 0.0"/>
-      <inertia ixx="0.000000167" ixy="0" ixz="0" iyy="0.000000167" iyz="0" izz="0.000000167"/>
+      <mass value="0.1"/>
+      <origin rpy="0 0 0" xyz="0 0.0 0.0"/>
+      <inertia ixx="0.00000167" ixy="0" ixz="0" iyy="0.00000167" iyz="0" izz="0.00000167"/>
     </inertial>
     <visual>
@@ -374,7 +374,7 @@
   <link name="right_shoulder_xx_link">
     <inertial>
-      <mass value="0.01"/>
-      <origin rpy="0 0 0" xyz="0 0.0 0.0"/>
-      <inertia ixx="0.000000167" ixy="0" ixz="0" iyy="0.000000167" iyz="0" izz="0.000000167"/>
+      <mass value="1.0"/>
+      <origin rpy="0 0 0" xyz="0 0.0 0.0"/>
+      <inertia ixx="0.0000167" ixy="0" ixz="0" iyy="0.0000167" iyz="0" izz="0.0000167"/>
     </inertial>
     <visual>
@@ -395,7 +395,7 @@
   <link name="right_shoulder_psi_link">
     <inertial>
-      <mass value="0.01"/>
-      <origin rpy="0 0 0" xyz="0 0.0 0.0"/>
-      <inertia ixx="0.000000167" ixy="0" ixz="0" iyy="0.000000167" iyz="0" izz="0.000000167"/>
+      <mass value="1.0"/>
+      <origin rpy="0 0 0" xyz="0 0.0 0.0"/>
+      <inertia ixx="0.0000167" ixy="0" ixz="0" iyy="0.0000167" iyz="0" izz="0.0000167"/>
     </inertial>
     <visual>
@@ -425,7 +425,7 @@
   <link name="right_elbow_theta_link">
     <inertial>
-      <mass value="0.01"/>
-      <origin rpy="0 0 0" xyz="0 0.0 0.0"/>
-      <inertia ixx="0.000000167" ixy="0" ixz="0" iyy="0.000000167" iyz="0" izz="0.000000167"/>
+      <mass value="1.0"/>
+      <origin rpy="0 0 0" xyz="0 0.0 0.0"/>
+      <inertia ixx="0.0000167" ixy="0" ixz="0" iyy="0.0000167" iyz="0" izz="0.0000167"/>
     </inertial>
     <visual>
@@ -446,7 +446,7 @@
   <link name="right_elbow_psi_link">
     <inertial>
-      <mass value="0.01"/>
-      <origin rpy="0 0 0" xyz="0 0.0 0.0"/>
-      <inertia ixx="0.000000167" ixy="0" ixz="0" iyy="0.000000167" iyz="0" izz="0.000000167"/>
+      <mass value="1.0"/>
+      <origin rpy="0 0 0" xyz="0 0.0 0.0"/>
+      <inertia ixx="0.0000167" ixy="0" ixz="0" iyy="0.0000167" iyz="0" izz="0.0000167"/>
     </inertial>
     <visual>
@@ -476,7 +476,7 @@
   <link name="handle_right_l2">
     <inertial>
-      <mass value="0.01"/>
-      <origin rpy="0 0 0" xyz="0 0.0 0.0"/>
-      <inertia ixx="0.000000167" ixy="0" ixz="0" iyy="0.000000167" iyz="0" izz="0.000000167"/>
+      <mass value="0.1"/>
+      <origin rpy="0 0 0" xyz="0 0.0 0.0"/>
+      <inertia ixx="0.00000167" ixy="0" ixz="0" iyy="0.00000167" iyz="0" izz="0.00000167"/>
     </inertial>
     <visual>
@@ -497,7 +497,7 @@
   <link name="handle_right_l1">
     <inertial>
-      <mass value="0.01"/>
-      <origin rpy="0 0 0" xyz="0 0.0 0.0"/>
-      <inertia ixx="0.000000167" ixy="0" ixz="0" iyy="0.000000167" iyz="0" izz="0.000000167"/>
+      <mass value="0.1"/>
+      <origin rpy="0 0 0" xyz="0 0.0 0.0"/>
+      <inertia ixx="0.00000167" ixy="0" ixz="0" iyy="0.00000167" iyz="0" izz="0.00000167"/>
     </inertial>
     <visual>
@@ -1233,3 +1233,21 @@
     </actuator>
   </transmission>
+  <transmission name="tran27">
+    <type>transmission_interface/SimpleTransmission</type>
+    <joint name="elbow_xx_l">
+      <hardwareInterface>hardware_interface/EffortJointInterface</hardwareInterface>
+    </joint>
+    <actuator name="motor27">
+      <mechanicalReduction>1</mechanicalReduction>
+    </actuator>
+  </transmission>
+  <transmission name="tran28">
+    <type>transmission_interface/SimpleTransmission</type>
+    <joint name="elbow_xx_r">
+      <hardwareInterface>hardware_interface/EffortJointInterface</hardwareInterface>
+    </joint>
+    <actuator name="motor28">
+      <mechanicalReduction>1</mechanicalReduction>
+    </actuator>
+  </transmission>
 </robot>

File: testing/crash_boot.urdf (robot description, URDF)
Before this commit: robot myboat, 9 links, 8 joints
Links:
- link left_shoulder_xx_link: mass 0.01 -> 0.1
Joints:
- joint LShoulderTheta: limit lower=-2.0 upper=1.0 effort=100.0 velocity=1.0 -> lower=-0.5 upper=0.5 effort=100.0 velocity=1.0
- joint shoulder_l: limit lower=-1.5 upper=0.5 effort=100.0 velocity=1.0 -> lower=-0.5 upper=0.5 effort=100.0 velocity=1.0

File: testing/crash_boot.xacro (robot description, xacro)
@@ -70,7 +70,7 @@
 <link name="left_shoulder_xx_link">
   <inertial>
-    <mass value="0.01"/>
+    <mass value="0.1"/>
     <origin rpy="0 0 0" xyz="0 0.0 0.0"/>
-    <inertia ixx="0.000000167" ixy="0" ixz="0" iyy="0.000000167" iyz="0" izz="0.000000167"/>
+    <inertia ixx="0.00000167" ixy="0" ixz="0" iyy="0.00000167" iyz="0" izz="0.00000167"/>
   </inertial>
   <visual>

Commit message: another step

File: boot4_description/config/param.xacro (robot description, xacro)
@@ -11,5 +11,11 @@
 <!--  rower -->
 <xacro:property name="weight" value="70"/>
-<xacro:property name="lenght" value="1.80"/>
+<xacro:property name="lowerleg" value="0.53"/>
+<xacro:property name="upperleg" value="0.45"/>
+  <!-- don't change leg for the moment, connection has don by hand -->
+<xacro:property name="back" value="0.60"/>
+<xacro:property name="shoulder" value="0.37"/>
+<xacro:property name="upperarm" value="0.35"/>
+<xacro:property name="lowerarm" value="0.35"/>
 <!--
  lengths of links, musle power?
@@ -23,22 +29,22 @@
 <xacro:property name="port_blade" value="0.0"/>
 <xacro:property name="hip2" value="-0.329"/>
-<xacro:property name="back_lh" value="0.0110"/>
-<xacro:property name="shoulder_l" value="-0.4209"/>
-<xacro:property name="shoulder_psi_l" value="0.1234"/>
-<xacro:property name="shoulder_theta_l" value="-0.3724"/>
-<xacro:property name="elbow_xx_l" value="0.1150"/>
-<xacro:property name="elbow_theta_l" value="0.1356"/>
-<xacro:property name="elbow_left" value="0.2445"/>
-<xacro:property name="handle_left_j3" value="0.0181"/>
-<xacro:property name="handle_left_j2" value="-0.0254"/>
-<xacro:property name="handle_left_j1" value="-0.0396"/>
-<xacro:property name="shoulder_r" value="-0.4208"/>
-<xacro:property name="shoulder_psi_r" value="0.1086"/>
-<xacro:property name="shoulder_theta_r" value="-0.3731"/>
-<xacro:property name="elbow_xx_r" value="0.0271"/>
-<xacro:property name="elbow_theta_r" value="0.1332"/>
-<xacro:property name="elbow_right" value="0.1927"/>
-<xacro:property name="handle_right_j3" value="0.0001"/>
-<xacro:property name="handle_right_j2" value="-0.0074"/>
-<xacro:property name="handle_right_j1" value="-0.1168"/>
+<xacro:property name="back_lh" value="0.0182"/>
+<xacro:property name="shoulder_l" value="-0.5674"/>
+<xacro:property name="shoulder_psi_l" value="0.1546"/>
+<xacro:property name="shoulder_theta_l" value="-0.3847"/>
+<xacro:property name="elbow_xx_l" value="0.1878"/>
+<xacro:property name="elbow_theta_l" value="0.1514"/>
+<xacro:property name="elbow_left" value="0.2139"/>
+<xacro:property name="handle_left_j3" value="0.0805"/>
+<xacro:property name="handle_left_j2" value="-0.0566"/>
+<xacro:property name="handle_left_j1" value="-0.0905"/>
+<xacro:property name="shoulder_r" value="-0.5573"/>
+<xacro:property name="shoulder_psi_r" value="0.1429"/>
+<xacro:property name="shoulder_theta_r" value="-0.3884"/>
+<xacro:property name="elbow_xx_r" value="0.0939"/>
+<xacro:property name="elbow_theta_r" value="0.1502"/>
+<xacro:property name="elbow_right" value="0.1662"/>
+<xacro:property name="handle_right_j3" value="0.0429"/>
+<xacro:property name="handle_right_j2" value="-0.0329"/>
+<xacro:property name="handle_right_j1" value="-0.2017"/>
 </robot>

File: boot4_description/urdf/boot.xacro (robot description, xacro)
@@ -57,5 +57,5 @@
     <dynamics damping="0.005" />
     <axis xyz="0 0 1"/>
-    <limit effort="101.0" lower="-0.4" upper="1.4" velocity="1.0"/>
+    <limit effort="101.0" lower="-0.4" upper="2.0" velocity="1.0"/>
   </joint>
   <joint name="port_rowlock" type="${port_rowlock_type}">
@@ -65,5 +65,5 @@
     <dynamics damping="0.005" />
     <axis xyz="0 0 1"/>
-    <limit effort="101.0" lower="-1.4" upper="1.4" velocity="1.0"/>
+    <limit effort="101.0" lower="-2.0" upper="0.4" velocity="1.0"/>
   </joint>
   <joint name="starboard_oar" type="${starboard_oar_type}">
@@ -110,5 +110,5 @@
     <parent link="skiff"/>
     <child link="seat"/>
-    <origin rpy="0 0 0" xyz="-3.49514 0.0 0.1"/>
+    <origin rpy="0 0 0" xyz="-3.44455 0.0 0.1"/>
     <dynamics damping="0.005" />
     <axis xyz="1 0 0"/>
@@ -118,5 +118,5 @@
     <parent link="footplate"/>
     <child link="lowerleg"/>
-    <origin rpy="0.0  0.1001675 0.0" xyz="0.0 0.0   0.0"/>
+    <origin rpy="0.0  0.1071 0.0" xyz="0.0 0.0   0.0"/>
     <dynamics damping="0.005" />
     <axis xyz="0 1 0"/>
@@ -175,5 +175,5 @@
     <axis xyz="0 -1 0" />
     <dynamics damping="0.005" />
-    <limit effort="101.0" lower="-1.0" upper="1.0" velocity="1.0"/>
+    <limit effort="101.0" lower="-1.0" upper="2.2" velocity="1.0"/>
   </joint>
   <link name="left_shoulder_xx_link">
@@ -226,5 +226,5 @@
     <axis xyz="0 1 0" />
     <dynamics damping="0.5" />
-    <limit effort="101.0" lower="-${pi/2}" upper="${pi/2}" velocity="1.0"/>
+    <limit effort="101.0" lower="-${pi/2+0.2}" upper="${pi/2}" velocity="1.0"/>
   </joint>
   <link name="left_elbow_theta_link">
@@ -370,5 +370,5 @@
     <axis xyz="0 -1 0" />
     <dynamics damping="0.005" />
-    <limit effort="101.0" lower="-1.0" upper="1.0" velocity="1.0"/>
+    <limit effort="101.0" lower="-2.2" upper="1.0" velocity="1.0"/>
   </joint>
   <link name="right_shoulder_xx_link">
@@ -421,5 +421,5 @@
     <axis xyz="0 1 0" />
     <dynamics damping="0.5" />
-    <limit effort="101.0" lower="-${pi/2}" upper="${pi/2}" velocity="1.0"/>
+    <limit effort="101.0" lower="-${pi/2+0.2}" upper="${pi/2}" velocity="1.0"/>
   </joint>
   <link name="right_elbow_theta_link">
@@ -769,17 +769,17 @@
     <inertial>
       <mass value="1.0"/>
-      <origin rpy="0 0 0" xyz="-0.25 0.0 0.0"/>
+      <origin rpy="0 0 0" xyz="-${lowerleg/2} 0.0 0.0"/>
       <inertia ixx="0.00041" ixy="0" ixz="0" iyy="0.021" iyz="0" izz="0.021"/>
     </inertial>
     <collision>
-      <origin rpy="0 0 0" xyz="-0.25 0.0   0.0"/>
-      <geometry>
-        <box size="0.5 0.05 0.05"/>
-      </geometry>
-    </collision>
-    <visual>
-      <origin rpy="0 0 0" xyz="-0.25 0.0   0.0"/>
-      <geometry>
-        <box size="0.5 0.05 0.05"/>
+      <origin rpy="0 0 0" xyz="-${lowerleg/2} 0.0   0.0"/>
+      <geometry>
+        <box size="${lowerleg} 0.05 0.05"/>
+      </geometry>
+    </collision>
+    <visual>
+      <origin rpy="0 0 0" xyz="-${lowerleg/2} 0.0   0.0"/>
+      <geometry>
+        <box size="${lowerleg} 0.05 0.05"/>
       </geometry>
     </visual>
@@ -790,17 +790,17 @@
     <inertial>
       <mass value="1.0"/>
-      <origin rpy="0 0 0" xyz="-0.125 0.0 0.0"/>
+      <origin rpy="0 0 0" xyz="-${upperleg/4} 0.0 0.0"/>
       <inertia ixx="0.00041" ixy="0" ixz="0" iyy="0.0054" iyz="0" izz="0.0054"/>
     </inertial>
     <collision>
-      <origin rpy="0 0 0" xyz="-0.125  0.0   0.0"/>
-      <geometry>
-        <box size="0.25 0.05 0.05"/>
-      </geometry>
-    </collision>
-    <visual>
-      <origin rpy="0 0 0" xyz="-0.125   0.0   0.0"/>
-      <geometry>
-        <box size="0.25 0.05 0.05"/>
+      <origin rpy="0 0 0" xyz="-${upperleg/4}  0.0   0.0"/>
+      <geometry>
+        <box size="${upperleg/2} 0.05 0.05"/>
+      </geometry>
+    </collision>
+    <visual>
+      <origin rpy="0 0 0" xyz="-${upperleg/4}   0.0   0.0"/>
+      <geometry>
+        <box size="${upperleg/2} 0.05 0.05"/>
       </geometry>
     </visual>
@@ -809,17 +809,17 @@
     <inertial>
       <mass value="1.0"/>
-      <origin rpy="0 0 0" xyz="0.125 0.0 0.0"/>
+      <origin rpy="0 0 0" xyz="${upperleg/4} 0.0 0.0"/>
       <inertia ixx="0.00041" ixy="0" ixz="0" iyy="0.0054" iyz="0" izz="0.0054"/>
     </inertial>
     <collision>
-      <origin rpy="0 0 0" xyz="0.125  0.0   0.0"/>
-      <geometry>
-        <box size="0.25 0.05 0.05"/>
-      </geometry>
-    </collision>
-    <visual>
-      <origin rpy="0 0 0" xyz="0.125 0.0   0.0"/>
-      <geometry>
-        <box size="0.25 0.05 0.05"/>
+      <origin rpy="0 0 0" xyz="${upperleg/4}  0.0   0.0"/>
+      <geometry>
+        <box size="${upperleg/2} 0.05 0.05"/>
+      </geometry>
+    </collision>
+    <visual>
+      <origin rpy="0 0 0" xyz="${upperleg/4} 0.0   0.0"/>
+      <geometry>
+        <box size="${upperleg/2} 0.05 0.05"/>
       </geometry>
     </visual>
