Commit message: updated pos.py

File: boot4_description/urdf/boot.xacro (robot description, xacro)
@@ -370,5 +370,5 @@
     <axis xyz="0 -1 0" />
     <dynamics damping="0.005" />
-    <limit effort="101.0" lower="-2.2" upper="1.0" velocity="1.0"/>
+    <limit effort="101.0" lower="-1.0" upper="2.2" velocity="1.0"/>
   </joint>
   <link name="right_shoulder_xx_link">
@@ -493,5 +493,5 @@
     <dynamics damping="0.005" />
     <axis xyz="-1 0 0"/>
-    <limit effort="101.0" lower="-1" upper="1" velocity="1.0"/>
+    <limit effort="101.0" lower="-1" upper="1.2" velocity="1.0"/>
   </joint>
   <link name="handle_right_l1">
