Commit message: New testcase with instabilities

File: boot4_description/urdf/boot.urdf (robot description, URDF)
Before this commit: robot myboat, 41 links, 40 joints
Links:
- removed link shoulder_left
- removed link shoulder_right
- added link port_handle_l, mass 1.0; visual cylinder length=0.1 radius=0.02
- added link starboard_handle_l, mass 1.0; visual cylinder length=0.1 radius=0.02
- link Ldummy_link_1: mass 0.01 -> 0.1
- link Ldummy_link_2: mass 0.01 -> 0.1
- link Rdummy_link_1: mass 0.01 -> 0.1
- link Rdummy_link_2: mass 0.01 -> 0.1
- link arm_l_lower: geometry collision box size=0.35 0.05 0.05; visual box size=0.35 0.05 0.05
- link arm_l_upper: geometry collision box size=0.30 0.05 0.05; visual box size=0.30 0.05 0.05
- link arm_r_lower: geometry collision box size=0.35 0.05 0.05; visual box size=0.35 0.05 0.05
- link arm_r_upper: geometry collision box size=0.3 0.05 0.05; visual box size=0.3 0.05 0.05
- link handle_left_l1: mass 0.01 -> 0.1
- link handle_left_l2: mass 0.01 -> 0.1
- link handle_right_l1: mass 0.01 -> 0.1
- link handle_right_l2: mass 0.01 -> 0.1
- link l1: mass 0.01 -> 0.1; geometry visual box size=0.01 0.01 0.05
- link l2: mass 0.01 -> 0.1
- link left_elbow_psi_link: mass 0.01 -> 1.0
- link left_elbow_theta_link: mass 0.01 -> 1.0
- link left_shoulder_psi_link: mass 0.01 -> 1.0
- link left_shoulder_xx_link: mass 0.01 -> 1.0
- link lowerleg: geometry collision box size=0.53 0.05 0.05; visual box size=0.53 0.05 0.05
- link right_elbow_psi_link: mass 0.01 -> 1.0
- link right_elbow_theta_link: mass 0.01 -> 1.0
- link right_shoulder_psi_link: mass 0.01 -> 1.0
- link right_shoulder_xx_link: mass 0.01 -> 1.0
- link shoulder_link: geometry collision box size=0.05 0.4 0.05; visual box size=0.05 0.4 0.05
- link upperleg_1: geometry collision box size=0.225 0.05 0.05; visual box size=0.225 0.05 0.05
- link upperleg_2: geometry collision box size=0.225 0.05 0.05; visual box size=0.225 0.05 0.05
Joints:
- removed joint prism
- added joint the_course: type prismatic, parent world, child l1, origin xyz=0 0 0.0 rpy=0 0 0, axis 1 0 0, limit lower=0 upper=100 effort=101.0 velocity=0.5
- joint Ldummy_1: origin xyz=0.0 0.1 0.0 rpy=0 0 0.0 -> xyz=0 0 0.77  rpy=0 3.14159265359 1.57079632679; parent shoulder_link -> starboard_oar_l
- joint Ldummy_2: origin xyz=0.0 0.1 0.0 rpy=0 0 3.14159265359  -> xyz=0.0 0.0 0.075 rpy=0 0 0 ; parent shoulder_left -> starboard_handle_l
- joint Rdummy_1: origin xyz=0.0 -0.1 0.0 rpy=0 0 0.0 -> xyz=0.0 0.0 -0.77 rpy=0 0 -1.57079632679; parent shoulder_link -> port_oar_l
- joint Rdummy_2: origin xyz=0.0 -0.1 0.0 rpy=3.14159265359 0  0.0 -> xyz=0.0 0.0 -0.075 rpy=3.14159265359 0  0.0; parent shoulder_right -> port_handle_l
- joint back_lh: origin xyz=0.25 0.0   0.0 rpy=0  0.011 0.0 -> xyz=0.25 0.0   0.0 rpy=0  0.0182 0.0
- joint elbow_left: axis 0 0 1 -> 1 0 0; child left_elbow_psi_link -> arm_l_lower; origin xyz=-0.4 0.0 0.0 rpy=0 0 -1.9207 -> xyz=-0.0 0.0 0.0 rpy=0.2139 0 0; parent arm_l_lower -> left_elbow_psi_link
- joint elbow_right: axis 0 0 1 -> -1 0 0; child right_elbow_psi_link -> arm_r_lower; origin xyz=-0.4 0.0 0.0 rpy=0 0 1.2894 -> xyz=0.0 0.0 0.0 rpy=-0.1662 0 0; parent arm_r_lower -> right_elbow_psi_link
- joint elbow_theta_l: axis 0 1 0 -> 0 0 -1; child left_elbow_theta_link -> left_elbow_psi_link; origin xyz=-0.0 0.0  0.0 rpy=0.0 0.0003  0.0 -> xyz=-0.0 0.0  0.0 rpy=0 0.0  -0.1514; parent left_elbow_psi_link -> left_elbow_theta_link
- joint elbow_theta_r: axis 0 1 0 -> 0 0 1; child right_elbow_theta_link -> right_elbow_psi_link; origin xyz=0.0 0.0  0.0 rpy=0.0 0.0288  0.0 -> xyz=0.0 0.0  0.0 rpy=0.0 0.0  0.1502; parent right_elbow_psi_link -> right_elbow_theta_link
- joint elbow_xx_l: axis 1 0 0 -> 0 1 0; child arm_l_upper -> left_elbow_theta_link; limit lower=-0.7 upper=2.0 effort=101.0 velocity=1.0 -> lower=-1.77079632679 upper=1.57079632679 effort=101.0 velocity=1.0; origin xyz=-0.0 0.0  0.0 rpy=0.9796 0.0  0.0 -> xyz=-0.3 0.0  0.0 rpy= 3.14159265359 -1.75859632679  0.0; parent left_elbow_theta_link -> arm_l_upper
- joint elbow_xx_r: axis -1 0 0 -> 0 1 0; child arm_r_upper -> right_elbow_theta_link; limit lower=-1.0 upper=2.0 effort=101.0 velocity=1.0 -> lower=-1.77079632679 upper=1.57079632679 effort=101.0 velocity=1.0; origin xyz=0.0 0.0  0.0 rpy=0.2775 0.0  0.0 -> xyz=-0.3 0.0  0.0 rpy=0 1.66469632679  0.0; parent right_elbow_theta_link -> arm_r_upper
- joint fp_ll: origin xyz=0.0 0.0   0.0 rpy=0.0  0.1001675 0.0 -> xyz=0.0 0.0   0.0 rpy=0.0  0.1071 0.0
- joint handle_left_j1: axis 1 0 0 -> 0 0 1; child handle_left_l1 -> starboard_handle_l; origin xyz=0 0.0 0.87 rpy=0.1425 0 1.57079632679 -> xyz=0 0.0 0 rpy=0 0 -0.0905; parent starboard_oar_l -> handle_left_l1
- joint handle_left_j2: axis 0 0 1 -> 1 0 0; child handle_left_l2 -> handle_left_l1; origin xyz=0 0.0 0.0 rpy=0 0 0.0807 -> xyz=0 0.0 0.0 rpy=-0.0566 0 0; parent handle_left_l1 -> handle_left_l2
- joint handle_left_j3: child arm_l_lower -> handle_left_l2; origin xyz=0 0.0 0.0 rpy=0 -0.0503 0 -> xyz=-0.35 0.0 0.0 rpy=1.57079632679 0.0805 0; parent handle_left_l2 -> arm_l_lower
- joint handle_right_j1: axis -1 0 0 -> 0 0 1; child handle_right_l1 -> port_handle_l; origin xyz=0 0.0 -0.87 rpy=-0.0496 0 1.57079632679 -> xyz=0 0.0 0 rpy=0 0 -0.2017; parent port_oar_l -> handle_right_l1
- joint handle_right_j2: axis 0 0 1 -> -1 0 0; child handle_right_l2 -> handle_right_l1; limit lower=-1 upper=1 effort=101.0 velocity=1.0 -> lower=-1 upper=1.2 effort=101.0 velocity=1.0; origin xyz=0 0.0 0.0 rpy=0 0 0.0074 -> xyz=0 0.0 0.0 rpy=0.0329 0 0; parent handle_right_l1 -> handle_right_l2
- joint handle_right_j3: child arm_r_lower -> handle_right_l2; origin xyz=0 0.0 0.0 rpy=0 -0.0084 0 -> xyz=-0.35 0.0 0.0 rpy=1.57079632679 -0.0429 0; parent handle_right_l2 -> arm_r_lower
- joint port_blade: origin xyz=0.0 0.0   2.0 rpy=0.0  0 0.0 -> xyz=0.0 0.0   2.0 rpy=0.0  0.0 0.0
- joint port_oar: origin xyz=0.0 0.0   0.02 rpy=0.0  1.70669632679 -1.57079632679 -> xyz=0.0 0.0   0.02 rpy=0.0  1.68669632679 -1.57079632679
- joint port_rowlock: limit lower=-1.4 upper=1.4 effort=101.0 velocity=1.0 -> lower=-2.0 upper=0.4 effort=101.0 velocity=1.0
- joint rev1: origin xyz=0.0 0 -0.2 rpy=0 1.57079632679 0 -> xyz=0.0 0 0.05 rpy=0 1.57079632679 0
- joint shoulder_l: axis 0 0 1 -> 0 -1 0; child shoulder_left -> left_shoulder_xx_link; limit lower=-1.0 upper=1.0 effort=101.0 velocity=1.0 -> lower=-1.0 upper=2.2 effort=101.0 velocity=1.0; origin xyz=0.0 0.0   0.0 rpy=0.0 0.0 0.1516 -> xyz=0.0 0.2   0.0 rpy=0.0 0.5674 0.0; parent left_shoulder_xx_link -> shoulder_link
- joint shoulder_psi_l: axis 1 0 0 -> 0 0 -1; child left_shoulder_xx_link -> left_shoulder_psi_link; origin xyz=0.0 0.0   0.0 rpy=-0.0182 0.0 0.0 -> xyz=0.0 0.0   0.0 rpy=0 0.0 -0.1546; parent left_shoulder_psi_link -> left_shoulder_xx_link
- joint shoulder_psi_r: axis 1 0 0 -> 0 0 1; child right_shoulder_xx_link -> right_shoulder_psi_link; origin xyz=0.0 0.0   0.0 rpy=3.7462 0.0 0.0 -> xyz=0.0 0.0   0.0 rpy=0 0.0 0.1429; parent right_shoulder_psi_link -> right_shoulder_xx_link
- joint shoulder_r: axis 0 0 1 -> 0 -1 0; child shoulder_right -> right_shoulder_xx_link; limit lower=-1.0 upper=1.0 effort=101.0 velocity=1.0 -> lower=-1.0 upper=2.2 effort=101.0 velocity=1.0; origin xyz=0.0 -0.0   0.0 rpy=0.0 0  0.5698 -> xyz=0.0 -0.2   0.0 rpy=0.0 0.5573  0; parent right_shoulder_xx_link -> shoulder_link
- joint shoulder_theta_l: axis 0 1 0 -> 1 0 0; child left_shoulder_psi_link -> arm_l_upper; origin xyz=-0.35 0.0 0.0 rpy=0 0.5435 0 -> xyz=0.0 0.0 0.0 rpy=-0.3847 0 0; parent arm_l_upper -> left_shoulder_psi_link
- joint shoulder_theta_r: axis 0 -1 0 -> -1 0 0; child right_shoulder_psi_link -> arm_r_upper; origin xyz=0.35 0.0 0.0 rpy=3.14159265359 0.7384 0 -> xyz=0.0 0.0 0.0 rpy=3.52999265359 0 0; parent arm_r_upper -> right_shoulder_psi_link
- joint sliding: origin xyz=-3.49514 0.0 0.1 rpy=0 0 0 -> xyz=-3.44455 0.0 0.1 rpy=0 0 0
- joint starboard_blade: origin xyz=0.0 0.0   -2.0 rpy=0 0  0.0 -> xyz=0.0 0.0   -2.0 rpy=0  0.02  0.0
- joint starboard_oar: origin xyz=0.0 0.0   0.02 rpy=0.0  1.42499632679 -1.57079632679 -> xyz=0.0 0.0   0.02 rpy=0.0  1.44499632679 -1.57079632679
- joint starboard_rowlock: limit lower=-0.4 upper=1.4 effort=101.0 velocity=1.0 -> lower=-0.4 upper=2.0 effort=101.0 velocity=1.0
