Commit message: Simplified test2

File: test2/boot.urdf (robot description, URDF)
Before this commit: robot myboat, 8 links, 7 joints
Links:
- removed link left_shoulder_psi_link
- removed link left_shoulder_xx_link
- link arm_l_lower: geometry visual box size=0.35 0.05 0.05
- link arm_l_upper: geometry visual box size=0.30 0.05 0.05
- link shoulder_link: geometry visual box size=0.05 0.4 0.05
Joints:
- removed joint shoulder_l
- removed joint shoulder_psi_l
- joint elbow_theta_l: type revolute -> fixed
- joint shoulder_theta_l: origin xyz=0.0 0.0 0.0 rpy=-0.3847 0 0 -> xyz=0.0 0.0 0.0 rpy=0.3847 0 0; parent left_shoulder_psi_link -> shoulder_link

Commit message: Use dart with gazebo

File: test2/boot.urdf (robot description, URDF)
Before this commit: robot myboat, 6 links, 5 joints
Joints:
- joint elbow_theta_l: type fixed -> revolute
- joint shoulder: type fixed -> revolute
